File: Viehmann_GPS_2015.brd (EAGLE design)
At the start: 100 x 80 mm, 12 parts, among them J1 U.FL

Commit message: Finished first rev of the gps board
Shout out to board space and Judah
Parts:
- added C4, C5: 1uF, SparkFun-Capacitors:1206
- added U$1: V_REG_LD1117#50, SparkFun-PowerIC:SOT223
- added VIN: (no value), SparkFun-Connectors:1X02
- moved J1 93.5 mm to (42.5, 4.50), turned to 180 degrees
- moved R3 81.6 mm to (29.8, 8.38), turned to 180 degrees
- moved D1 67.7 mm to (35.4, 8.38)
- moved R2 66.8 mm to (20.9, 13.9)
- moved R1 64.6 mm to (21.1, 10.5)
- moved C3 55.7 mm to (21.7, 19.8), turned to 90 degrees
- moved U1 55.5 mm to (33.1, 18.3)
- moved CR1220 55.1 mm to (28.9, 6.58), flipped to the bottom, turned to 180 degrees
- moved C2 50.6 mm to (26.2, 29.5), turned to 180 degrees
- moved C1 44.0 mm to (21.9, 25.8), turned to 90 degrees
- renumbered JP1 to LEFTSIDE, JP2 to RIGHSIDE
Connections:
- new net 5V: C5.1, LEFTSIDE.2, U$1.3
- new net VIN: C4.1, U$1.1, VIN.1
- net GND: now also C4.2, C5.2, U$1.2, VIN.2
Routing:
- net GND: track 0.00 -> 42.1 mm, vias 0 -> 6
- net NRESET: track 0.00 -> 29.4 mm, vias 0 -> 1
- net DATA_OUT: track 0.00 -> 23.6 mm
- net DATA_IN: track 0.00 -> 22.3 mm
- net VBACKUP: track 0.00 -> 17.9 mm, vias 0 -> 1
- net N$1: track 0.00 -> 14.6 mm
- net VIN: track 0.00 -> 12.7 mm
- net 5V: track 0.00 -> 9.31 mm
- net EX_ANT: track 0.00 -> 7.85 mm
- net N$4: track 0.00 -> 3.80 mm
- net N$3: track 0.00 -> 3.65 mm
- net N$2: track 0.00 -> 2.76 mm
- added copper zone on layer 1, net 3.3V
- added copper zone on layer 16, net GND
Other:
- board size 100 x 80 mm -> 53.7 x 33 mm
- board text added: "+"
- board text added: "-"
- board text added: "DESING TEAM"
- board text added: "GPS"
- board text added: "I WILL KILL YOU IF YOU REMOVE THIS"
- board text added: "JUDAH RULES"
- board text added: "MARS ROVER"
