File: Viehmann_GPS_2015.sch (EAGLE design)
At the start: 12 parts, among them J1 U.FL

Commit message: Finished first rev of the gps board
Shout out to board space and Judah
Parts:
- added C4, C5: 1uF, SparkFun-Capacitors:CAP1206
- added U$1: V_REG_LD1117#50, SparkFun-PowerIC:V_REG_MIC2920
- added VIN: M02PTH, SparkFun-Connectors:M02PTH
- renumbered JP1 to LEFTSIDE, JP2 to RIGHSIDE
Connections:
- new net 5V: C5.1, LEFTSIDE.2, U$1.OUT
- new net VIN: C4.1, U$1.IN, VIN.1
- net GND: now also C4.2, C5.2, U$1.GND, VIN.2
Changed lines of the file:
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@@
 <part name="GND1" library="SparkFun-Aesthetics" deviceset="GND" device=""/>
 <part name="GND2" library="SparkFun-Aesthetics" deviceset="GND" device=""/>
-<part name="JP1" library="SparkFun-Connectors" deviceset="M10X2" device=""/>
-<part name="JP2" library="SparkFun-Connectors" deviceset="M10X2" device=""/>
+<part name="LEFTSIDE" library="SparkFun-Connectors" deviceset="M10X2" device=""/>
+<part name="RIGHSIDE" library="SparkFun-Connectors" deviceset="M10X2" device=""/>
 <part name="SUPPLY2" library="SparkFun-Aesthetics" deviceset="3.3V" device=""/>
 <part name="GND3" library="SparkFun-Aesthetics" deviceset="GND" device=""/>
@@
 <part name="GND6" library="SparkFun-Aesthetics" deviceset="GND" device=""/>
 <part name="GND7" library="SparkFun-Aesthetics" deviceset="GND" device=""/>
+<part name="GND8" library="SparkFun-Aesthetics" deviceset="GND" device=""/>
+<part name="SUPPLY3" library="SparkFun-Aesthetics" deviceset="5V" device=""/>
+<part name="SUPPLY4" library="SparkFun-Aesthetics" deviceset="5V" device=""/>
+<part name="SUPPLY5" library="SparkFun-Aesthetics" deviceset="VIN" device=""/>
+<part name="C4" library="SparkFun-Capacitors" deviceset="CAP" device="1206" value="1uF"/>
+<part name="C5" library="SparkFun-Capacitors" deviceset="CAP" device="1206" value="1uF"/>
+<part name="VIN" library="SparkFun-Connectors" deviceset="M02" device="PTH" value=""/>
+<part name="SUPPLY6" library="SparkFun-Aesthetics" deviceset="VIN" device=""/>
+<part name="GND9" library="SparkFun-Aesthetics" deviceset="GND" device=""/>
+<part name="U$1" library="SparkFun-PowerIC" deviceset="V_REG_MIC2920" device="" value="V_REG_LD1117#50"/>
 </parts>
 <sheets>
@@
 <instance part="GND1" gate="1" x="35.56" y="53.34"/>
 <instance part="GND2" gate="1" x="40.64" y="71.12"/>
-<instance part="JP1" gate="G$1" x="-7.62" y="99.06"/>
-<instance part="JP2" gate="G$1" x="-7.62" y="66.04"/>
+<instance part="LEFTSIDE" gate="G$1" x="-7.62" y="99.06"/>
+<instance part="RIGHSIDE" gate="G$1" x="-7.62" y="66.04"/>
 <instance part="SUPPLY2" gate="G$1" x="-20.32" y="114.3"/>
 <instance part="GND3" gate="1" x="71.12" y="22.86"/>
@@
 <instance part="GND6" gate="1" x="10.16" y="96.52"/>
 <instance part="GND7" gate="1" x="10.16" y="66.04"/>
+<instance part="GND8" gate="1" x="50.8" y="99.06"/>
+<instance part="SUPPLY3" gate="G$1" x="60.96" y="119.38"/>
+<instance part="SUPPLY4" gate="G$1" x="7.62" y="114.3"/>
+<instance part="SUPPLY5" gate="G$1" x="40.64" y="121.92"/>
+<instance part="C4" gate="G$1" x="40.64" y="109.22"/>
+<instance part="C5" gate="G$1" x="60.96" y="109.22"/>
+<instance part="VIN" gate="G$1" x="33.02" y="149.86" rot="R180"/>
+<instance part="SUPPLY6" gate="G$1" x="20.32" y="152.4"/>
+<instance part="GND9" gate="1" x="20.32" y="139.7"/>
+<instance part="U$1" gate="G$1" x="50.8" y="116.84"/>
 </instances>
 <busses>
@@
 </segment>
 <segment>
-<pinref part="JP1" gate="G$1" pin="1"/>
+<pinref part="LEFTSIDE" gate="G$1" pin="1"/>
 <pinref part="SUPPLY2" gate="G$1" pin="3.3V"/>
 <wire x1="-15.24" y1="109.22" x2="-20.32" y2="109.22" width="0.1524" layer="91"/>
@@
 </segment>
 <segment>
-<pinref part="JP1" gate="G$1" pin="4"/>
+<pinref part="LEFTSIDE" gate="G$1" pin="4"/>
 <wire x1="0" y1="106.68" x2="10.16" y2="106.68" width="0.1524" layer="91"/>
 <wire x1="10.16" y1="106.68" x2="10.16" y2="99.06" width="0.1524" layer="91"/>
@@
 </segment>
 <segment>
-<pinref part="JP2" gate="G$1" pin="2"/>
+<pinref part="RIGHSIDE" gate="G$1" pin="2"/>
 <wire x1="0" y1="76.2" x2="10.16" y2="76.2" width="0.1524" layer="91"/>
 <wire x1="10.16" y1="76.2" x2="10.16" y2="68.58" width="0.1524" layer="91"/>
 <pinref part="GND7" gate="1" pin="GND"/>
 </segment>
+<segment>
+<pinref part="GND8" gate="1" pin="GND"/>
+<pinref part="C4" gate="G$1" pin="2"/>
+<wire x1="50.8" y1="106.68" x2="50.8" y2="101.6" width="0.1524" layer="91"/>
+<wire x1="40.64" y1="106.68" x2="50.8" y2="106.68" width="0.1524" layer="91"/>
+<junction x="50.8" y="106.68"/>
+<pinref part="C5" gate="G$1" pin="2"/>
+<wire x1="60.96" y1="106.68" x2="50.8" y2="106.68" width="0.1524" layer="91"/>
+<pinref part="U$1" gate="G$1" pin="GND"/>
+<wire x1="50.8" y1="109.22" x2="50.8" y2="106.68" width="0.1524" layer="91"/>
+</segment>
+<segment>
+<pinref part="VIN" gate="G$1" pin="2"/>
+<pinref part="GND9" gate="1" pin="GND"/>
+<wire x1="25.4" y1="147.32" x2="20.32" y2="147.32" width="0.1524" layer="91"/>
+<wire x1="20.32" y1="147.32" x2="20.32" y2="142.24" width="0.1524" layer="91"/>
+</segment>
 </net>
 <net name="NRESET" class="0">
@@
 </segment>
 <segment>
-<pinref part="JP1" gate="G$1" pin="3"/>
+<pinref part="LEFTSIDE" gate="G$1" pin="3"/>
 <wire x1="-15.24" y1="106.68" x2="-25.4" y2="106.68" width="0.1524" layer="91"/>
 <label x="-22.86" y="106.68" size="1.778" layer="95"/>
@@
 </segment>
 <segment>
-<pinref part="JP1" gate="G$1" pin="5"/>
+<pinref part="LEFTSIDE" gate="G$1" pin="5"/>
 <wire x1="-15.24" y1="104.14" x2="-25.4" y2="104.14" width="0.1524" layer="91"/>
 <label x="-22.86" y="104.14" size="1.778" layer="95"/>
@@
 </segment>
 <segment>
-<pinref part="JP1" gate="G$1" pin="7"/>
+<pinref part="LEFTSIDE" gate="G$1" pin="7"/>
 <wire x1="-15.24" y1="101.6" x2="-25.4" y2="101.6" width="0.1524" layer="91"/>
 <label x="-22.86" y="101.6" size="1.778" layer="95"/>
@@
 </segment>
 </net>
+<net name="VIN" class="0">
+<segment>
+<pinref part="SUPPLY5" gate="G$1" pin="VIN"/>
+<wire x1="40.64" y1="114.3" x2="40.64" y2="116.84" width="0.1524" layer="91"/>
+<pinref part="C4" gate="G$1" pin="1"/>
+<pinref part="U$1" gate="G$1" pin="IN"/>
+<wire x1="40.64" y1="116.84" x2="40.64" y2="121.92" width="0.1524" layer="91"/>
+<wire x1="43.18" y1="116.84" x2="40.64" y2="116.84" width="0.1524" layer="91"/>
+<junction x="40.64" y="116.84"/>
+</segment>
+<segment>
+<pinref part="VIN" gate="G$1" pin="1"/>
+<pinref part="SUPPLY6" gate="G$1" pin="VIN"/>
+<wire x1="25.4" y1="149.86" x2="20.32" y2="149.86" width="0.1524" layer="91"/>
+<wire x1="20.32" y1="149.86" x2="20.32" y2="152.4" width="0.1524" layer="91"/>
+</segment>
+</net>
+<net name="5V" class="0">
+<segment>
+<pinref part="SUPPLY3" gate="G$1" pin="5V"/>
+<pinref part="C5" gate="G$1" pin="1"/>
+<wire x1="60.96" y1="119.38" x2="60.96" y2="116.84" width="0.1524" layer="91"/>
+<pinref part="U$1" gate="G$1" pin="OUT"/>
+<wire x1="60.96" y1="116.84" x2="60.96" y2="114.3" width="0.1524" layer="91"/>
+<wire x1="58.42" y1="116.84" x2="60.96" y2="116.84" width="0.1524" layer="91"/>
+<junction x="60.96" y="116.84"/>
+</segment>
+<segment>
+<pinref part="LEFTSIDE" gate="G$1" pin="2"/>
+<pinref part="SUPPLY4" gate="G$1" pin="5V"/>
+<wire x1="0" y1="109.22" x2="7.62" y2="109.22" width="0.1524" layer="91"/>
+<wire x1="7.62" y1="109.22" x2="7.62" y2="114.3" width="0.1524" layer="91"/>
+</segment>
+</net>
