File: 2019NavBoard/2019NavBoard.sch (KiCad schematic (older format))
At the start: 21 parts, among them J1 Conn_Coaxial, U3 TM4C129E_Launchpad, U5 FGPMMOPA6H_GPS_MTK_MT3339_Chi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

Commit message: Started editing netlist
Parts:
- C2: footprint (none) -> MRDT_Devices:OKI_Horizontal
- Conn1, Conn2: footprint (none) -> MRDT_Connectors:Anderson_1_Horisontal
- Conn3: footprint (none) -> MRDT_Connectors:MOLEX_SL_08_Horizontal
- U3: footprint (none) -> MRDT_Shields:TM4C129E_Launchpad_X9
- renumbered U4 to ~1
Changed lines of the file:
@@
 EESchema Schematic File Version 4
+LIBS:2019NavBoard-cache
 EELAYER 26 0
 EELAYER END
@@
 F 0 "U3" H 8700 5100 60  0000 L CNN
 F 1 "TM4C129E_Launchpad" H 8550 7750 60  0000 L CNN
-F 2 "" H 8650 5200 60  0001 C CNN
+F 2 "MRDT_Shields:TM4C129E_Launchpad_X9" H 8650 5200 60  0001 C CNN
 F 3 "" H 8650 5200 60  0001 C CNN
 	3    8650 5200
@@
 $EndComp
 $Comp
-L MRDT_Shields:TM4C129E_Launchpad U4
+L MRDT_Shields:TM4C129E_Launchpad ~1
 U 4 1 5BC4AB1E
 P 9300 5200
-F 0 "U4" H 9400 5100 60  0000 C CNN
+F 0 "~1" H 9400 5100 60  0000 C CNN
 F 1 "~" H 8900 5000 60  0000 C CNN
 F 2 "" H 9300 5200 60  0001 C CNN
@@
 F 0 "Conn1" H 7306 2437 60  0000 C CNN
 F 1 "AndersonPP" H 7306 2331 60  0000 C CNN
-F 2 "" H 6950 1500 60  0001 C CNN
+F 2 "MRDT_Connectors:Anderson_1_Horisontal" H 6950 1500 60  0001 C CNN
 F 3 "" H 6950 1500 60  0001 C CNN
 	1    7100 2050
@@
 F 0 "Conn2" H 7306 2137 60  0000 C CNN
 F 1 "AndersonPP" H 7306 2031 60  0000 C CNN
-F 2 "" H 6950 1200 60  0001 C CNN
+F 2 "MRDT_Connectors:Anderson_1_Horisontal" H 6950 1200 60  0001 C CNN
 F 3 "" H 6950 1200 60  0001 C CNN
 	2    7100 1750
@@
 F 0 "C2" H 8200 1700 60  0001 C CNN
 F 1 "OKI" H 8350 2031 60  0000 C CNN
-F 2 "" H 7950 1650 60  0001 C CNN
+F 2 "MRDT_Devices:OKI_Horizontal" H 7950 1650 60  0001 C CNN
 F 3 "" H 7950 1650 60  0001 C CNN
 	1    8150 1750
@@
 F 0 "Conn3" H 6727 6008 60  0000 L CNN
 F 1 "Molex_SL_08" H 6727 5902 60  0000 L CNN
-F 2 "" H 6600 5850 60  0001 C CNN
+F 2 "MRDT_Connectors:MOLEX_SL_08_Horizontal" H 6600 5850 60  0001 C CNN
 F 3 "" H 6600 5850 60  0001 C CNN
 	1    6600 5550

Commit message: saved wor
Parts:
- Conn4: footprint (none) -> MRDT_Connectors:CR1220_Battery_Holder
- renumbered ~1 to U4
Changed lines of the file:
@@
 $EndComp
 $Comp
-L MRDT_Shields:TM4C129E_Launchpad ~1
+L MRDT_Shields:TM4C129E_Launchpad U4
 U 4 1 5BC4AB1E
 P 9300 5200
-F 0 "~1" H 9400 5100 60  0000 C CNN
+F 0 "U4" H 9400 5100 60  0000 C CNN
 F 1 "~" H 8900 5000 60  0000 C CNN
 F 2 "" H 9300 5200 60  0001 C CNN
@@
 Wire Wire Line
 	5000 2750 5300 2750
-Connection ~ 5000 2750
 Connection ~ 5300 2750
 Wire Wire Line
@@
 F 0 "Conn4" H 3662 5225 60  0000 L CNN
 F 1 "12mm_Coin_Cell_Battery_Holder" H 3550 4950 60  0001 C CNN
-F 2 "" H 3450 5000 60  0001 C CNN
+F 2 "MRDT_Connectors:CR1220_Battery_Holder" H 3450 5000 60  0001 C CNN
 F 3 "" H 3450 5000 60  0001 C CNN
 	1    3450 5000

Commit message: Assigned all parts
Parts:
- C1, C6: footprint (none) -> Capacitor_SMD:C_1206_3216Metric_Pad1.42x1.75mm_HandSolder
- C3, C4, C5: footprint (none) -> Capacitor_SMD:C_0805_2012Metric_Pad1.15x1.40mm_HandSolder
- D1, D2: footprint (none) -> LED_SMD:LED_0805_2012Metric_Pad1.15x1.40mm_HandSolder
- J1: footprint (none) -> Connector_Coaxial:SMA_Amphenol_132134-16_Vertical
- L1: value EXC3BP -> INDUCTOR; footprint (none) -> Inductor_SMD:L_0603_1608Metric_Pad1.05x0.95mm_HandSolder
- R1, R2: footprint (none) -> Resistor_SMD:R_0805_2012Metric_Pad1.15x1.40mm_HandSolder
- U1, U2, U4: value ~ -> TM4C129E_Launchpad; footprint (none) -> MRDT_Shields:TM4C129E_Launchpad_X9
Changed lines of the file:
@@
 P 8700 4000
 F 0 "U1" H 8750 5150 60  0000 L CNN
-F 1 "~" H 9001 4492 60  0000 L CNN
-F 2 "" H 8700 4000 60  0001 C CNN
+F 1 "TM4C129E_Launchpad" H 9001 4492 60  0000 L CNN
+F 2 "MRDT_Shields:TM4C129E_Launchpad_X9" H 8700 4000 60  0001 C CNN
 F 3 "" H 8700 4000 60  0001 C CNN
 	1    8700 4000
@@
 P 9300 4000
 F 0 "U2" H 9400 5150 60  0000 C CNN
-F 1 "~" H 9332 5171 60  0000 C CNN
-F 2 "" H 9300 4000 60  0001 C CNN
+F 1 "TM4C129E_Launchpad" H 9332 5171 60  0000 C CNN
+F 2 "MRDT_Shields:TM4C129E_Launchpad_X9" H 9300 4000 60  0001 C CNN
 F 3 "" H 9300 4000 60  0001 C CNN
 	2    9300 4000
@@
 P 9300 5200
 F 0 "U4" H 9400 5100 60  0000 C CNN
-F 1 "~" H 8900 5000 60  0000 C CNN
-F 2 "" H 9300 5200 60  0001 C CNN
+F 1 "TM4C129E_Launchpad" H 8900 5000 60  0000 C CNN
+F 2 "MRDT_Shields:TM4C129E_Launchpad_X9" H 9300 5200 60  0001 C CNN
 F 3 "" H 9300 5200 60  0001 C CNN
 	4    9300 5200
@@
 F 0 "C6" H 7915 1846 50  0000 L CNN
 F 1 "10uF" H 7915 1755 50  0000 L CNN
-F 2 "" H 7800 1800 50  0001 C CNN
+F 2 "Capacitor_SMD:C_1206_3216Metric_Pad1.42x1.75mm_HandSolder" H 7800 1800 50  0001 C CNN
 F 3 "~" H 7800 1800 50  0001 C CNN
 	1    7800 1800
@@
 F 0 "C1" H 8915 1896 50  0000 L CNN
 F 1 "10uF" H 8915 1805 50  0000 L CNN
-F 2 "" H 8800 1850 50  0001 C CNN
+F 2 "Capacitor_SMD:C_1206_3216Metric_Pad1.42x1.75mm_HandSolder" H 8800 1850 50  0001 C CNN
 F 3 "~" H 8800 1850 50  0001 C CNN
 	1    8800 1850
@@
 F 0 "J1" H 5099 2526 50  0000 L CNN
 F 1 "Conn_Coaxial" H 5099 2435 50  0000 L CNN
-F 2 "" H 5000 2550 50  0001 C CNN
+F 2 "Connector_Coaxial:SMA_Amphenol_132134-16_Vertical" H 5000 2550 50  0001 C CNN
 F 3 " ~" H 5000 2550 50  0001 C CNN
 	1    5000 2550
@@
 P 1850 1500
 F 0 "L1" H 1850 1715 50  0000 C CNN
-F 1 "EXC3BP" H 1850 1624 50  0000 C CNN
-F 2 "" H 1850 1500 50  0001 C CNN
+F 1 "INDUCTOR" H 1850 1624 50  0000 C CNN
+F 2 "Inductor_SMD:L_0603_1608Metric_Pad1.05x0.95mm_HandSolder" H 1850 1500 50  0001 C CNN
 F 3 "" H 1850 1500 50  0001 C CNN
 	1    1850 1500
@@
 F 0 "C4" H 2965 1746 50  0000 L CNN
 F 1 "0.01uF" H 2965 1655 50  0000 L CNN
-F 2 "" H 2850 1700 50  0001 C CNN
+F 2 "Capacitor_SMD:C_0805_2012Metric_Pad1.15x1.40mm_HandSolder" H 2850 1700 50  0001 C CNN
 F 3 "~" H 2850 1700 50  0001 C CNN
 	1    2850 1700
@@
 F 0 "C3" H 2215 1746 50  0000 L CNN
 F 1 "1uF" H 2215 1655 50  0000 L CNN
-F 2 "" H 2100 1700 50  0001 C CNN
+F 2 "Capacitor_SMD:C_0805_2012Metric_Pad1.15x1.40mm_HandSolder" H 2100 1700 50  0001 C CNN
 F 3 "~" H 2100 1700 50  0001 C CNN
 	1    2100 1700
@@
 F 0 "R1" V 2545 2050 50  0000 C CNN
 F 1 "1k" V 2636 2050 50  0000 C CNN
-F 2 "" V 2790 2040 50  0001 C CNN
+F 2 "Resistor_SMD:R_0805_2012Metric_Pad1.15x1.40mm_HandSolder" V 2790 2040 50  0001 C CNN
 F 3 "~" H 2750 2050 50  0001 C CNN
 	1    2750 2050
@@
 F 0 "D1" H 2400 2285 50  0000 C CNN
 F 1 "FIX" H 2400 2194 50  0000 C CNN
-F 2 "" V 2400 2050 50  0001 C CNN
+F 2 "LED_SMD:LED_0805_2012Metric_Pad1.15x1.40mm_HandSolder" V 2400 2050 50  0001 C CNN
 F 3 "~" V 2400 2050 50  0001 C CNN
 	1    2400 2050
@@
 F 0 "C5" H 3165 4846 50  0000 L CNN
 F 1 "1uF" H 3165 4755 50  0000 L CNN
-F 2 "" H 3050 4800 50  0001 C CNN
+F 2 "Capacitor_SMD:C_0805_2012Metric_Pad1.15x1.40mm_HandSolder" H 3050 4800 50  0001 C CNN
 F 3 "~" H 3050 4800 50  0001 C CNN
 	1    3050 4800
@@
 F 0 "R2" H 6518 3196 50  0000 L CNN
 F 1 "1K" H 6518 3105 50  0000 L CNN
-F 2 "" V 6490 3140 50  0001 C CNN
+F 2 "Resistor_SMD:R_0805_2012Metric_Pad1.15x1.40mm_HandSolder" V 6490 3140 50  0001 C CNN
 F 3 "~" H 6450 3150 50  0001 C CNN
 	1    6450 3150
@@
 F 0 "D2" V 6496 3482 50  0000 R CNN
 F 1 "PWR" V 6405 3482 50  0000 R CNN
-F 2 "" V 6450 3550 50  0001 C CNN
+F 2 "LED_SMD:LED_0805_2012Metric_Pad1.15x1.40mm_HandSolder" V 6450 3550 50  0001 C CNN
 F 3 "~" V 6450 3550 50  0001 C CNN
 	1    6450 3550

Commit message: Finalized high lvl schematic
Parts:
- removed U5: FGPMMOPA6H_GPS_MTK_MT3339_Chipset, symbol NavBoard:FGPMMOPA6H_GPS_MTK_MT3339_Chipset
- added U5: FGPMMOPA6H, MRDT_Sensors:FGPMMOPA6H, symbol MRDT_Sensors:FGPMMOPA6H
- Conn1: footprint MRDT_Connectors:Anderson_1_Horisontal -> MRDT_Connectors:Anderson_2_Horisontal_Side_by_Side
- Conn1: renamed from Conn2; footprint MRDT_Connectors:Anderson_1_Horisontal -> MRDT_Connectors:Anderson_2_Horisontal_Side_by_Side
- U1: value TM4C129E_Launchpad -> ~
- U1: renamed from U2; value TM4C129E_Launchpad -> ~
- U1: renamed from U4; value TM4C129E_Launchpad -> ~
- renumbered U3 to U1
Other:
- note added: "Connector to off board ISM and Board Power LED"
- note added: "GPS and Battery Backup\n"
- note added: "Power Distribution"
- note added: "TIVA\n"

Commit message: Fixed Errors and added a LIDAR
Some of the gobal labels had to be fixed and I added a LIDAR to the schematic. Also added some .txt files for pdr.
Parts:
- added 1K1: R3, Resistor_SMD:R_0603_1608Metric_Pad1.05x0.95mm_HandSolder, symbol Device:R_US
- added LIDAR1: Molex_SL_03, MRDT_Connectors:MOLEX_SL_03_Horizontal, symbol MRDT_Connectors:Molex_SL_03
- R1: value 1k -> 1K
- renumbered U1 to U1C1
Connections:
- net labels added: LIDAR_MONITOR, LIDAR_TRIGGER
- net labels removed: GPS_RX5, GPS_TX5, INT1, INT2, SCL, SDA
- wire segments 74 -> 83
Other:
- note added: "GPS, Battery Backup, and LiDAR\n"
- note removed: "GPS and Battery Backup\n"

Commit message: Added LIDAR 4SL
Parts:
- removed 1K1: R3, Resistor_SMD:R_0603_1608Metric_Pad1.05x0.95mm_HandSolder, symbol Device:R_US
- removed LIDAR1: Molex_SL_03, MRDT_Connectors:MOLEX_SL_03_Horizontal, symbol MRDT_Connectors:Molex_SL_03
- added C7: 680uF, Capacitor_SMD:C_1206_3216Metric_Pad1.42x1.75mm_HandSolder, symbol Device:C
- added LIDAR1: Molex_SL_04, MRDT_Connectors:MOLEX_SL_04_Horizontal, symbol MRDT_Connectors:Molex_SL_04
- added R3, R4: 4.7K, Resistor_SMD:R_0805_2012Metric_Pad1.15x1.40mm_HandSolder, symbol Device:R_US
Connections:
- wire segments 83 -> 94
Other:
- note added: "GPS, and LiDAR\n"
- note added: "TIVA and Battery Backup\n\n"
- note removed: "GPS, Battery Backup, and LiDAR\n"
- note removed: "TIVA\n"
Changed lines of the file:
@@
 L MRDT_Connectors:12mm_Coin_Cell_Battery_Holder Conn4
 U 1 1 5BC5B0C6
-P 4450 3750
-F 0 "Conn4" H 4662 3975 60  0000 L CNN
-F 1 "12mm_Coin_Cell_Battery_Holder" H 4550 3700 60  0001 C CNN
-F 2 "MRDT_Connectors:CR1220_Battery_Holder" H 4450 3750 60  0001 C CNN
-F 3 "" H 4450 3750 60  0001 C CNN
-	1    4450 3750
-	1    0    0    -1
-$EndComp
-Wire Wire Line
-	4450 3750 4250 3750
-Wire Wire Line
-	4050 3300 4350 3300
-Wire Wire Line
-	4250 3750 4250 3850
-Connection ~ 4250 3750
-Wire Wire Line
-	4250 3750 4050 3750
+P 10600 3950
+F 0 "Conn4" H 10812 4175 60  0000 L CNN
+F 1 "12mm_Coin_Cell_Battery_Holder" H 10700 3900 60  0001 C CNN
+F 2 "MRDT_Connectors:CR1220_Battery_Holder" H 10600 3950 60  0001 C CNN
+F 3 "" H 10600 3950 60  0001 C CNN
+	1    10600 3950
+	1    0    0    -1
+$EndComp
+Wire Wire Line
+	10600 3950 10400 3950
+Wire Wire Line
+	10200 3500 10500 3500
+Wire Wire Line
+	10400 3950 10400 4050
+Connection ~ 10400 3950
+Wire Wire Line
+	10400 3950 10200 3950
 $Comp
 L power:GND #PWR0106
 U 1 1 5BC5C835
-P 4250 3850
-F 0 "#PWR0106" H 4250 3600 50  0001 C CNN
-F 1 "GND" H 4255 3677 50  0000 C CNN
-F 2 "" H 4250 3850 50  0001 C CNN
-F 3 "" H 4250 3850 50  0001 C CNN
-	1    4250 3850
+P 10400 4050
+F 0 "#PWR0106" H 10400 3800 50  0001 C CNN
+F 1 "GND" H 10405 3877 50  0000 C CNN
+F 2 "" H 10400 4050 50  0001 C CNN
+F 3 "" H 10400 4050 50  0001 C CNN
+	1    10400 4050
 	1    0    0    -1
 $EndComp
@@
 L Device:CP1 C5
 U 1 1 5BC5C880
-P 4050 3550
-F 0 "C5" H 4165 3596 50  0000 L CNN
-F 1 "1uF" H 4165 3505 50  0000 L CNN
-F 2 "Capacitor_SMD:C_0805_2012Metric_Pad1.15x1.40mm_HandSolder" H 4050 3550 50  0001 C CNN
-F 3 "~" H 4050 3550 50  0001 C CNN
-	1    4050 3550
-	1    0    0    -1
-$EndComp
-Wire Wire Line
-	4050 3750 4050 3700
-Wire Wire Line
-	4050 3300 4050 3400
-Wire Wire Line
-	4350 3300 4350 3200
-Wire Wire Line
-	4350 3200 4150 3200
-Connection ~ 4350 3300
-Wire Wire Line
-	4350 3300 4450 3300
-Text GLabel 4150 3200 0    50   Input ~ 0
+P 10200 3750
+F 0 "C5" H 10315 3796 50  0000 L CNN
+F 1 "1uF" H 10315 3705 50  0000 L CNN
+F 2 "Capacitor_SMD:C_0805_2012Metric_Pad1.15x1.40mm_HandSolder" H 10200 3750 50  0001 C CNN
+F 3 "~" H 10200 3750 50  0001 C CNN
+	1    10200 3750
+	1    0    0    -1
+$EndComp
+Wire Wire Line
+	10200 3950 10200 3900
+Wire Wire Line
+	10200 3500 10200 3600
+Wire Wire Line
+	10500 3500 10500 3400
+Wire Wire Line
+	10500 3400 10300 3400
+Connection ~ 10500 3500
+Wire Wire Line
+	10500 3500 10600 3500
+Text GLabel 10300 3400 0    50   Input ~ 0
 VBACKUP
 Wire Wire Line
@@
 	7450 4350 7450 450
 Text Notes 8200 800  0    50   ~ 10
-TIVA\n
+TIVA and Battery Backup\n\n
 Text Notes 4550 900  0    50   ~ 10
-GPS, Battery Backup, and LiDAR\n
+GPS, and LiDAR\n
 Wire Notes Line
 	450  4350 11200 4350
 Text Notes 1050 2600 0    50   ~ 10
 Connector to off board ISM and Board Power LED
-$Comp
-L MRDT_Connectors:Molex_SL_03 LIDAR1
-U 1 1 5BCB1845
-P 6800 3400
-F 0 "LIDAR1" V 7050 3850 60  0000 R CNN
-F 1 "Molex_SL_03" V 6950 3850 60  0000 R CNN
-F 2 "MRDT_Connectors:MOLEX_SL_03_Horizontal" H 6800 3400 60  0001 C CNN
-F 3 "" H 6800 3400 60  0001 C CNN
-	1    6800 3400
-	1    0    0    -1
-$EndComp
-$Comp
-L power:+5V #PWR0114
-U 1 1 5BCB67EE
-P 6600 2850
-F 0 "#PWR0114" H 6600 2700 50  0001 C CNN
-F 1 "+5V" H 6600 3050 50  0000 C CNN
-F 2 "" H 6600 2850 50  0001 C CNN
-F 3 "" H 6600 2850 50  0001 C CNN
-	1    6600 2850
-	1    0    0    -1
-$EndComp
-$Comp
-L power:GND #PWR0115
-U 1 1 5BCB9D15
-P 6600 3700
-F 0 "#PWR0115" H 6600 3450 50  0001 C CNN
-F 1 "GND" H 6600 3500 50  0000 C CNN
-F 2 "" H 6600 3700 50  0001 C CNN
-F 3 "" H 6600 3700 50  0001 C CNN
-	1    6600 3700
-	1    0    0    -1
-$EndComp
-$Comp
-L Device:R_US 1K1
-U 1 1 5BCB9E2D
-P 6300 3500
-F 0 "1K1" V 6400 3450 50  0000 L CNN
-F 1 "R3" V 6200 3450 50  0000 L CNN
-F 2 "Resistor_SMD:R_0603_1608Metric_Pad1.05x0.95mm_HandSolder" V 6340 3490 50  0001 C CNN
-F 3 "~" H 6300 3500 50  0001 C CNN
-	1    6300 3500
-	-1   0    0    1
-$EndComp
-Wire Wire Line
-	6600 3250 6300 3250
-Text GLabel 6250 3250 0    50   Input ~ 0
+Text GLabel 4550 3150 0    50   Input ~ 0
 LIDAR_MONITOR
-Text GLabel 6250 3800 0    50   Input ~ 0
+Text GLabel 4450 3300 0    50   Input ~ 0
 LIDAR_TRIGGER
-Wire Wire Line
-	6300 3250 6300 3350
-Wire Wire Line
-	6300 3650 6300 3800
 Text GLabel 8150 1750 0    50   Input ~ 0
 LIDAR_MONITOR
@@
 Wire Wire Line
 	8000 1950 8250 1950
-Wire Wire Line
-	6600 3350 6600 3700
-Wire Wire Line
-	6600 2850 6600 3150
 Wire Notes Line
 	3450 450  3450 4350
@@
 Wire Wire Line
 	8250 1850 8150 1850
-Wire Wire Line
-	6250 3800 6300 3800
-Wire Wire Line
-	6250 3250 6300 3250
-Connection ~ 6300 3250
+$Comp
+L MRDT_Connectors:Molex_SL_04 LIDAR1
+U 1 1 5BCF7588
+P 6050 3450
+F 0 "LIDAR1" H 6177 3708 60  0000 L CNN
+F 1 "Molex_SL_04" H 6177 3602 60  0000 L CNN
+F 2 "MRDT_Connectors:MOLEX_SL_04_Horizontal" H 6050 3450 60  0001 C CNN
+F 3 "" H 6050 3450 60  0001 C CNN
+	1    6050 3450
+	1    0    0    -1
+$EndComp
+Wire Wire Line
+	5850 3400 5650 3400
+Wire Wire Line
+	5850 3100 5650 3100
+Wire Wire Line
+	5650 3100 5650 2950
+Wire Wire Line
+	5650 2950 6850 2950
+Wire Wire Line
+	6850 2950 6850 3100
+$Comp
+L Device:C C7
+U 1 1 5BD0BD22
+P 6850 3250
+F 0 "C7" H 6965 3296 50  0000 L CNN
+F 1 "680uF" H 6965 3205 50  0000 L CNN
+F 2 "Capacitor_SMD:C_1206_3216Metric_Pad1.42x1.75mm_HandSolder" H 6888 3100 50  0001 C CNN
+F 3 "~" H 6850 3250 50  0001 C CNN
+	1    6850 3250
+	1    0    0    -1
+$EndComp
+Wire Wire Line
+	6850 3400 6850 3550
+Wire Wire Line
+	6850 3550 5650 3550
+Wire Wire Line
+	5650 3550 5650 3400
+Wire Wire Line
+	5650 3100 5450 3100
+Connection ~ 5650 3100
+$Comp
+L power:GND #PWR0114
+U 1 1 5BD16850
+P 5450 3100
+F 0 "#PWR0114" H 5450 2850 50  0001 C CNN
+F 1 "GND" H 5455 2927 50  0000 C CNN
+F 2 "" H 5450 3100 50  0001 C CNN
+F 3 "" H 5450 3100 50  0001 C CNN
+	1    5450 3100
+	-1   0    0    1
+$EndComp
+Wire Wire Line
+	5650 3400 5400 3400
+Connection ~ 5650 3400
+$Comp
+L power:+5V #PWR0115
+U 1 1 5BD195C6
+P 5400 3400
+F 0 "#PWR0115" H 5400 3250 50  0001 C CNN
+F 1 "+5V" H 5415 3573 50  0000 C CNN
+F 2 "" H 5400 3400 50  0001 C CNN
+F 3 "" H 5400 3400 50  0001 C CNN
+	1    5400 3400
+	-1   0    0    1
+$EndComp
+Wire Wire Line
+	5850 3200 5400 3200
+Wire Wire Line
+	5400 3200 5400 3150
+$Comp
+L Device:R_US R3
+U 1 1 5BD211F8
+P 5250 3150
+F 0 "R3" V 5045 3150 50  0000 C CNN
+F 1 "4.7K" V 5136 3150 50  0000 C CNN
+F 2 "Resistor_SMD:R_0805_2012Metric_Pad1.15x1.40mm_HandSolder" V 5290 3140 50  0001 C CNN
+F 3 "~" H 5250 3150 50  0001 C CNN
+	1    5250 3150
+	0    1    1    0
+$EndComp
+$Comp
+L Device:R_US R4
+U 1 1 5BD2760A
+P 4700 3300
+F 0 "R4" V 4905 3300 50  0000 C CNN
+F 1 "4.7K" V 4814 3300 50  0000 C CNN
+F 2 "Resistor_SMD:R_0805_2012Metric_Pad1.15x1.40mm_HandSolder" V 4740 3290 50  0001 C CNN
+F 3 "~" H 4700 3300 50  0001 C CNN
+	1    4700 3300
+	0    -1   -1   0
+$EndComp
+Wire Wire Line
+	4550 3300 4450 3300
+Wire Wire Line
+	4550 3150 4550 3300
+Connection ~ 4550 3300
+Wire Wire Line
+	5850 3300 4850 3300
+Wire Wire Line
+	4550 3150 5100 3150
+Wire Wire Line
+	4450 3300 4450 3400
+Wire Wire Line
+	4450 3400 5400 3400
+Connection ~ 5400 3400
 $EndSCHEMATC

Commit message: Final PDR edits
Other:
- note added: "Connector to off board IMU and Board Power LED"
- note removed: "Connector to off board ISM and Board Power LED"
Changed lines of the file:
@@
 	450  4350 11200 4350
 Text Notes 1050 2600 0    50   ~ 10
-Connector to off board ISM and Board Power LED
+Connector to off board IMU and Board Power LED
 Text GLabel 4550 3150 0    50   Input ~ 0
 LIDAR_MONITOR

Commit message: Changed indicators
Connections:
- wire segments 94 -> 96
Changed lines of the file:
@@
 Wire Wire Line
 	8250 2450 7800 2450
-Text GLabel 8050 3350 0    50   Input ~ 0
+Text GLabel 8050 2750 0    50   Input ~ 0
 INT2AG
-Text GLabel 8050 3450 0    50   Input ~ 0
+Text GLabel 8050 2850 0    50   Input ~ 0
 INT1AG
 Text GLabel 8050 3550 0    50   Input ~ 0
@@
 Power Distribution
 Wire Notes Line
-	7450 4350 7450 450
+	7400 4350 7400 450
 Text Notes 8200 800  0    50   ~ 10
 TIVA and Battery Backup\n\n
@@
 Text GLabel 4450 3300 0    50   Input ~ 0
 LIDAR_TRIGGER
-Text GLabel 8150 1750 0    50   Input ~ 0
+Text GLabel 8050 3350 0    50   Input ~ 0
 LIDAR_MONITOR
-Text GLabel 8150 1850 0    50   Input ~ 0
+Text GLabel 8050 3450 0    50   Input ~ 0
 LIDAR_TRIGGER
 Wire Wire Line
@@
 	4450 3400 5400 3400
 Connection ~ 5400 3400
+Wire Wire Line
+	8050 2750 8200 2750
+Wire Wire Line
+	8050 2850 8200 2850
 $EndSCHEMATC
