File: 2019NavBoard/2019NavBoard.sch (KiCad schematic (older format))
At the start: 22 parts, among them J1 Conn_Coaxial, U1C1 TM4C129E_Launchpad, U5 FGPMMOPA6H

Commit message: PDR Ready
Parts:
- Conn2: renamed from LIDAR1; value Molex_SL_04 -> LiDAR
Connections:
- net labels added: LIDAR_SCL, LIDAR_SDA
- net labels removed: LIDAR_MONITOR, LIDAR_TRIGGER
- wire segments 96 -> 95
Other:
- note added: "Blue"
- note added: "Green"
Changed lines of the file:
@@
 Text Notes 1050 2600 0    50   ~ 10
 Connector to off board IMU and Board Power LED
-Text GLabel 4550 3150 0    50   Input ~ 0
-LIDAR_MONITOR
-Text GLabel 4450 3300 0    50   Input ~ 0
-LIDAR_TRIGGER
-Text GLabel 8050 3350 0    50   Input ~ 0
-LIDAR_MONITOR
-Text GLabel 8050 3450 0    50   Input ~ 0
-LIDAR_TRIGGER
+Text GLabel 5000 3600 0    50   Input ~ 0
+LIDAR_SDA
+Text GLabel 5000 3500 0    50   Input ~ 0
+LIDAR_SCL
 Wire Wire Line
 	8000 1950 8250 1950
@@
 	8250 1850 8150 1850
 $Comp
-L MRDT_Connectors:Molex_SL_04 LIDAR1
+L MRDT_Connectors:Molex_SL_04 Conn2
 U 1 1 5BCF7588
-P 6050 3450
-F 0 "LIDAR1" H 6177 3708 60  0000 L CNN
-F 1 "Molex_SL_04" H 6177 3602 60  0000 L CNN
-F 2 "MRDT_Connectors:MOLEX_SL_04_Horizontal" H 6050 3450 60  0001 C CNN
-F 3 "" H 6050 3450 60  0001 C CNN
-	1    6050 3450
+P 5850 3750
+F 0 "Conn2" H 5977 4008 60  0000 L CNN
+F 1 "LiDAR" H 5977 3902 60  0000 L CNN
+F 2 "MRDT_Connectors:MOLEX_SL_04_Horizontal" H 5850 3750 60  0001 C CNN
+F 3 "" H 5850 3750 60  0001 C CNN
+	1    5850 3750
 	1    0    0    -1
 $EndComp
 Wire Wire Line
-	5850 3400 5650 3400
+	5650 3700 5450 3700
 Wire Wire Line
-	5850 3100 5650 3100
+	5450 3700 5450 3850
 Wire Wire Line
-	5650 3100 5650 2950
+	5450 3850 6650 3850
 Wire Wire Line
-	5650 2950 6850 2950
-Wire Wire Line
-	6850 2950 6850 3100
+	6650 3850 6650 3700
 $Comp
 L Device:C C7
 U 1 1 5BD0BD22
-P 6850 3250
-F 0 "C7" H 6965 3296 50  0000 L CNN
-F 1 "680uF" H 6965 3205 50  0000 L CNN
-F 2 "Capacitor_SMD:C_1206_3216Metric_Pad1.42x1.75mm_HandSolder" H 6888 3100 50  0001 C CNN
-F 3 "~" H 6850 3250 50  0001 C CNN
-	1    6850 3250
-	1    0    0    -1
+P 6650 3550
+F 0 "C7" H 6765 3596 50  0000 L CNN
+F 1 "680uF" H 6765 3505 50  0000 L CNN
+F 2 "Capacitor_SMD:C_1206_3216Metric_Pad1.42x1.75mm_HandSolder" H 6688 3400 50  0001 C CNN
+F 3 "~" H 6650 3550 50  0001 C CNN
+	1    6650 3550
+	1    0    0    1
 $EndComp
 Wire Wire Line
-	6850 3400 6850 3550
-Wire Wire Line
-	6850 3550 5650 3550
-Wire Wire Line
-	5650 3550 5650 3400
-Wire Wire Line
-	5650 3100 5450 3100
-Connection ~ 5650 3100
+	5450 3700 5250 3700
+Connection ~ 5450 3700
 $Comp
 L power:GND #PWR0114
 U 1 1 5BD16850
-P 5450 3100
-F 0 "#PWR0114" H 5450 2850 50  0001 C CNN
-F 1 "GND" H 5455 2927 50  0000 C CNN
-F 2 "" H 5450 3100 50  0001 C CNN
-F 3 "" H 5450 3100 50  0001 C CNN
-	1    5450 3100
-	-1   0    0    1
+P 5250 3700
+F 0 "#PWR0114" H 5250 3450 50  0001 C CNN
+F 1 "GND" H 5255 3527 50  0000 C CNN
+F 2 "" H 5250 3700 50  0001 C CNN
+F 3 "" H 5250 3700 50  0001 C CNN
+	1    5250 3700
+	-1   0    0    -1
 $EndComp
-Wire Wire Line
-	5650 3400 5400 3400
-Connection ~ 5650 3400
 $Comp
 L power:+5V #PWR0115
 U 1 1 5BD195C6
-P 5400 3400
-F 0 "#PWR0115" H 5400 3250 50  0001 C CNN
-F 1 "+5V" H 5415 3573 50  0000 C CNN
-F 2 "" H 5400 3400 50  0001 C CNN
-F 3 "" H 5400 3400 50  0001 C CNN
-	1    5400 3400
-	-1   0    0    1
+P 6050 3200
+F 0 "#PWR0115" H 6050 3050 50  0001 C CNN
+F 1 "+5V" H 6065 3373 50  0000 C CNN
+F 2 "" H 6050 3200 50  0001 C CNN
+F 3 "" H 6050 3200 50  0001 C CNN
+	1    6050 3200
+	-1   0    0    -1
 $EndComp
-Wire Wire Line
-	5850 3200 5400 3200
-Wire Wire Line
-	5400 3200 5400 3150
 $Comp
 L Device:R_US R3
 U 1 1 5BD211F8
-P 5250 3150
-F 0 "R3" V 5045 3150 50  0000 C CNN
-F 1 "4.7K" V 5136 3150 50  0000 C CNN
-F 2 "Resistor_SMD:R_0805_2012Metric_Pad1.15x1.40mm_HandSolder" V 5290 3140 50  0001 C CNN
-F 3 "~" H 5250 3150 50  0001 C CNN
-	1    5250 3150
-	0    1    1    0
+P 5050 3400
+F 0 "R3" V 4845 3400 50  0000 C CNN
+F 1 "4.7K" V 4936 3400 50  0000 C CNN
+F 2 "Resistor_SMD:R_0805_2012Metric_Pad1.15x1.40mm_HandSolder" V 5090 3390 50  0001 C CNN
+F 3 "~" H 5050 3400 50  0001 C CNN
+	1    5050 3400
+	-1   0    0    -1
 $EndComp
 $Comp
 L Device:R_US R4
 U 1 1 5BD2760A
-P 4700 3300
-F 0 "R4" V 4905 3300 50  0000 C CNN
-F 1 "4.7K" V 4814 3300 50  0000 C CNN
-F 2 "Resistor_SMD:R_0805_2012Metric_Pad1.15x1.40mm_HandSolder" V 4740 3290 50  0001 C CNN
-F 3 "~" H 4700 3300 50  0001 C CNN
-	1    4700 3300
-	0    -1   -1   0
+P 5350 3350
+F 0 "R4" V 5555 3350 50  0000 C CNN
+F 1 "4.7K" V 5464 3350 50  0000 C CNN
+F 2 "Resistor_SMD:R_0805_2012Metric_Pad1.15x1.40mm_HandSolder" V 5390 3340 50  0001 C CNN
+F 3 "~" H 5350 3350 50  0001 C CNN
+	1    5350 3350
+	1    0    0    1
 $EndComp
-Wire Wire Line
-	4550 3300 4450 3300
-Wire Wire Line
-	4550 3150 4550 3300
-Connection ~ 4550 3300
-Wire Wire Line
-	5850 3300 4850 3300
-Wire Wire Line
-	4550 3150 5100 3150
-Wire Wire Line
-	4450 3300 4450 3400
-Wire Wire Line
-	4450 3400 5400 3400
-Connection ~ 5400 3400
 Wire Wire Line
 	8050 2750 8200 2750
 Wire Wire Line
 	8050 2850 8200 2850
+Text GLabel 8050 3350 0    50   Output ~ 0
+LIDAR_SDA
+Text GLabel 8050 3450 0    50   Output ~ 0
+LIDAR_SCL
+Text Notes 4300 3650 0    50   ~ 0
+Blue
+Text Notes 4300 3550 0    50   ~ 0
+Green
+Wire Wire Line
+	5650 3600 5050 3600
+Wire Wire Line
+	5050 3600 5050 3550
+Wire Wire Line
+	5650 3500 5350 3500
+Wire Wire Line
+	5050 3250 5050 3200
+Wire Wire Line
+	5050 3200 5350 3200
+Connection ~ 5350 3200
+Wire Wire Line
+	5350 3200 5650 3200
+Connection ~ 6050 3200
+Wire Wire Line
+	6050 3200 6650 3200
+Wire Wire Line
+	6650 3400 6650 3200
+Wire Wire Line
+	5000 3600 5050 3600
+Connection ~ 5050 3600
+Wire Wire Line
+	5350 3500 5000 3500
+Connection ~ 5350 3500
+Wire Wire Line
+	5650 3400 5650 3200
+Connection ~ 5650 3200
+Wire Wire Line
+	5650 3200 6050 3200
 $EndSCHEMATC

Commit message: Finalized Rev1
Parts:
- removed Conn4: 12mm_Coin_Cell_Battery_Holder, MRDT_Connectors:CR1220_Battery_Holder, symbol MRDT_Connectors:12mm_Coin_Cell_Battery_Holder
- added U2: 12mm_Coin_Battery_Cell_Holder, MRDT_Connectors:CR1220_Battery_Holder, symbol 2019_NavB:12mm_Coin_Battery_Cell_Holder
Changed lines of the file:
@@
 EESchema Schematic File Version 4
-LIBS:2019NavBoard-cache
 EELAYER 26 0
 EELAYER END
@@
 F 3 "" H 4200 2400 50  0001 C CNN
 	1    4200 2400
-	1    0    0    -1
-$EndComp
-$Comp
-L MRDT_Connectors:12mm_Coin_Cell_Battery_Holder Conn4
-U 1 1 5BC5B0C6
-P 10600 3950
-F 0 "Conn4" H 10812 4175 60  0000 L CNN
-F 1 "12mm_Coin_Cell_Battery_Holder" H 10700 3900 60  0001 C CNN
-F 2 "MRDT_Connectors:CR1220_Battery_Holder" H 10600 3950 60  0001 C CNN
-F 3 "" H 10600 3950 60  0001 C CNN
-	1    10600 3950
 	1    0    0    -1
 $EndComp
@@
 Wire Wire Line
 	5650 3200 6050 3200
+$Comp
+L 2019_NavB:12mm_Coin_Battery_Cell_Holder U2
+U 1 1 5BE8F78F
+P 10600 4050
+F 0 "U2" H 10812 4421 50  0000 L CNN
+F 1 "12mm_Coin_Battery_Cell_Holder" H 10812 4330 50  0000 L CNN
+F 2 "MRDT_Connectors:CR1220_Battery_Holder" H 10600 4050 50  0001 C CNN
+F 3 "" H 10600 4050 50  0001 C CNN
+	1    10600 4050
+	1    0    0    -1
+$EndComp
 $EndSCHEMATC

Commit message: After meeting
Connections:
- net labels removed: 1PPS
- wire segments 95 -> 92
Changed lines of the file:
@@
 EESchema Schematic File Version 4
+LIBS:2019NavBoard-cache
 EELAYER 26 0
 EELAYER END
@@
 	7000 1450 7000 2150
 Wire Wire Line
-	6700 2450 7000 2450
-Connection ~ 7000 2450
-Wire Wire Line
-	7000 2450 7000 2550
-Wire Wire Line
 	7000 2550 6700 2550
 Wire Wire Line
@@
 	6400 2150 7000 2150
 Connection ~ 7000 2150
-Wire Wire Line
-	7000 2150 7000 2450
-Wire Wire Line
-	6400 2050 6500 2050
-Text GLabel 6500 2050 2    50   Input ~ 0
-1PPS
 Wire Wire Line
 	5500 2250 5350 2250
@@
 $EndComp
 Wire Wire Line
-	10600 3950 10400 3950
-Wire Wire Line
-	10200 3500 10500 3500
-Wire Wire Line
-	10400 3950 10400 4050
-Connection ~ 10400 3950
-Wire Wire Line
-	10400 3950 10200 3950
+	4200 4000 4000 4000
+Wire Wire Line
+	3800 3550 4100 3550
+Wire Wire Line
+	4000 4000 4000 4100
+Connection ~ 4000 4000
+Wire Wire Line
+	4000 4000 3800 4000
 $Comp
 L power:GND #PWR0106
 U 1 1 5BC5C835
-P 10400 4050
-F 0 "#PWR0106" H 10400 3800 50  0001 C CNN
-F 1 "GND" H 10405 3877 50  0000 C CNN
-F 2 "" H 10400 4050 50  0001 C CNN
-F 3 "" H 10400 4050 50  0001 C CNN
-	1    10400 4050
+P 4000 4100
+F 0 "#PWR0106" H 4000 3850 50  0001 C CNN
+F 1 "GND" H 4005 3927 50  0000 C CNN
+F 2 "" H 4000 4100 50  0001 C CNN
+F 3 "" H 4000 4100 50  0001 C CNN
+	1    4000 4100
 	1    0    0    -1
 $EndComp
@@
 L Device:CP1 C5
 U 1 1 5BC5C880
-P 10200 3750
-F 0 "C5" H 10315 3796 50  0000 L CNN
-F 1 "1uF" H 10315 3705 50  0000 L CNN
-F 2 "Capacitor_SMD:C_0805_2012Metric_Pad1.15x1.40mm_HandSolder" H 10200 3750 50  0001 C CNN
-F 3 "~" H 10200 3750 50  0001 C CNN
-	1    10200 3750
-	1    0    0    -1
-$EndComp
-Wire Wire Line
-	10200 3950 10200 3900
-Wire Wire Line
-	10200 3500 10200 3600
-Wire Wire Line
-	10500 3500 10500 3400
-Wire Wire Line
-	10500 3400 10300 3400
-Connection ~ 10500 3500
-Wire Wire Line
-	10500 3500 10600 3500
-Text GLabel 10300 3400 0    50   Input ~ 0
+P 3800 3800
+F 0 "C5" H 3915 3846 50  0000 L CNN
+F 1 "1uF" H 3915 3755 50  0000 L CNN
+F 2 "Capacitor_SMD:C_0805_2012Metric_Pad1.15x1.40mm_HandSolder" H 3800 3800 50  0001 C CNN
+F 3 "~" H 3800 3800 50  0001 C CNN
+	1    3800 3800
+	1    0    0    -1
+$EndComp
+Wire Wire Line
+	3800 4000 3800 3950
+Wire Wire Line
+	3800 3550 3800 3650
+Wire Wire Line
+	4100 3550 4100 3450
+Wire Wire Line
+	4100 3450 3900 3450
+Connection ~ 4100 3550
+Wire Wire Line
+	4100 3550 4200 3550
+Text GLabel 3900 3450 0    50   Input ~ 0
 VBACKUP
 Wire Wire Line
@@
 	0    -1   -1   0
 $EndComp
-Text GLabel 1200 3250 0    50   Input ~ 0
+Text GLabel 1200 3250 0    50   Output ~ 0
 INT2AG
-Text GLabel 1200 3350 0    50   Input ~ 0
+Text GLabel 1200 3350 0    50   Output ~ 0
 INT1AG
-Text GLabel 1200 3450 0    50   Input ~ 0
+Text GLabel 1200 3450 0    50   Output ~ 0
 INTM
-Text GLabel 1200 3550 0    50   Input ~ 0
+Text GLabel 1200 3550 0    50   Output ~ 0
 DRDYM
 Text GLabel 1200 3650 0    50   Input ~ 0
@@
 Wire Wire Line
 	8200 3650 8050 3650
-Text GLabel 8000 1950 0    50   Input ~ 0
+Text GLabel 8150 1850 0    50   Input ~ 0
 RX(7)
-Text GLabel 7900 2250 0    50   Input ~ 0
+Text GLabel 8150 1750 0    50   Input ~ 0
 TX(7)
 Wire Wire Line
@@
 	1    0    0    -1
 $EndComp
-Connection ~ 6700 2450
 Wire Notes Line
 	3400 2350 450  2350
@@
 Text Notes 1050 2600 0    50   ~ 10
 Connector to off board IMU and Board Power LED
-Text GLabel 5000 3600 0    50   Input ~ 0
+Text GLabel 1500 5450 0    50   Input ~ 0
 LIDAR_SDA
-Text GLabel 5000 3500 0    50   Input ~ 0
+Text GLabel 1500 5350 0    50   Input ~ 0
 LIDAR_SCL
 Wire Wire Line
@@
 L MRDT_Connectors:Molex_SL_04 Conn2
 U 1 1 5BCF7588
-P 5850 3750
-F 0 "Conn2" H 5977 4008 60  0000 L CNN
-F 1 "LiDAR" H 5977 3902 60  0000 L CNN
-F 2 "MRDT_Connectors:MOLEX_SL_04_Horizontal" H 5850 3750 60  0001 C CNN
-F 3 "" H 5850 3750 60  0001 C CNN
-	1    5850 3750
-	1    0    0    -1
-$EndComp
-Wire Wire Line
-	5650 3700 5450 3700
-Wire Wire Line
-	5450 3700 5450 3850
-Wire Wire Line
-	5450 3850 6650 3850
-Wire Wire Line
-	6650 3850 6650 3700
+P 2350 5600
+F 0 "Conn2" H 2477 5858 60  0000 L CNN
+F 1 "LiDAR" H 2477 5752 60  0000 L CNN
+F 2 "MRDT_Connectors:MOLEX_SL_04_Horizontal" H 2350 5600 60  0001 C CNN
+F 3 "" H 2350 5600 60  0001 C CNN
+	1    2350 5600
+	1    0    0    -1
+$EndComp
+Wire Wire Line
+	2150 5550 1950 5550
+Wire Wire Line
+	1950 5550 1950 5700
+Wire Wire Line
+	1950 5700 3150 5700
+Wire Wire Line
+	3150 5700 3150 5550
 $Comp
 L Device:C C7
 U 1 1 5BD0BD22
-P 6650 3550
-F 0 "C7" H 6765 3596 50  0000 L CNN
-F 1 "680uF" H 6765 3505 50  0000 L CNN
-F 2 "Capacitor_SMD:C_1206_3216Metric_Pad1.42x1.75mm_HandSolder" H 6688 3400 50  0001 C CNN
-F 3 "~" H 6650 3550 50  0001 C CNN
-	1    6650 3550
+P 3150 5400
+F 0 "C7" H 3265 5446 50  0000 L CNN
+F 1 "680uF" H 3265 5355 50  0000 L CNN
+F 2 "Capacitor_SMD:C_1206_3216Metric_Pad1.42x1.75mm_HandSolder" H 3188 5250 50  0001 C CNN
+F 3 "~" H 3150 5400 50  0001 C CNN
+	1    3150 5400
 	1    0    0    1
 $EndComp
 Wire Wire Line
-	5450 3700 5250 3700
-Connection ~ 5450 3700
+	1950 5550 1750 5550
+Connection ~ 1950 5550
 $Comp
 L power:GND #PWR0114
 U 1 1 5BD16850
-P 5250 3700
-F 0 "#PWR0114" H 5250 3450 50  0001 C CNN
-F 1 "GND" H 5255 3527 50  0000 C CNN
-F 2 "" H 5250 3700 50  0001 C CNN
-F 3 "" H 5250 3700 50  0001 C CNN
-	1    5250 3700
+P 1750 5550
+F 0 "#PWR0114" H 1750 5300 50  0001 C CNN
+F 1 "GND" H 1755 5377 50  0000 C CNN
+F 2 "" H 1750 5550 50  0001 C CNN
+F 3 "" H 1750 5550 50  0001 C CNN
+	1    1750 5550
 	-1   0    0    -1
 $EndComp
@@
 L power:+5V #PWR0115
 U 1 1 5BD195C6
-P 6050 3200
-F 0 "#PWR0115" H 6050 3050 50  0001 C CNN
-F 1 "+5V" H 6065 3373 50  0000 C CNN
-F 2 "" H 6050 3200 50  0001 C CNN
-F 3 "" H 6050 3200 50  0001 C CNN
-	1    6050 3200
+P 2550 5050
+F 0 "#PWR0115" H 2550 4900 50  0001 C CNN
+F 1 "+5V" H 2565 5223 50  0000 C CNN
+F 2 "" H 2550 5050 50  0001 C CNN
+F 3 "" H 2550 5050 50  0001 C CNN
+	1    2550 5050
 	-1   0    0    -1
 $EndComp
@@
 L Device:R_US R3
 U 1 1 5BD211F8
-P 5050 3400
-F 0 "R3" V 4845 3400 50  0000 C CNN
-F 1 "4.7K" V 4936 3400 50  0000 C CNN
-F 2 "Resistor_SMD:R_0805_2012Metric_Pad1.15x1.40mm_HandSolder" V 5090 3390 50  0001 C CNN
-F 3 "~" H 5050 3400 50  0001 C CNN
-	1    5050 3400
+P 1550 5250
+F 0 "R3" V 1345 5250 50  0000 C CNN
+F 1 "4.7K" V 1436 5250 50  0000 C CNN
+F 2 "Resistor_SMD:R_0805_2012Metric_Pad1.15x1.40mm_HandSolder" V 1590 5240 50  0001 C CNN
+F 3 "~" H 1550 5250 50  0001 C CNN
+	1    1550 5250
 	-1   0    0    -1
 $EndComp
@@
 L Device:R_US R4
 U 1 1 5BD2760A
-P 5350 3350
-F 0 "R4" V 5555 3350 50  0000 C CNN
-F 1 "4.7K" V 5464 3350 50  0000 C CNN
-F 2 "Resistor_SMD:R_0805_2012Metric_Pad1.15x1.40mm_HandSolder" V 5390 3340 50  0001 C CNN
-F 3 "~" H 5350 3350 50  0001 C CNN
-	1    5350 3350
+P 1850 5200
+F 0 "R4" V 2055 5200 50  0000 C CNN
+F 1 "4.7K" V 1964 5200 50  0000 C CNN
+F 2 "Resistor_SMD:R_0805_2012Metric_Pad1.15x1.40mm_HandSolder" V 1890 5190 50  0001 C CNN
+F 3 "~" H 1850 5200 50  0001 C CNN
+	1    1850 5200
 	1    0    0    1
 $EndComp
@@
 Text GLabel 8050 3450 0    50   Output ~ 0
 LIDAR_SCL
-Text Notes 4300 3650 0    50   ~ 0
+Text Notes 800  5500 0    50   ~ 0
 Blue
-Text Notes 4300 3550 0    50   ~ 0
+Text Notes 800  5400 0    50   ~ 0
 Green
 Wire Wire Line
-	5650 3600 5050 3600
-Wire Wire Line
-	5050 3600 5050 3550
-Wire Wire Line
-	5650 3500 5350 3500
-Wire Wire Line
-	5050 3250 5050 3200
-Wire Wire Line
-	5050 3200 5350 3200
-Connection ~ 5350 3200
-Wire Wire Line
-	5350 3200 5650 3200
-Connection ~ 6050 3200
-Wire Wire Line
-	6050 3200 6650 3200
-Wire Wire Line
-	6650 3400 6650 3200
-Wire Wire Line
-	5000 3600 5050 3600
-Connection ~ 5050 3600
-Wire Wire Line
-	5350 3500 5000 3500
-Connection ~ 5350 3500
-Wire Wire Line
-	5650 3400 5650 3200
-Connection ~ 5650 3200
-Wire Wire Line
-	5650 3200 6050 3200
+	2150 5450 1550 5450
+Wire Wire Line
+	1550 5450 1550 5400
+Wire Wire Line
+	2150 5350 1850 5350
+Wire Wire Line
+	1550 5100 1550 5050
+Wire Wire Line
+	1550 5050 1850 5050
+Connection ~ 1850 5050
+Wire Wire Line
+	1850 5050 2150 5050
+Connection ~ 2550 5050
+Wire Wire Line
+	2550 5050 3150 5050
+Wire Wire Line
+	3150 5250 3150 5050
+Wire Wire Line
+	1500 5450 1550 5450
+Connection ~ 1550 5450
+Wire Wire Line
+	1850 5350 1500 5350
+Connection ~ 1850 5350
+Wire Wire Line
+	2150 5250 2150 5050
+Connection ~ 2150 5050
+Wire Wire Line
+	2150 5050 2550 5050
 $Comp
 L 2019_NavB:12mm_Coin_Battery_Cell_Holder U2
 U 1 1 5BE8F78F
-P 10600 4050
-F 0 "U2" H 10812 4421 50  0000 L CNN
-F 1 "12mm_Coin_Battery_Cell_Holder" H 10812 4330 50  0000 L CNN
-F 2 "MRDT_Connectors:CR1220_Battery_Holder" H 10600 4050 50  0001 C CNN
-F 3 "" H 10600 4050 50  0001 C CNN
-	1    10600 4050
-	1    0    0    -1
-$EndComp
+P 4200 4100
+F 0 "U2" H 4412 4471 50  0000 L CNN
+F 1 "12mm_Coin_Battery_Cell_Holder" H 4412 4380 50  0000 L CNN
+F 2 "MRDT_Connectors:CR1220_Battery_Holder" H 4200 4100 50  0001 C CNN
+F 3 "" H 4200 4100 50  0001 C CNN
+	1    4200 4100
+	1    0    0    -1
+$EndComp
+Wire Wire Line
+	7000 2150 7000 2550
 $EndSCHEMATC
