File: 2019NavBoard/2019NavBoard.kicad_pcb (KiCad board)
At the start: 2 copper layers, 61 x 88.7 mm, 23 parts, among them J1 Conn_Coaxial, U5 FGPMMOPA6H

Commit message: Finalized Rev1
Parts:
- removed Conn3: Molex_SL_08, MRDT_Connectors:MOLEX_SL_08_Horizontal
- removed Conn4: 12mm_Coin_Cell_Battery_Holder, MRDT_Connectors:CR1220_Battery_Holder
- removed G***: LOGO, MRDT_Silkscreens:MRDT_Retro_Logo_34mmX21.5mm
- removed G***: LOGO, MRDT_Silkscreens:MRDT_Logo_20mm
- removed LIDAR1: Molex_SL_04, MRDT_Connectors:MOLEX_SL_04_Horizontal
- added IMU CONNECTOR: Molex_SL_08, MRDT_Connectors:MOLEX_SL_08_Horizontal, F.Cu at (149.6, 69.1)
- added LIDAR: LiDAR, MRDT_Connectors:MOLEX_SL_04_Horizontal, F.Cu at (169.5, 69.1)
- added U2: 12mm_Coin_Battery_Cell_Holder, MRDT_Connectors:CR1220_Battery_Holder, F.Cu at (126.0, 61.1)
- moved C7 1.77 mm to (173.4, 78.3)
- moved Conn1 0.24 mm to (131.2, 111.7)
- turned R3 to 90 degrees
- turned R4 to 180 degrees
Connections:
- C1 pad 1: LIDAR_MONITOR -> +5V
- C2 pad 3: LIDAR_MONITOR -> +5V
- C7 pad 2: LIDAR_MONITOR -> +5V
- R3 pad 1: Net-(LIDAR1-Pad2) -> +5V
- R3 pad 2: LIDAR_MONITOR -> LIDAR_SDA
- R4 pad 1: LIDAR_MONITOR -> LIDAR_SCL
- R4 pad 2: Net-(LIDAR1-Pad3) -> +5V
- U1 pad +5V: LIDAR_MONITOR -> +5V
- U1 pad PC4: LIDAR_MONITOR -> Net-(U1-PadPC4)
- U1 pad PC5: LIDAR_MONITOR -> Net-(U1-PadPC5)
Routing:
- net LIDAR_MONITOR: track 102.5 -> 0.00 mm, vias 2 -> 0
- net +5V: track 0.00 -> 90.3 mm, vias 0 -> 2
- net GND: track 21.3 -> 76.7 mm, vias 0 -> 2
- net VBACKUP: track 20.6 -> 72.5 mm, vias 0 -> 3
- net LIDAR_SCL: track 0.00 -> 13.5 mm, vias 0 -> 1
- net Net-(LIDAR1-Pad3): track 13.0 -> 0.00 mm, vias 1 -> 0
- net LIDAR_SDA: track 0.00 -> 7.53 mm
- net Net-(LIDAR1-Pad2): track 7.48 -> 0.00 mm
- net SCL(0): track 59.5 -> 60.8 mm
- net SDA(0): track 54.3 -> 55.5 mm
- net +3V3: track 44.7 -> 44.1 mm
- net TX(7): track 38.4 -> 38.9 mm

Commit message: Edit traces
Routing:
- net VBACKUP: track 72.5 -> 74.2 mm
Changed lines of the file:
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@@
     (thickness 1.6)
     (drawings 27)
-    (tracks 144)
+    (tracks 149)
     (zones 0)
     (modules 21)
@@
   (segment (start 152.439 95.1738) (end 153.5218 94.091) (width 0.381) (layer F.Cu) (net 4))
   (segment (start 144.1988 95.1738) (end 152.439 95.1738) (width 0.381) (layer F.Cu) (net 4))
-  (via (at 133.3246 69.3928) (size 0.8) (drill 0.4) (layers F.Cu B.Cu) (net 4))
   (segment (start 133.3246 61.3664) (end 133.6294 61.0616) (width 0.381) (layer F.Cu) (net 4))
-  (segment (start 133.3246 69.3928) (end 133.3246 61.3664) (width 0.381) (layer F.Cu) (net 4))
   (via (at 135.2296 87.249) (size 0.8) (drill 0.4) (layers F.Cu B.Cu) (net 4))
-  (segment (start 134.017502 86.036902) (end 135.2296 87.249) (width 0.381) (layer B.Cu) (net 4))
-  (segment (start 133.3246 69.3928) (end 134.017502 70.085702) (width 0.381) (layer B.Cu) (net 4))
-  (segment (start 134.017502 70.085702) (end 134.017502 86.036902) (width 0.381) (layer B.Cu) (net 4))
   (segment (start 136.274 87.249) (end 137.5 88.475) (width 0.381) (layer F.Cu) (net 4))
   (segment (start 135.2296 87.249) (end 136.274 87.249) (width 0.381) (layer F.Cu) (net 4))
@@
   (segment (start 118.3894 66.5734) (end 118.3894 66.5734) (width 0.381) (layer F.Cu) (net 4))
   (via (at 118.3894 66.5734) (size 0.8) (drill 0.4) (layers F.Cu B.Cu) (net 4))
-  (segment (start 120.4976 69.3928) (end 133.3246 69.3928) (width 0.381) (layer B.Cu) (net 4))
   (segment (start 118.3894 66.5734) (end 118.3894 67.2846) (width 0.381) (layer B.Cu) (net 4))
   (segment (start 118.3894 67.2846) (end 120.4976 69.3928) (width 0.381) (layer B.Cu) (net 4))
+  (segment (start 133.6294 61.0616) (end 133.6294 64.6176) (width 0.381) (layer F.Cu) (net 4))
+  (segment (start 133.6294 64.6176) (end 133.6294 66.5226) (width 0.381) (layer F.Cu) (net 4))
+  (segment (start 133.6294 66.5226) (end 133.6294 66.5226) (width 0.381) (layer F.Cu) (net 4))
+  (via (at 133.6294 66.5226) (size 0.8) (drill 0.4) (layers F.Cu B.Cu) (net 4))
+  (segment (start 120.4976 69.3928) (end 130.7592 69.3928) (width 0.381) (layer B.Cu) (net 4))
+  (segment (start 130.7592 69.3928) (end 133.6294 66.5226) (width 0.381) (layer B.Cu) (net 4))
+  (segment (start 134.829601 86.849001) (end 135.2296 87.249) (width 0.381) (layer B.Cu) (net 4))
+  (segment (start 134.2565 86.2759) (end 134.829601 86.849001) (width 0.381) (layer B.Cu) (net 4))
+  (segment (start 134.2565 67.715385) (end 134.2565 86.2759) (width 0.381) (layer B.Cu) (net 4))
+  (segment (start 133.6294 67.088285) (end 134.2565 67.715385) (width 0.381) (layer B.Cu) (net 4))
+  (segment (start 133.6294 66.5226) (end 133.6294 67.088285) (width 0.381) (layer B.Cu) (net 4))
   (segment (start 169.328732 88.519) (end 169.412592 88.43514) (width 0.381) (layer F.Cu) (net 9))
   (segment (start 162.123676 81.146224) (end 162.123676 79.375) (width 0.381) (layer F.Cu) (net 9))
