File: 2019NavBoard/2019NavBoard.kicad_pcb (KiCad board)
At the start: 2 copper layers, 61 x 88.7 mm, 21 parts, among them J1 Conn_Coaxial, U2 12mm_Coin_Battery_Cell_Holder, U5 FGPMMOPA6H

Commit message: After meeting
Routing:
- net GND: track 76.7 -> 62.2 mm
- net SDA(0): track 55.5 -> 54.9 mm
Other:
- board text added: "5V"
- board text added: "Nav Board Rev 1 Mars Rover Design Team Missouri S&T, 2019 Andre Biasella, Austin Christman"
- board text removed: "Nav Board Rev 1 2019 Mars Rover Design Team Missouri S&T Andre Biasella Austin Christman"
Changed lines of the file:
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@@
   (general
     (thickness 1.6)
-    (drawings 27)
-    (tracks 147)
+    (drawings 28)
+    (tracks 141)
     (zones 0)
     (modules 21)
@@
     (tags "capacitor handsolder")
     (attr smd)
-    (fp_text reference C1 (at 0 -1.82 180) (layer F.SilkS)
+    (fp_text reference C1 (at -0.0524 1.7526 180) (layer F.SilkS)
       (effects (font (size 1 1) (thickness 0.15)))
     )
@@
       (effects (font (size 1 1) (thickness 0.15)))
     )
-    (fp_text value OKI (at 6.35 -1.27) (layer F.SilkS)
+    (fp_text value OKI (at -1.6764 4.6101) (layer F.SilkS)
       (effects (font (size 1 1) (thickness 0.15)))
     )
@@
   (module MRDT_Connectors:CR1220_Battery_Holder (layer F.Cu)
     (at 126.0094 61.0616 180)
-    (fp_text reference U2 (at 4.3434 6.3246 180) (layer F.SilkS)
+    (fp_text reference U2 (at 7.5946 4.2164 180) (layer F.SilkS)
       (effects (font (size 1 1) (thickness 0.15)))
     )
@@
       (net 1 GND))
   )
+  (gr_text 5V (at 151.9174 110.5662) (layer F.SilkS)
+    (effects (font (size 1.5 1.5) (thickness 0.3)))
+  )
   (gr_line (start 165.5064 83.439) (end 165.5318 90.1192) (layer F.SilkS) (width 0.2))
   (gr_line (start 177.3174 55.6006) (end 116.3574 55.626) (layer Edge.Cuts) (width 0.15))
@@
   (gr_line (start 175.9585 83.439) (end 175.9458 90.1192) (layer F.SilkS) (width 0.2))
   (gr_line (start 165.5318 83.439) (end 175.9458 83.439) (layer F.SilkS) (width 0.2))
-  (gr_text "Nav Board Rev 1 2019\nMars Rover Design Team\nMissouri S&T\nAndre Biasella\nAustin Christman" (at 137.033 131.445) (layer F.SilkS)
-    (effects (font (size 1.5 1.5) (thickness 0.3)))
+  (gr_text "Nav Board Rev 1\nMars Rover Design Team\nMissouri S&T, 2019\nAndre Biasella, Austin Christman" (at 119.9134 126.1618) (layer F.SilkS)
+    (effects (font (size 1.5 1.5) (thickness 0.3)) (justify left))
   )
   (gr_line (start 118.4402 144.272) (end 175.2854 144.272) (layer Edge.Cuts) (width 0.15))
@@
   (segment (start 134.747 111.186502) (end 132.827302 113.1062) (width 0.381) (layer F.Cu) (net 1))
   (segment (start 134.747 107.5944) (end 134.747 111.186502) (width 0.381) (layer F.Cu) (net 1))
-  (segment (start 117.627001 69.443999) (end 126.0094 61.0616) (width 0.381) (layer F.Cu) (net 1))
-  (segment (start 117.627001 71.881001) (end 117.627001 69.443999) (width 0.381) (layer F.Cu) (net 1))
-  (segment (start 117.627001 71.881001) (end 117.627001 72.955803) (width 0.381) (layer F.Cu) (net 1))
-  (segment (start 117.627001 72.955803) (end 117.941698 73.2705) (width 0.381) (layer F.Cu) (net 1))
-  (segment (start 117.941698 73.2705) (end 118.2793 73.2705) (width 0.381) (layer F.Cu) (net 1))
-  (segment (start 118.2793 73.2705) (end 118.8974 73.8886) (width 0.381) (layer F.Cu) (net 1))
-  (segment (start 118.3386 82.05121) (end 118.3386 83.6422) (width 0.381) (layer F.Cu) (net 1))
-  (segment (start 118.8974 81.49241) (end 118.3386 82.05121) (width 0.381) (layer F.Cu) (net 1))
-  (segment (start 118.8974 73.8886) (end 118.8974 81.49241) (width 0.381) (layer F.Cu) (net 1))
   (via (at 140.8684 85.4202) (size 0.8) (drill 0.4) (layers F.Cu B.Cu) (net 1))
   (segment (start 137.4902 85.353) (end 140.8012 85.353) (width 0.381) (layer F.Cu) (net 1))
@@
   (segment (start 143.5608 82.7278) (end 145.0086 82.7278) (width 0.381) (layer B.Cu) (net 1))
   (segment (start 140.8684 85.4202) (end 143.5608 82.7278) (width 0.381) (layer B.Cu) (net 1))
+  (segment (start 118.8974 73.1514) (end 117.627001 71.881001) (width 0.381) (layer F.Cu) (net 1))
+  (segment (start 118.8974 81.49241) (end 118.8974 73.1514) (width 0.381) (layer F.Cu) (net 1))
+  (segment (start 118.3386 83.6422) (end 118.3386 82.05121) (width 0.381) (layer F.Cu) (net 1))
+  (segment (start 118.3386 82.05121) (end 118.8974 81.49241) (width 0.381) (layer F.Cu) (net 1))
   (segment (start 143.4719 99.5934) (end 134.747 99.5934) (width 0.381) (layer F.Cu) (net 2))
   (segment (start 147.066 103.1875) (end 143.4719 99.5934) (width 0.381) (layer F.Cu) (net 2))
@@
   (segment (start 152.3492 72.7202) (end 155.9814 69.088) (width 0.381) (layer B.Cu) (net 17))
   (segment (start 150.749 72.7202) (end 152.3492 72.7202) (width 0.381) (layer B.Cu) (net 17))
-  (segment (start 140.487001 117.601001) (end 141.174199 117.601001) (width 0.381) (layer F.Cu) (net 18))
   (segment (start 150.9268 71.6026) (end 153.4414 69.088) (width 0.381) (layer B.Cu) (net 18))
   (segment (start 149.2504 71.6026) (end 150.9268 71.6026) (width 0.381) (layer B.Cu) (net 18))
