File: NavBoard_Hardware/2019NavBoard.kicad_pcb (KiCad board)
At the start: 2 copper layers, 61 x 100 mm, 44 parts, among them J1 Conn_Coaxial, U2 12mm_Coin_Battery_Cell_Holder, U3 AP1059, U4 AP1059, U5 FGPMMOPA6H

Commit message: rev1
Parts:
- removed D3, D4: D_Schottky, Diode_SMD:D_0603_1608Metric_Pad1.05x0.95mm_HandSolder
- removed L2, L3: 47u, MRDT_Passives:ETQ-P4M470YFN_Inductor
- added G***: LOGO, MRDT_Silkscreens:MRDT_Logo_20mm, F.Cu at (127.8, 138.8)
- added G***: LOGO, NavBoard_Hardware_2:Andrea_Biasella_22mmx9.3mm, F.Cu at (140.1, 146.8)
- U3, U4: value AP1059 -> OKI; footprint Package_SO:SOIC-8_3.9x4.9mm_P1.27mm -> MRDT_Devices:OKI_Horizontal
- moved D8 37.4 mm to (121.3, 73.0)
- moved R7 37.4 mm to (124.7, 75.9)
- moved R8 37.4 mm to (124.7, 73.0)
- moved D7 37.4 mm to (121.3, 75.9)
- moved C9 29.9 mm to (146.2, 106.9), turned to 0 degrees
- moved C10 12.4 mm to (149.6, 106.9), turned to 180 degrees
- moved C11 11.6 mm to (156.9, 91.0), turned to 270 degrees
- moved U4 11.3 mm to (159.5, 97.8), turned to 90 degrees
- moved U3 9.07 mm to (152.9, 104.5), turned to 180 degrees
- moved C8 8.84 mm to (156.9, 94.4), turned to 90 degrees
- moved D1 3.85 mm to (143.3, 80.1), turned to 270 degrees
- moved U5 3.05 mm to (148.2, 71.9)
- moved R1 2.30 mm to (145.2, 80.1), turned to 270 degrees
- moved C5 1.80 mm to (144.3, 77.7)
- moved Conn2 0.51 mm to (168.9, 65.5)
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Connections:
- C10 pad 1: GND -> Net-(C10-Pad1)
- C10 pad 2: +3V3 -> GND
- C11 pad 1: GND -> +3V3
- C11 pad 2: +5V -> GND
- C8 pad 1: Net-(C8-Pad1) -> Net-(C10-Pad1)
- C9 pad 1: Net-(C8-Pad1) -> +5V
- Conn1 pad 2: Net-(C8-Pad1) -> Net-(C10-Pad1)
- U3 pad 1: Net-(C8-Pad1) -> Net-(C10-Pad1)
- U3 pad 2: Net-(D3-Pad1) -> GND
- U3 pad 3: +3V3 -> +5V
- U4 pad 1: Net-(C8-Pad1) -> Net-(C10-Pad1)
- U4 pad 2: Net-(D4-Pad1) -> GND
- U4 pad 3: +5V -> +3V3
Routing:
- net Net-(C8-Pad1): track 70.1 -> 0.00 mm, vias 3 -> 0
- net Net-(C10-Pad1): track 0.00 -> 49.1 mm, vias 0 -> 1
- net +3V3: track 72.7 -> 38.8 mm
- net Net-(D3-Pad1): track 14.3 -> 0.00 mm
- net TivaTX(7): track 79.4 -> 68.9 mm, vias 5 -> 2
- net Net-(D4-Pad1): track 10.2 -> 0.00 mm
- net GND: track 26.2 -> 18.4 mm, vias 4 -> 2
- net TivaRX(7): track 78.5 -> 72.0 mm
- net +5V: track 112.9 -> 106.5 mm
- net VBACKUP: track 62.1 -> 56.7 mm
- net LIDAR_SDA: track 93.1 -> 88.5 mm, vias 5 -> 4
- net Net-(R1-Pad1): track 5.45 -> 3.93 mm
- net /EXAnt: track 49.0 -> 50.3 mm
- net SW_Flg2: track 16.1 -> 17.2 mm
- net LIDAR_SCL: track 69.7 -> 70.6 mm
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Other:
- board text added: "+3.3V"
- board text added: "Autonomy"
- board text added: "GPS"
- board text added: "RX(SRC)"
- board text added: "TX(SRC)"
- board text removed: "Autonomy LEDS"
- board text removed: "GPS SCR"
- board text removed: "RX"
- board text removed: "TX"

Commit message: worked on Board
Parts:
- removed U2: 12mm_Coin_Battery_Cell_Holder, MRDT_Connectors:CR1220_Battery_Holder
- added BT1: Battery_Cell, MRDT_Connectors:CR1220_Battery_Holder, F.Cu at (126.2, 58.2)
- added G***: LOGO, NavBoard_Hardware_2:Austin_Christman_22mmx8.3mm, F.Cu at (162.8, 147.6)
- C7: footprint Capacitor_SMD:C_0603_1608Metric_Pad1.05x0.95mm_HandSolder -> Capacitor_THT:CP_Radial_D6.3mm_P2.50mm
- moved C9 32.1 mm to (171.8, 87.6), turned to 180 degrees
- moved C5 28.5 mm to (118.5, 65.5)
- moved C10 26.5 mm to (167.8, 87.6), turned to 0 degrees
- moved D10 25.5 mm to (155.4, 107.8), turned to 180 degrees
- moved D9 23.4 mm to (155.6, 104.5), turned to 180 degrees
- moved Conn1 21.6 mm to (130.0, 110.5), turned to 0 degrees
- moved D12 21.2 mm to (155.5, 125.1)
- moved D11 21.1 mm to (155.5, 122.0)
- moved D5 21.1 mm to (155.5, 114.8)
- moved D6 21.0 mm to (155.4, 118.9)
- moved D2 21.0 mm to (155.5, 111.6)
- moved R12 20.7 mm to (151.5, 125.1)
- moved R5 20.7 mm to (151.7, 114.8)
- moved R11 20.6 mm to (151.5, 122.0)
- moved R2 20.5 mm to (151.6, 111.6)
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Connections:
- net SCL(0) renamed IMU_SCL
- net SDA(0) renamed IMU_SDA
- net TivaRX(7) renamed TivaRX
- net TivaTX(7) renamed TivaTX
Routing:
- net LIDAR_SDA: track 88.5 -> 74.2 mm
- net Error_LED: track 20.2 -> 32.4 mm
- net SW_Flg1: track 17.5 -> 29.3 mm
- net SW_Flg2: track 17.2 -> 28.9 mm
- net LIDAR_SCL: track 70.6 -> 59.1 mm
- net +5V: track 106.5 -> 116.9 mm, vias 0 -> 2
- net GND: track 18.4 -> 12.2 mm, vias 2 -> 0
- net +3V3: track 38.8 -> 34.8 mm
- net TivaRX: track 72.0 -> 69.5 mm
- net IMU_SCL: track 76.6 -> 78.9 mm
- net /EXAnt: track 50.3 -> 48.0 mm
- net IMU_SDA: track 89.4 -> 87.4 mm
- net TivaTX: track 68.9 -> 70.5 mm, vias 2 -> 3
- net Net-(C3-Pad2): track 5.86 -> 7.13 mm
- net VBACKUP: track 56.7 -> 55.5 mm
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Other:
- board size 61 x 100 mm -> 61 x 100.1 mm
- board text added: "CR 1220 Battery"
- board text removed: "+3.3V Backup"
