File: NavBoard_Hardware/2019NavBoard.sch (KiCad schematic (older format))
At the start: 22 parts, among them J1 Conn_Coaxial, U1C1 TM4C129E_Launchpad, U2 12mm_Coin_Battery_Cell_Holder, U5 FGPMMOPA6H

Commit message: Did good work
Parts:
- removed C1, C6: 10uF, Capacitor_SMD:C_1206_3216Metric_Pad1.42x1.75mm_HandSolder, symbol Device:CP1
- removed C2: OKI, MRDT_Devices:OKI_Horizontal, symbol MRDT_Devices:OKI
- added C10, C11, C8, C9: 10u, symbol Device:C_Small
- added D3, D4: D_Schottky, symbol Device:D_Schottky
- added D? (x6): PWR, LED_SMD:LED_0805_2012Metric_Pad1.15x1.40mm_HandSolder, symbol Device:LED
- added L2, L3: 47u, symbol pspice:INDUCTOR
- added R? (x6): 500, Resistor_SMD:R_0805_2012Metric_Pad1.15x1.40mm_HandSolder, symbol Device:R
- added U3, U4: AP1059, symbol MRDT_ICs:AP1059
- C3, C4, C5: symbol Device:CP1 -> Device:C_Small
- D1, D2: symbol Device:LED_Small -> Device:LED
- R1, R3, R4: symbol Device:R_US -> Device:R
- R2: value 1K -> 500; symbol Device:R_US -> Device:R
Connections:
- net labels added: +3.3V, EXAnt, SW_Error, SW_Flag1, SW_Flag2, Serial7, TivaRX(7), TivaTX(7)
- net labels removed: RX(7), TX(7)
- wire segments 92 -> 155
Other:
- note added: "BLU\n"
- note added: "Battery Backup\n"
- note added: "Connections"
- note added: "GPS and Backup Battery"
- note added: "GPS: FGPMMOPA6H"
- note added: "GREN\n"
- note added: "IMU"
- note added: "Indicators"
- note added: "LIDAR\n"
- note added: "RED\n"
- note added: "TIVA\n"
- note added: "YELO\n"
- note removed: "Connector to off board IMU and Board Power LED"
- note removed: "GPS, and LiDAR\n"
- note removed: "TIVA and Battery Backup\n\n"
- moved on the sheet: C7

Commit message: Editied schematic and made PCB
Parts:
- C10, C11, C8, C9: footprint (none) -> Capacitor_SMD:C_0603_1608Metric_Pad1.05x0.95mm_HandSolder
- C3, C4, C5: footprint Capacitor_SMD:C_0805_2012Metric_Pad1.15x1.40mm_HandSolder -> Capacitor_SMD:C_0603_1608Metric_Pad1.05x0.95mm_HandSolder
- C7: footprint Capacitor_SMD:C_1206_3216Metric_Pad1.42x1.75mm_HandSolder -> Capacitor_SMD:C_0603_1608Metric_Pad1.05x0.95mm_HandSolder
- D1, D2: footprint LED_SMD:LED_0805_2012Metric_Pad1.15x1.40mm_HandSolder -> LED_SMD:LED_0603_1608Metric_Pad1.05x0.95mm_HandSolder
- D10, D5, D6, D7, D8, D9: renamed from D?; footprint LED_SMD:LED_0805_2012Metric_Pad1.15x1.40mm_HandSolder -> LED_SMD:LED_0603_1608Metric_Pad1.05x0.95mm_HandSolder
- D3, D4: footprint (none) -> Diode_SMD:D_0603_1608Metric_Pad1.05x0.95mm_HandSolder
- L2, L3: footprint (none) -> MRDT_Passives:ETQ-P4M470YFN_Inductor
- R1, R2, R3, R4: footprint Resistor_SMD:R_0805_2012Metric_Pad1.15x1.40mm_HandSolder -> Resistor_SMD:R_0603_1608Metric_Pad1.05x0.95mm_HandSolder
- R10, R5, R6, R7, R8, R9: renamed from R?; footprint Resistor_SMD:R_0805_2012Metric_Pad1.15x1.40mm_HandSolder -> Resistor_SMD:R_0603_1608Metric_Pad1.05x0.95mm_HandSolder
- U3, U4: footprint (none) -> Package_SO:SOIC-8_3.9x4.9mm_P1.27mm
Connections:
- net labels added: Error_LED
- net labels removed: SW_Error, SW_Flag1, SW_Flag2
- wire segments 155 -> 156

Commit message: Fixed traces
Parts:
- added D11, D12: PWR, LED_SMD:LED_0603_1608Metric_Pad1.05x0.95mm_HandSolder, symbol Device:LED
- added R11, R12: 500, Resistor_SMD:R_0603_1608Metric_Pad1.05x0.95mm_HandSolder, symbol Device:R
- U1: renamed from U1C1; value TM4C129E_Launchpad -> ~
Connections:
- net labels added: SW_Flg1, SW_Flg2
- wire segments 156 -> 165
Other:
- moved on the sheet: D10, D2, D5, D6, D7, D8, D9, R10, R2, R5, R6, R7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

Commit message: rev1
Parts:
- removed D3, D4: D_Schottky, Diode_SMD:D_0603_1608Metric_Pad1.05x0.95mm_HandSolder, symbol Device:D_Schottky
- removed L2, L3: 47u, MRDT_Passives:ETQ-P4M470YFN_Inductor, symbol pspice:INDUCTOR
- removed U3, U4: AP1059, Package_SO:SOIC-8_3.9x4.9mm_P1.27mm, symbol MRDT_ICs:AP1059
- added U3, U4: OKI, MRDT_Devices:OKI_Horizontal, symbol MRDT_Devices:OKI
Connections:
- wire segments 165 -> 134

Commit message: worked on Board
Parts:
- removed U2: 12mm_Coin_Battery_Cell_Holder, MRDT_Connectors:CR1220_Battery_Holder, symbol 2019_NavB:12mm_Coin_Battery_Cell_Holder
- added BT1: Battery_Cell, MRDT_Connectors:CR1220_Battery_Holder, symbol Device:Battery_Cell
- C7: footprint Capacitor_SMD:C_0603_1608Metric_Pad1.05x0.95mm_HandSolder -> Capacitor_THT:CP_Radial_D6.3mm_P2.50mm
Connections:
- net labels added: IMU_SCL, IMU_SDA, TivaRX, TivaTX
- net labels removed: SCL(0), SDA(0), Serial7, TivaRX(7), TivaTX(7)
- wire segments 134 -> 136
Other:
- note added: "I2C2"
- note added: "Serial 7\n"
- note added: "YELO"
Changed lines of the file:
@@
 	6550 2200 7000 2200
 Text GLabel 5550 2300 0    50   Output ~ 0
-TivaRX(7)
+TivaRX
 Text GLabel 5550 2200 0    50   Input ~ 0
-TivaTX(7)
+TivaTX
 $Comp
 L pspice:INDUCTOR L1
@@
 	1    0    0    -1
 $EndComp
-Wire Wire Line
-	4216 2686 4016 2686
-Wire Wire Line
-	3816 2236 4116 2236
-Wire Wire Line
-	4016 2686 4016 2786
-Connection ~ 4016 2686
-Wire Wire Line
-	4016 2686 3816 2686
 $Comp
 L power:GND #PWR0106
 U 1 1 5BC5C835
-P 4016 2786
-F 0 "#PWR0106" H 4016 2536 50  0001 C CNN
-F 1 "GND" H 4021 2613 50  0000 C CNN
-F 2 "" H 4016 2786 50  0001 C CNN
-F 3 "" H 4016 2786 50  0001 C CNN
-	1    4016 2786
+P 4250 2900
+F 0 "#PWR0106" H 4250 2650 50  0001 C CNN
+F 1 "GND" H 4255 2727 50  0000 C CNN
+F 2 "" H 4250 2900 50  0001 C CNN
+F 3 "" H 4250 2900 50  0001 C CNN
+	1    4250 2900
 	1    0    0    -1
 $EndComp
@@
 L Device:C_Small C5
 U 1 1 5BC5C880
-P 3816 2486
-F 0 "C5" H 3931 2532 50  0000 L CNN
-F 1 "1uF" H 3931 2441 50  0000 L CNN
-F 2 "Capacitor_SMD:C_0603_1608Metric_Pad1.05x0.95mm_HandSolder" H 3816 2486 50  0001 C CNN
-F 3 "~" H 3816 2486 50  0001 C CNN
-	1    3816 2486
-	1    0    0    -1
-$EndComp
-Wire Wire Line
-	4116 2236 4116 2136
-Wire Wire Line
-	4116 2136 3916 2136
-Connection ~ 4116 2236
-Wire Wire Line
-	4116 2236 4216 2236
-Text GLabel 3916 2136 0    50   Input ~ 0
+P 3950 2650
+F 0 "C5" H 4065 2696 50  0000 L CNN
+F 1 "1uF" H 4065 2605 50  0000 L CNN
+F 2 "Capacitor_SMD:C_0603_1608Metric_Pad1.05x0.95mm_HandSolder" H 3950 2650 50  0001 C CNN
+F 3 "~" H 3950 2650 50  0001 C CNN
+	1    3950 2650
+	1    0    0    -1
+$EndComp
+Text GLabel 3900 2250 0    50   Input ~ 0
 VBACKUP
 Wire Wire Line
@@
 DRDYM
 Text GLabel 1050 4100 2    50   Input ~ 0
-SDA(0)
+IMU_SDA
 Text GLabel 1050 4000 2    50   Input ~ 0
-SCL(0)
+IMU_SCL
 $Comp
 L Device:R R2
@@
 $EndComp
 Text GLabel 8850 2000 0    50   Input ~ 0
-SCL(0)
+IMU_SCL
 Text GLabel 8850 2100 0    50   Input ~ 0
-SDA(0)
-Text GLabel 8850 2400 0    50   Output ~ 0
+IMU_SDA
+Text GLabel 8850 2400 0    50   Input ~ 0
 INT2AG
-Text GLabel 8850 2500 0    50   Output ~ 0
+Text GLabel 8850 2500 0    50   Input ~ 0
 INT1AG
 Text GLabel 8850 3200 0    50   Input ~ 0
@@
 Text GLabel 8850 3300 0    50   Input ~ 0
 DRDYM
-Text GLabel 8650 1400 0    50   Output ~ 0
-TivaRX(7)
-Text GLabel 8850 1500 0    50   Input ~ 0
-TivaTX(7)
+Text GLabel 8850 1400 0    50   Input ~ 0
+TivaRX
+Text GLabel 8850 1500 0    50   Output ~ 0
+TivaTX
 $Comp
 L MRDT_Sensors:FGPMMOPA6H U5
@@
 F 0 "C7" H 3100 4300 50  0000 L CNN
 F 1 "680uF" H 3100 4100 50  0000 L CNN
-F 2 "Capacitor_SMD:C_0603_1608Metric_Pad1.05x0.95mm_HandSolder" H 3088 4050 50  0001 C CNN
+F 2 "Capacitor_THT:CP_Radial_D6.3mm_P2.50mm" H 3088 4050 50  0001 C CNN
 F 3 "~" H 3050 4200 50  0001 C CNN
 	1    3050 4200
@@
 	1    0    0    1
 $EndComp
-Text GLabel 8850 3000 0    50   Output ~ 0
+Text GLabel 8850 3000 0    50   Input ~ 0
 LIDAR_SDA
-Text GLabel 8850 3100 0    50   Output ~ 0
+Text GLabel 8850 3100 0    50   Input ~ 0
 LIDAR_SCL
 Text Notes 1500 4250 0    50   ~ 0
@@
 	2600 4050 2600 3850
 Connection ~ 2600 3850
-$Comp
-L 2019_NavB:12mm_Coin_Battery_Cell_Holder U2
-U 1 1 5BE8F78F
-P 4216 2786
-F 0 "U2" H 4300 3222 50  0000 L CNN
-F 1 "12mm_Coin_Battery_Cell_Holder" H 3500 2472 50  0000 L CNN
-F 2 "MRDT_Connectors:CR1220_Battery_Holder" H 4216 2786 50  0001 C CNN
-F 3 "" H 4216 2786 50  0001 C CNN
-	1    4216 2786
-	1    0    0    -1
-$EndComp
 $Comp
 L Device:C_Small C10
@@
 	7000 1500 7000 2200
 Wire Wire Line
-	3816 2236 3816 2386
-Wire Wire Line
-	3816 2586 3816 2686
-Wire Wire Line
 	9950 1150 9950 1200
 Wire Wire Line
@@
 Wire Wire Line
 	8850 3300 8950 3300
-Text Label 8950 1400 2    50   ~ 0
-Serial7
-Wire Wire Line
-	8650 1400 8950 1400
 Text Notes 600  3750 0    79   ~ 16
 IMU
@@
 	4800 3950 4800 4000
 Text GLabel 5100 3950 1    39   Input ~ 0
-SDA(0)
+IMU_SDA
 $Comp
 L Device:R R10
@@
 	5100 4000 5100 3950
 Text GLabel 5450 3950 1    39   Input ~ 0
-TivaRX(7)
+TivaRX
 Wire Wire Line
 	5450 3950 5450 4000
 Text GLabel 5800 4000 1    39   Input ~ 0
-TivaTX(7)
+TivaTX
 Text Notes 3700 5100 0    39   ~ 0
 GREN\n
@@
 Text Notes 4400 5100 0    39   ~ 0
 RED\n
-Text GLabel 9950 1400 2    50   Input ~ 0
+Text GLabel 9950 1400 2    50   Output ~ 0
 Error_LED
 Wire Wire Line
@@
 Text GLabel 6500 3950 1    50   Input ~ 0
 SW_Flg2
-Text GLabel 9950 1500 2    50   Input ~ 0
+Text GLabel 9950 1500 2    50   Output ~ 0
 SW_Flg1
-Text GLabel 9950 1600 2    50   Input ~ 0
+Text GLabel 9950 1600 2    50   Output ~ 0
 SW_Flg2
 Wire Wire Line
@@
 Wire Wire Line
 	1600 2350 1700 2350
+Wire Wire Line
+	3950 2450 3950 2550
+Wire Wire Line
+	4250 2900 4250 2850
+Connection ~ 4250 2850
+Wire Wire Line
+	4250 2850 3950 2850
+Wire Wire Line
+	3900 2250 4200 2250
+Wire Wire Line
+	4200 2250 4200 2450
+Connection ~ 4200 2450
+Wire Wire Line
+	4200 2450 3950 2450
+Wire Wire Line
+	4450 2450 4200 2450
+Wire Wire Line
+	4450 2850 4250 2850
+Wire Wire Line
+	8850 1400 8950 1400
+Text Notes 8500 1350 0    50   ~ 0
+Serial 7\n
+Text Notes 8700 2350 2    50   ~ 0
+I2C2
+$Comp
+L Device:Battery_Cell BT1
+U 1 1 5C1A9C73
+P 4450 2700
+F 0 "BT1" H 4568 2796 50  0000 L CNN
+F 1 "Battery_Cell" H 4568 2705 50  0000 L CNN
+F 2 "MRDT_Connectors:CR1220_Battery_Holder" V 4450 2760 50  0001 C CNN
+F 3 "~" V 4450 2760 50  0001 C CNN
+	1    4450 2700
+	1    0    0    -1
+$EndComp
+Wire Wire Line
+	4450 2450 4450 2500
+Wire Wire Line
+	4450 2800 4450 2850
+Wire Wire Line
+	3950 2850 3950 2750
+Text Notes 6250 5100 2    39   ~ 0
+YELO
+Text Notes 6600 5100 2    39   ~ 0
+YELO\n
 $EndSCHEMATC
