File: NavBoard_Hardware/NavBoard_Hardware.sch (KiCad schematic (older format))
At the start: 40 parts, among them J1 Conn_Coaxial, U3 OKI, U4 OKI, U5 FGPMMOPA6H

Commit message: just in case push
Other:
- note added: "I2C0"
Changed lines of the file:
@@
 EESchema Schematic File Version 4
-LIBS:2019NavBoard-cache
+LIBS:NavBoard_Hardware-cache
 EELAYER 26 0
 EELAYER END
@@
 Text Notes 3700 5100 0    39   ~ 0
 GREN\n
-Text Notes 5400 5100 0    39   ~ 0
+Text Notes 6100 5100 0    39   ~ 0
 BLU\n
-Text Notes 5750 5100 0    39   ~ 0
+Text Notes 6450 5100 0    39   ~ 0
 BLU\n
 Text Notes 5050 5100 0    39   ~ 0
@@
 Text Notes 8500 1350 0    50   ~ 0
 Serial 7\n
-Text Notes 8700 2350 2    50   ~ 0
-I2C2
+Text Notes 8450 2050 2    50   ~ 0
+I2C0
 $Comp
 L Device:Battery_Cell BT1
@@
 Wire Wire Line
 	3950 2850 3950 2750
-Text Notes 6250 5100 2    39   ~ 0
+Text Notes 5550 5100 2    39   ~ 0
 YELO
-Text Notes 6600 5100 2    39   ~ 0
+Text Notes 5900 5100 2    39   ~ 0
 YELO\n
+Text Notes 8400 3100 2    50   ~ 0
+I2C2
 $EndSCHEMATC

Commit message: Updated to rev2 libraries
Parts:
- BT1: footprint MRDT_Connectors:CR1220_Battery_Holder -> MRDT_Shields:TM4C129E_Launchpad_X9_SMD_BOTTOM
- C7: symbol Device:C -> Device:CP1
- Conn1: footprint MRDT_Connectors:Anderson_2_Horisontal_Side_by_Side -> MRDT_Connectors:Anderson_2_Horizontal_Side_by_Side
- J1: footprint Connector_Coaxial:SMA_Amphenol_132134-16_Vertical -> Connector_Coaxial:SMB_Jack_Vertical
Changed lines of the file:
@@
 F 0 "Conn1" H 1300 2400 60  0000 C CNN
 F 1 "AndersonPP" H 1300 2300 60  0000 C CNN
-F 2 "MRDT_Connectors:Anderson_2_Horisontal_Side_by_Side" H 1050 1900 60  0001 C CNN
+F 2 "MRDT_Connectors:Anderson_2_Horizontal_Side_by_Side" H 1050 1900 60  0001 C CNN
 F 3 "" H 1050 1900 60  0001 C CNN
 	1    1200 2450
@@
 F 0 "Conn1" H 1306 1937 60  0000 C CNN
 F 1 "AndersonPP" H 1306 1831 60  0000 C CNN
-F 2 "MRDT_Connectors:Anderson_2_Horisontal_Side_by_Side" H 950 1000 60  0001 C CNN
+F 2 "MRDT_Connectors:Anderson_2_Horizontal_Side_by_Side" H 950 1000 60  0001 C CNN
 F 3 "" H 950 1000 60  0001 C CNN
 	2    1100 1550
@@
 F 0 "J1" H 6949 2276 50  0000 L CNN
 F 1 "Conn_Coaxial" H 6850 2500 50  0000 L CNN
-F 2 "Connector_Coaxial:SMA_Amphenol_132134-16_Vertical" H 6850 2300 50  0001 C CNN
+F 2 "Connector_Coaxial:SMB_Jack_Vertical" H 6850 2300 50  0001 C CNN
 F 3 " ~" H 6850 2300 50  0001 C CNN
 	1    6850 2300
@@
 	2600 4350 2600 4500
 $Comp
-L Device:C C7
+L Device:CP1 C7
 U 1 1 5BD0BD22
 P 3050 4200
 F 0 "C7" H 3100 4300 50  0000 L CNN
-F 1 "680uF" H 3100 4100 50  0000 L CNN
+F 1 "680uF" H 2800 4100 50  0000 L CNN
 F 2 "Capacitor_THT:CP_Radial_D6.3mm_P2.50mm" H 3088 4050 50  0001 C CNN
 F 3 "~" H 3050 4200 50  0001 C CNN
 	1    3050 4200
-	1    0    0    1
+	-1   0    0    -1
 $EndComp
 $Comp
@@
 $EndComp
 $Comp
-L power:+5V #PWR0115
-U 1 1 5BD195C6
-P 3050 3850
-F 0 "#PWR0115" H 3050 3700 50  0001 C CNN
-F 1 "+5V" H 3065 4023 50  0000 C CNN
-F 2 "" H 3050 3850 50  0001 C CNN
-F 3 "" H 3050 3850 50  0001 C CNN
-	1    3050 3850
-	-1   0    0    -1
-$EndComp
-$Comp
 L Device:R R3
 U 1 1 5BD211F8
@@
 Wire Wire Line
 	3050 4350 3050 4500
-Connection ~ 3050 3850
 Wire Wire Line
 	2600 3850 3050 3850
@@
 F 0 "BT1" H 4568 2796 50  0000 L CNN
 F 1 "Battery_Cell" H 4568 2705 50  0000 L CNN
-F 2 "MRDT_Connectors:CR1220_Battery_Holder" V 4450 2760 50  0001 C CNN
+F 2 "MRDT_Shields:TM4C129E_Launchpad_X9_SMD_BOTTOM" V 4450 2760 50  0001 C CNN
 F 3 "~" V 4450 2760 50  0001 C CNN
 	1    4450 2700
@@
 Text Notes 8400 3100 2    50   ~ 0
 I2C2
+$Comp
+L power:+3V3 #PWR0115
+U 1 1 5C6D088C
+P 3050 3850
+F 0 "#PWR0115" H 3050 3700 50  0001 C CNN
+F 1 "+3V3" H 3065 4023 50  0000 C CNN
+F 2 "" H 3050 3850 50  0001 C CNN
+F 3 "" H 3050 3850 50  0001 C CNN
+	1    3050 3850
+	1    0    0    -1
+$EndComp
+Connection ~ 3050 3850
 $EndSCHEMATC
