File: NavBoard_Hardware/NavBoard_Hardware.kicad_sch (KiCad schematic)
At the start: 16 parts, among them J1 6 Pin Molex Micro-Fit, J2 Raspberry Pi - Header Socket

Commit message: Swapped TX and RX for GPS pins
Connections:
- net M8Q-RX: now also J2.8 (GPIO14/TXD); no longer J2.10 (GPIO15/RXD)
- net M8Q-TX: now also J2.10 (GPIO15/RXD); no longer J2.8 (GPIO14/TXD)
Changed lines of the file:
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@@
     (effects (font (size 1.27 1.27)) (justify left bottom))
   )
-  (label "M8Q-RX" (at 139.065 97.79 180)
+  (label "M8Q-RX" (at 139.065 95.25 180)
     (effects (font (size 1.27 1.27)) (justify right bottom))
   )
@@
     (effects (font (size 1.27 1.27)) (justify left bottom))
   )
-  (label "M8Q-TX" (at 139.065 95.25 180)
+  (label "M8Q-TX" (at 139.065 97.79 180)
     (effects (font (size 1.27 1.27)) (justify right bottom))
   )
