File: NavBoard_Hardware/_autosave-main_board.kicad_sch (KiCad schematic)
At the start: 10 parts, among them J2 8P8C_LED_Shielded, J3 Conn_01x06

Commit message: Added connectors, cleaned up file directory
Parts:
- J2: value 8P8C_LED_Shielded -> Ethernet Jack w/ Magnetics; footprint Connector_RJ:RJ45_Amphenol_RJHSE538X -> Connector_RJ:RJ45_Cetus_J1B1211CCD_Horizontal; Part Opt 1 (none) -> Link-PP LPJ4012AHNL; Part Opt 2 (none) -> Cetus J1B1211CCD
- J3: value Conn_01x06 -> Conn_02x03; footprint (none) -> Connector_PinSocket_2.00mm:PinSocket_2x03_P2.00mm_Vertical; Field4 (none) -> 2.00mm Pins
- J? (x2): footprint Nav_Board:24Pin_To_16Pin_2.54mm -> Nav_Board:24Pin_To_16Pin_2.54mm_Separate_Pins; symbol Nav_Board:24Pin_To_16Pin_2.54mm_Alt -> Nav_Board:24Pin_To_16Pin_2.54mm_Separate_Pins_Alt
Connections:
- net ETHERNET_RX- is gone; now on net GND: J2.6, J3.1 (Pin_1)
- net Pin1L is gone; now on net GND: J?.1
- net Pin1R is gone; now on net +5V: J?.48
- net Pin2R is gone; now on net GND: J?.47
- net GND: now also C15.2, J2.8
- net Pin10L_Small: now also J?.18a; no longer J?.18
- net Pin10R_Small: now also J?.31a; no longer J?.31
- net Pin11L_Small: now also J?.19a; no longer J?.19
- net Pin11R_Small: now also J?.30a; no longer J?.30
- net Pin12L_Small: now also J?.20a; no longer J?.20
- net Pin12R_Small: now also J?.29a; no longer J?.29
- net Pin13L_Small: now also J?.21a; no longer J?.21
- net Pin13R_Small: now also J?.28a; no longer J?.28
- net Pin14L_Small: now also J?.22a; no longer J?.22
- net Pin14R_Small: now also J?.27a; no longer J?.27
- net Pin15L_Small: now also J?.23a; no longer J?.23
- net Pin15R_Small: now also J?.26a; no longer J?.26
- net Pin16L_Small: now also J?.24a; no longer J?.24
- net Pin16R_Small: now also J?.25a; no longer J?.25
- net Pin1L_Small: now also J?.9a; no longer J?.9
- net Pin1R_Small: now also J?.40a; no longer J?.40
- net Pin2L_Small: now also J?.10a; no longer J?.10
- net Pin2R_Small: now also J?.39a; no longer J?.39
- net Pin3L_Small: now also J?.11a; no longer J?.11
- net Pin3R_Small: now also J?.38a; no longer J?.38
- net Pin4L_Small: now also J?.12a; no longer J?.12
- net Pin4R_Small: now also J?.37a; no longer J?.37
- net Pin5L_Small: now also J?.13a; no longer J?.13
- net Pin5R_Small: now also J?.36a; no longer J?.36
- net Pin6L_Small: now also J?.14a; no longer J?.14
- net Pin6R_Small: now also J?.35a; no longer J?.35
- net Pin7L_Small: now also J?.15a; no longer J?.15
- net Pin7R_Small: now also J?.34a; no longer J?.34
- net Pin8L_Small: now also J?.16a; no longer J?.16
- net Pin8R_Small: now also J?.33a; no longer J?.33
- net Pin9L_Small: now also J?.17a; no longer J?.17
- net Pin9R_Small: now also J?.32a; no longer J?.32
- net OKI - 3V3/+12V renamed +12V
- net Pin15L: no longer names the net of J?.15
- net Pin3R: no longer names the net of J?.46
- no-connect marks 1 -> 3
Other:
- moved on the sheet: C15, Conn1A, Conn1B, D1, D2, J2, J3, J?A, J?B, R8, R9
