File: NavBoard_Hardware/NavBoard_Hardware.kicad_pcb (KiCad board)
At the start: 4 copper layers, 210.6 x 29 mm, 61 parts, among them J1 8P8C_LED_Shielded, J10 Conn_01x16, J11 Conn_01x16, J12 Conn_01x24, J13 Conn_01x16, J14 Conn_01x16, J15 Conn_01x03, J16 Conn_01x03, J2 6 Pin Molex Micro-Fit, J3 Conn_01x24, J4 Conn_01x24, J6 Conn_01x24, J7 Conn_01x24, J8 Conn_01x06, J9 Conn_01x24, U1 BHI160B, U2 OKI-5V, U3 OKI-3V3, U4 ICM-20608-G, U5 Teensy4.1

Commit message: Annotated Schematic, assigned footprints, recovered accelerometer footprints
Parts:
- removed C1, C11, C13, C3, C4: 0.1uF, Capacitor_SMD:C_0603_1608Metric_Pad1.08x0.95mm_HandSolder
- removed C10, C7: 10uF, Capacitor_SMD:C_0603_1608Metric_Pad1.08x0.95mm_HandSolder
- removed C12: 2.2uF, Capacitor_SMD:C_0603_1608Metric_Pad1.08x0.95mm_HandSolder
- removed C14: 0.47uF, Capacitor_SMD:C_0603_1608Metric_Pad1.08x0.95mm_HandSolder
- removed C15: 10nF, Capacitor_SMD:C_0603_1608Metric_Pad1.08x0.95mm_HandSolder
- removed C2: 1uF, Capacitor_SMD:C_0603_1608Metric_Pad1.08x0.95mm_HandSolder
- removed C5: 0.47uF, Capacitor_THT:CP_Radial_D6.3mm_P2.50mm
- removed C6, C9: 22uF 50V, Capacitor_SMD:C_0603_1608Metric_Pad1.08x0.95mm_HandSolder
- removed C8: 0.1uF, Capacitor_THT:CP_Radial_D6.3mm_P2.50mm
- removed Conn1: AndersonPP, MRDT_Connectors:Anderson_2_Horizontal_Side_by_Side
- removed D1, D2: GREEN, LED_SMD:LED_0603_1608Metric_Pad1.05x0.95mm_HandSolder
- removed D3, D4, D5: BLUE, LED_SMD:LED_0603_1608Metric_Pad1.05x0.95mm_HandSolder
- removed J1: 8P8C_LED_Shielded, Connector_RJ:RJ45_Amphenol_RJHSE538X
- removed J10, J11, J13, J14: Conn_01x16, Connector_PinSocket_2.54mm:PinSocket_1x16_P2.54mm_Vertical
- removed J12, J9: Conn_01x24, Connector_PinHeader_2.54mm:PinHeader_1x24_P2.54mm_Vertical
- removed J15, J16: Conn_01x03, Connector_PinSocket_2.54mm:PinSocket_1x03_P2.54mm_Vertical
- removed J2: 6 Pin Molex Micro-Fit, Connector_Molex:Molex_Micro-Fit_3.0_43650-0600_1x06_P3.00mm_Horizontal
- removed J3, J4, J6, J7: Conn_01x24, Connector_PinSocket_2.54mm:PinSocket_1x24_P2.54mm_Vertical
- removed J8: Conn_01x06, Connector_PinSocket_2.00mm:PinSocket_2x03_P2.00mm_Vertical
- removed JP1: Solder Jumper, Jumper:SolderJumper-2_P1.3mm_Open_RoundedPad1.0x1.5mm
- removed R1: 43, Resistor_SMD:R_0603_1608Metric_Pad0.98x0.95mm_HandSolder
- removed R10, R11, R3, R4, R5, R6, R7, R8, R9: 4.7k, Resistor_SMD:R_0603_1608Metric_Pad0.98x0.95mm_HandSolder
- removed R12, R13, R14, R2: 100, Resistor_SMD:R_0603_1608Metric_Pad0.98x0.95mm_HandSolder
- removed TP1, TP2, TP3, TP4: TestPoint, TestPoint:TestPoint_Pad_D2.0mm
- removed U1: BHI160B, BHI160B:BHI160B
- removed U2: OKI-5V, MRDT_Devices:OKI_Horizontal
- removed U3: OKI-3V3, MRDT_Devices:OKI_Horizontal
- removed U4: ICM-20608-G, ICM-20608-G:ICM-20608-G
- removed U5 (x2): Teensy4.1, teensy:Teensy41
Routing:
- net GND: track 15.2 -> 0.00 mm
- net /Teensy Shield/Pin41: track 5.08 -> 0.00 mm
- net /Teensy Shield/Pin39: track 5.08 -> 0.00 mm
- net /Teensy Shield/Pin36: track 5.08 -> 0.00 mm
- net /Teensy Shield/Pin22: track 5.08 -> 0.00 mm
- net /Teensy Shield/Pin20: track 5.08 -> 0.00 mm
- net /Teensy Shield/Pin34: track 5.08 -> 0.00 mm
- net /Teensy Shield/Pin18: track 5.08 -> 0.00 mm
- net /Teensy Shield/Pin15: track 5.08 -> 0.00 mm
- net /Teensy Shield/Pin13: track 5.08 -> 0.00 mm
- net /Teensy Shield/Pin3V3_Right: track 5.08 -> 0.00 mm
- net +5V: track 5.08 -> 0.00 mm
- net /Teensy Shield/Pin38: track 5.08 -> 0.00 mm
- net /Teensy Shield/Pin35: track 5.08 -> 0.00 mm
- net /Teensy Shield/Pin33: track 5.08 -> 0.00 mm
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Other:
- outline, holes or cut-outs redrawn
