File: NavBoard_Hardware/teensy-shield.kicad_sch (KiCad schematic)
At the start: 4 parts

Commit message: Annotated Schematic, assigned footprints, recovered accelerometer footprints
Parts:
- removed J?: Teensy_Ethernet_2.54, symbol Connector_Generic:Conn_01x06
- gave numbers to parts that had none: 2
Changed lines of the file:
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@@
     (stroke (width 0) (type default) (color 0 0 0 0))
   )
-  (wire (pts (xy 218.44 43.18) (xy 218.44 50.165))
+  (wire (pts (xy 224.155 43.18) (xy 224.155 50.165))
     (stroke (width 0) (type default) (color 0 0 0 0))
   )
@@
     (stroke (width 0) (type default) (color 0 0 0 0))
   )
-  (wire (pts (xy 177.165 125.095) (xy 200.025 125.095))
-    (stroke (width 0) (type default) (color 0 0 0 0))
-  )
-  (wire (pts (xy 177.165 120.015) (xy 200.025 120.015))
-    (stroke (width 0) (type default) (color 0 0 0 0))
-  )
   (wire (pts (xy 66.675 50.165) (xy 66.675 52.705))
     (stroke (width 0) (type default) (color 0 0 0 0))
@@
     (stroke (width 0) (type default) (color 0 0 0 0))
   )
+  (wire (pts (xy 177.165 114.935) (xy 180.34 114.935))
+    (stroke (width 0) (type default) (color 0 0 0 0))
+  )
+  (wire (pts (xy 177.165 125.095) (xy 180.34 125.095))
+    (stroke (width 0) (type default) (color 0 0 0 0))
+  )
   (wire (pts (xy 90.805 50.165) (xy 121.285 50.165))
     (stroke (width 0) (type default) (color 0 0 0 0))
@@
     (stroke (width 0) (type default) (color 0 0 0 0))
   )
+  (wire (pts (xy 177.165 120.015) (xy 180.34 120.015))
+    (stroke (width 0) (type default) (color 0 0 0 0))
+  )
   (wire (pts (xy 77.47 60.325) (xy 80.645 60.325))
     (stroke (width 0) (type default) (color 0 0 0 0))
@@
     (stroke (width 0) (type default) (color 0 0 0 0))
   )
-  (wire (pts (xy 177.165 122.555) (xy 200.025 122.555))
+  (wire (pts (xy 177.165 127.635) (xy 180.34 127.635))
     (stroke (width 0) (type default) (color 0 0 0 0))
   )
@@
     (stroke (width 0) (type default) (color 0 0 0 0))
   )
-  (wire (pts (xy 198.12 129.54) (xy 198.12 117.475))
-    (stroke (width 0) (type default) (color 0 0 0 0))
-  )
   (wire (pts (xy 210.185 88.265) (xy 213.36 88.265))
     (stroke (width 0) (type default) (color 0 0 0 0))
@@
     (stroke (width 0) (type default) (color 0 0 0 0))
   )
-  (wire (pts (xy 210.185 50.165) (xy 218.44 50.165))
+  (wire (pts (xy 210.185 50.165) (xy 224.155 50.165))
     (stroke (width 0) (type default) (color 0 0 0 0))
   )
@@
     (stroke (width 0) (type default) (color 0 0 0 0))
   )
-  (wire (pts (xy 177.165 114.935) (xy 200.025 114.935))
-    (stroke (width 0) (type default) (color 0 0 0 0))
-  )
   (wire (pts (xy 210.185 57.785) (xy 213.36 57.785))
     (stroke (width 0) (type default) (color 0 0 0 0))
@@
     (stroke (width 0) (type default) (color 0 0 0 0))
   )
+  (wire (pts (xy 177.165 122.555) (xy 180.34 122.555))
+    (stroke (width 0) (type default) (color 0 0 0 0))
+  )
   (wire (pts (xy 210.185 106.045) (xy 213.36 106.045))
     (stroke (width 0) (type default) (color 0 0 0 0))
@@
     (stroke (width 0) (type default) (color 0 0 0 0))
   )
-  (wire (pts (xy 177.165 127.635) (xy 200.025 127.635))
-    (stroke (width 0) (type default) (color 0 0 0 0))
-  )
-  (wire (pts (xy 198.12 117.475) (xy 200.025 117.475))
-    (stroke (width 0) (type default) (color 0 0 0 0))
-  )
   (wire (pts (xy 210.185 95.885) (xy 213.36 95.885))
     (stroke (width 0) (type default) (color 0 0 0 0))
@@
   (symbol (lib_id "power:GND") (at 178.435 129.54 0) (unit 1)
     (in_bom yes) (on_board yes)
-    (property "Reference" "#PWR?" (id 0) (at 178.435 135.89 0)
+    (property "Reference" "#PWR037" (id 0) (at 178.435 135.89 0)
       (effects (font (size 1.27 1.27)) hide)
     )
@@
   (symbol (lib_id "power:GND") (at 120.65 130.175 0) (unit 1)
     (in_bom yes) (on_board yes)
-    (property "Reference" "#PWR?" (id 0) (at 120.65 136.525 0)
+    (property "Reference" "#PWR039" (id 0) (at 120.65 136.525 0)
       (effects (font (size 1.27 1.27)) hide)
     )
@@
   (symbol (lib_id "power:GND") (at 149.225 137.795 0) (unit 1)
     (in_bom yes) (on_board yes)
-    (property "Reference" "#PWR?" (id 0) (at 149.225 144.145 0)
+    (property "Reference" "#PWR040" (id 0) (at 149.225 144.145 0)
       (effects (font (size 1.27 1.27)) hide)
     )
@@
     (pin "1")
   )
-  (symbol (lib_id "Connector_Generic:Conn_01x06") (at 205.105 120.015 0) (unit 1)
-    (in_bom yes) (on_board yes) (fields_autoplaced)
-    (property "Reference" "J?" (id 0) (at 207.137 120.3765 0)
-      (effects (font (size 1.27 1.27)) (justify left))
-    )
-    (property "Value" "Teensy_Ethernet_2.54" (id 1) (at 207.137 123.1516 0)
-      (effects (font (size 1.27 1.27)) (justify left))
-    )
-    (property "Footprint" "" (id 2) (at 205.105 120.015 0)
-      (effects (font (size 1.27 1.27)) hide)
-    )
-    (property "Datasheet" "~" (id 3) (at 205.105 120.015 0)
-      (effects (font (size 1.27 1.27)) hide)
-    )
-    (pin "1")
-    (pin "2")
-    (pin "3")
-    (pin "4")
-    (pin "5")
-    (pin "6")
-  )
-  (symbol (lib_id "power:+5V") (at 218.44 43.18 0) (unit 1)
-    (in_bom yes) (on_board yes)
-    (property "Reference" "#PWR?" (id 0) (at 218.44 46.99 0)
-      (effects (font (size 1.27 1.27)) hide)
-    )
-    (property "Value" "+5V" (id 1) (at 218.821 38.7858 0))
-    (property "Footprint" "" (id 2) (at 218.44 43.18 0)
-      (effects (font (size 1.27 1.27)) hide)
-    )
-    (property "Datasheet" "" (id 3) (at 218.44 43.18 0)
+  (symbol (lib_id "power:+5V") (at 224.155 43.18 0) (unit 1)
+    (in_bom yes) (on_board yes)
+    (property "Reference" "#PWR033" (id 0) (at 224.155 46.99 0)
+      (effects (font (size 1.27 1.27)) hide)
+    )
+    (property "Value" "+5V" (id 1) (at 224.536 38.7858 0))
+    (property "Footprint" "" (id 2) (at 224.155 43.18 0)
+      (effects (font (size 1.27 1.27)) hide)
+    )
+    (property "Datasheet" "" (id 3) (at 224.155 43.18 0)
       (effects (font (size 1.27 1.27)) hide)
     )
@@
   (symbol (lib_id "power:GND") (at 66.675 52.705 0) (unit 1)
     (in_bom yes) (on_board yes)
-    (property "Reference" "#PWR?" (id 0) (at 66.675 59.055 0)
+    (property "Reference" "#PWR034" (id 0) (at 66.675 59.055 0)
       (effects (font (size 1.27 1.27)) hide)
     )
@@
   (symbol (lib_id "Nav_Board:Teensy-2.54mm_Adapter") (at 205.105 48.895 0) (unit 2)
     (in_bom yes) (on_board yes)
-    (property "Reference" "J?" (id 0) (at 205.105 44.9285 0))
+    (property "Reference" "J5" (id 0) (at 205.105 44.9285 0))
     (property "Value" "Teensy-2.54mm_Adapter" (id 1) (at 205.105 47.7036 0))
     (property "Footprint" "Nav_Board:Teensy-2.54mm_Adapter" (id 2) (at 205.105 42.545 0)
@@
       (effects (font (size 1.27 1.27)) hide)
     )
-    (property "Inner Type" "2.54mm Sockets" (id 4) (at 194.945 111.76 0))
-    (property "Outer Type" "2.54mm Pins" (id 5) (at 213.995 111.76 0))
+    (property "Inner Type" "2.54mm Sockets" (id 4) (at 193.04 45.085 0))
+    (property "Outer Type" "2.54mm Pins" (id 5) (at 215.9 45.085 0))
     (pin "25")
     (pin "25")
@@
   (symbol (lib_id "Nav_Board:Teensy-2.54mm_Adapter") (at 85.725 48.895 0) (unit 1)
     (in_bom yes) (on_board yes)
-    (property "Reference" "J?" (id 0) (at 85.725 44.9285 0))
+    (property "Reference" "J5" (id 0) (at 85.725 44.9285 0))
     (property "Value" "Teensy-2.54mm_Adapter" (id 1) (at 85.725 47.7036 0))
     (property "Footprint" "Nav_Board:Teensy-2.54mm_Adapter" (id 2) (at 85.725 42.545 0)
@@
   (symbol (lib_id "teensy:Teensy4.1") (at 149.225 104.775 0) (unit 1)
     (in_bom yes) (on_board yes)
-    (property "Reference" "U?" (id 0) (at 149.225 39.9755 0))
+    (property "Reference" "U5" (id 0) (at 149.225 39.9755 0))
     (property "Value" "Teensy4.1" (id 1) (at 149.225 42.7506 0))
     (property "Footprint" "teensy:Teensy41" (id 2) (at 139.065 94.615 0)
@@
     (pin "4")
   )
-  (symbol (lib_id "power:GND") (at 198.12 129.54 0) (unit 1)
-    (in_bom yes) (on_board yes)
-    (property "Reference" "#PWR?" (id 0) (at 198.12 135.89 0)
-      (effects (font (size 1.27 1.27)) hide)
-    )
-    (property "Value" "GND" (id 1) (at 198.247 133.9342 0))
-    (property "Footprint" "" (id 2) (at 198.12 129.54 0)
-      (effects (font (size 1.27 1.27)) hide)
-    )
-    (property "Datasheet" "" (id 3) (at 198.12 129.54 0)
-      (effects (font (size 1.27 1.27)) hide)
-    )
-    (pin "1")
-  )
   (symbol (lib_id "power:GND") (at 229.87 86.995 0) (unit 1)
     (in_bom yes) (on_board yes)
-    (property "Reference" "#PWR?" (id 0) (at 229.87 93.345 0)
+    (property "Reference" "#PWR036" (id 0) (at 229.87 93.345 0)
       (effects (font (size 1.27 1.27)) hide)
     )
@@
   (symbol (lib_id "power:GND") (at 229.87 53.975 0) (unit 1)
     (in_bom yes) (on_board yes)
-    (property "Reference" "#PWR?" (id 0) (at 229.87 60.325 0)
-      (effects (font (size 1.27 1.27)) hide)
-    )
+    (property "Reference" "#PWR035" (id 0) (at 229.87 60.325 0)
+      (effects (font (size 1.27 1.27)) hide)
+    )

Commit message: Corrected pinout of RJ45 symbol, squashed some bugs
Parts:
- renumbered J5 to J4
Changed lines of the file:
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@@
   (symbol (lib_id "power:GND") (at 120.65 130.175 0) (unit 1)
     (in_bom yes) (on_board yes)
-    (property "Reference" "#PWR039" (id 0) (at 120.65 136.525 0)
+    (property "Reference" "#PWR038" (id 0) (at 120.65 136.525 0)
       (effects (font (size 1.27 1.27)) hide)
     )
@@
   (symbol (lib_id "power:GND") (at 149.225 137.795 0) (unit 1)
     (in_bom yes) (on_board yes)
-    (property "Reference" "#PWR040" (id 0) (at 149.225 144.145 0)
+    (property "Reference" "#PWR039" (id 0) (at 149.225 144.145 0)
       (effects (font (size 1.27 1.27)) hide)
     )
@@
   (symbol (lib_id "Nav_Board:Teensy-2.54mm_Adapter") (at 205.105 48.895 0) (unit 2)
     (in_bom yes) (on_board yes)
-    (property "Reference" "J5" (id 0) (at 205.105 44.9285 0))
+    (property "Reference" "J4" (id 0) (at 205.105 44.9285 0))
     (property "Value" "Teensy-2.54mm_Adapter" (id 1) (at 205.105 47.7036 0))
     (property "Footprint" "Nav_Board:Teensy-2.54mm_Adapter" (id 2) (at 205.105 42.545 0)
@@
   (symbol (lib_id "Nav_Board:Teensy-2.54mm_Adapter") (at 85.725 48.895 0) (unit 1)
     (in_bom yes) (on_board yes)
-    (property "Reference" "J5" (id 0) (at 85.725 44.9285 0))
+    (property "Reference" "J4" (id 0) (at 85.725 44.9285 0))
     (property "Value" "Teensy-2.54mm_Adapter" (id 1) (at 85.725 47.7036 0))
     (property "Footprint" "Nav_Board:Teensy-2.54mm_Adapter" (id 2) (at 85.725 42.545 0)

Commit message: Resized Ethernet to 2.54mm
Parts:
- added J?: Teensy Ethernet, Connector_PinSocket_2.00mm:PinSocket_2x03_P2.00mm_Vertical, symbol Connector_Generic:Conn_01x06
Connections:
- net ETHERNET_LED: now also J?.5 (Pin_5)
- net ETHERNET_RX+: now also J?.6 (Pin_6)
- net ETHERNET_RX-: now also J?.1 (Pin_1)
- net ETHERNET_TX+: now also J?.3 (Pin_3)
- net ETHERNET_TX-: now also J?.4 (Pin_4)
- net GND: now also J?.2 (Pin_2)
Changed lines of the file:
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@@
     (stroke (width 0) (type default) (color 0 0 0 0))
   )
-  (wire (pts (xy 177.165 114.935) (xy 180.34 114.935))
-    (stroke (width 0) (type default) (color 0 0 0 0))
-  )
-  (wire (pts (xy 177.165 125.095) (xy 180.34 125.095))
+  (wire (pts (xy 177.165 114.935) (xy 198.755 114.935))
+    (stroke (width 0) (type default) (color 0 0 0 0))
+  )
+  (wire (pts (xy 177.165 125.095) (xy 198.755 125.095))
     (stroke (width 0) (type default) (color 0 0 0 0))
   )
@@
     (stroke (width 0) (type default) (color 0 0 0 0))
   )
+  (wire (pts (xy 196.85 117.475) (xy 198.755 117.475))
+    (stroke (width 0) (type default) (color 0 0 0 0))
+  )
   (wire (pts (xy 90.805 100.965) (xy 121.285 100.965))
     (stroke (width 0) (type default) (color 0 0 0 0))
@@
     (stroke (width 0) (type default) (color 0 0 0 0))
   )
-  (wire (pts (xy 177.165 120.015) (xy 180.34 120.015))
+  (wire (pts (xy 177.165 120.015) (xy 198.755 120.015))
     (stroke (width 0) (type default) (color 0 0 0 0))
   )
@@
     (stroke (width 0) (type default) (color 0 0 0 0))
   )
-  (wire (pts (xy 177.165 127.635) (xy 180.34 127.635))
+  (wire (pts (xy 177.165 127.635) (xy 198.755 127.635))
     (stroke (width 0) (type default) (color 0 0 0 0))
   )
@@
     (stroke (width 0) (type default) (color 0 0 0 0))
   )
+  (wire (pts (xy 196.85 129.54) (xy 196.85 117.475))
+    (stroke (width 0) (type default) (color 0 0 0 0))
+  )
   (wire (pts (xy 177.165 70.485) (xy 200.025 70.485))
     (stroke (width 0) (type default) (color 0 0 0 0))
@@
     (stroke (width 0) (type default) (color 0 0 0 0))
   )
-  (wire (pts (xy 177.165 122.555) (xy 180.34 122.555))
+  (wire (pts (xy 177.165 122.555) (xy 198.755 122.555))
     (stroke (width 0) (type default) (color 0 0 0 0))
   )
@@
   (hierarchical_label "Pin0" (shape input) (at 77.47 52.705 180)
     (effects (font (size 1.27 1.27)) (justify right))
+  )
+  (symbol (lib_id "power:GND") (at 196.85 129.54 0) (unit 1)
+    (in_bom yes) (on_board yes)
+    (property "Reference" "#PWR?" (id 0) (at 196.85 135.89 0)
+      (effects (font (size 1.27 1.27)) hide)
+    )
+    (property "Value" "GND" (id 1) (at 196.977 133.9342 0))
+    (property "Footprint" "" (id 2) (at 196.85 129.54 0)
+      (effects (font (size 1.27 1.27)) hide)
+    )
+    (property "Datasheet" "" (id 3) (at 196.85 129.54 0)
+      (effects (font (size 1.27 1.27)) hide)
+    )
+    (pin "1")
   )
   (symbol (lib_id "power:GND") (at 178.435 129.54 0) (unit 1)
@@
     (pin "1")
   )
+  (symbol (lib_id "Connector_Generic:Conn_01x06") (at 203.835 120.015 0) (unit 1)
+    (in_bom yes) (on_board yes)
+    (property "Reference" "J?" (id 0) (at 206.375 114.3 0)
+      (effects (font (size 1.27 1.27)) (justify left))
+    )
+    (property "Value" "Teensy Ethernet" (id 1) (at 206.375 117.475 0)
+      (effects (font (size 1.27 1.27)) (justify left))
+    )
+    (property "Footprint" "Connector_PinSocket_2.00mm:PinSocket_2x03_P2.00mm_Vertical" (id 2) (at 203.835 120.015 0)
+      (effects (font (size 1.27 1.27)) hide)
+    )
+    (property "Datasheet" "~" (id 3) (at 203.835 120.015 0)
+      (effects (font (size 1.27 1.27)) hide)
+    )
+    (property "Field4" " 2.54mm Pins" (id 4) (at 209.55 131.445 0))
+    (pin "1")
+    (pin "2")
+    (pin "3")
+    (pin "4")
+    (pin "5")
+    (pin "6")
+  )
   (symbol (lib_id "power:+5V") (at 224.155 43.18 0) (unit 1)

Commit message: Placed and aligned all headers
Parts:
- J5: renamed from J?; footprint Connector_PinSocket_2.00mm:PinSocket_2x03_P2.00mm_Vertical -> Connector_PinHeader_2.54mm:PinHeader_2x03_P2.54mm_Vertical
Changed lines of the file:
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@@
   (symbol (lib_id "power:GND") (at 196.85 129.54 0) (unit 1)
     (in_bom yes) (on_board yes)
-    (property "Reference" "#PWR?" (id 0) (at 196.85 135.89 0)
+    (property "Reference" "#PWR038" (id 0) (at 196.85 135.89 0)
       (effects (font (size 1.27 1.27)) hide)
     )
@@
   (symbol (lib_id "power:GND") (at 120.65 130.175 0) (unit 1)
     (in_bom yes) (on_board yes)
-    (property "Reference" "#PWR038" (id 0) (at 120.65 136.525 0)
+    (property "Reference" "#PWR039" (id 0) (at 120.65 136.525 0)
       (effects (font (size 1.27 1.27)) hide)
     )
@@
   (symbol (lib_id "power:GND") (at 149.225 137.795 0) (unit 1)
     (in_bom yes) (on_board yes)
-    (property "Reference" "#PWR039" (id 0) (at 149.225 144.145 0)
+    (property "Reference" "#PWR040" (id 0) (at 149.225 144.145 0)
       (effects (font (size 1.27 1.27)) hide)
     )
@@
   (symbol (lib_id "Connector_Generic:Conn_01x06") (at 203.835 120.015 0) (unit 1)
     (in_bom yes) (on_board yes)
-    (property "Reference" "J?" (id 0) (at 206.375 114.3 0)
+    (property "Reference" "J5" (id 0) (at 206.375 114.3 0)
       (effects (font (size 1.27 1.27)) (justify left))
     )
@@
       (effects (font (size 1.27 1.27)) (justify left))
     )
-    (property "Footprint" "Connector_PinSocket_2.00mm:PinSocket_2x03_P2.00mm_Vertical" (id 2) (at 203.835 120.015 0)
+    (property "Footprint" "Connector_PinHeader_2.54mm:PinHeader_2x03_P2.54mm_Vertical" (id 2) (at 203.835 120.015 0)
       (effects (font (size 1.27 1.27)) hide)
     )

Commit message: Placed OKI SMD components, aligned ethernet pins
Connections:
- net Pin32 is gone; now on net GND: J4.24
- net Pin33 is gone; now on net GND: J4.25
- net ETHERNET_LED: now also J5.6 (Pin_6); no longer J5.5 (Pin_5)
- net ETHERNET_RX+: now also J5.3 (Pin_3); no longer J5.6 (Pin_6)
- net ETHERNET_RX-: now also J5.5 (Pin_5); no longer J5.1 (Pin_1)
- net ETHERNET_TX+: now also J5.2 (Pin_2); no longer J5.3 (Pin_3)
- net ETHERNET_TX-: now also J5.1 (Pin_1); no longer J5.4 (Pin_4)
- net GND: now also J5.4 (Pin_4); no longer J5.2 (Pin_2)
Other:
- moved on the sheet: J5
