File: NavBoard_Hardware/top_board.kicad_sch (KiCad schematic)
At the start: 11 parts, among them J4 01x03, J5 6 Pin Molex Micro-Fit, J6 01x03

Commit message: Annotated Schematic, assigned footprints, recovered accelerometer footprints
Parts:
- J7: renamed from J4; footprint (none) -> Connector_PinSocket_2.54mm:PinSocket_1x03_P2.54mm_Vertical; Field4 2.54 mm -> 2.54 mm Socket
- J8: renamed from J6; footprint (none) -> Connector_PinSocket_2.54mm:PinSocket_1x03_P2.54mm_Vertical; Field4 2.54 mm -> 2.54 mm Socket
- gave numbers to parts that had none: 4
- renumbered J5 to J10, JP1 to JP2
Changed lines of the file:
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@@
   (symbol (lib_id "Device:R_US") (at 100.33 132.715 0) (unit 1)
     (in_bom yes) (on_board yes)
-    (property "Reference" "R?" (id 0) (at 94.615 131.445 0)
+    (property "Reference" "R12" (id 0) (at 94.615 131.445 0)
       (effects (font (size 1.27 1.27)) (justify left))
     )
@@
   (symbol (lib_id "power:GND") (at 100.33 137.795 0) (unit 1)
     (in_bom yes) (on_board yes)
-    (property "Reference" "#PWR?" (id 0) (at 100.33 144.145 0)
+    (property "Reference" "#PWR047" (id 0) (at 100.33 144.145 0)
       (effects (font (size 1.27 1.27)) hide)
     )
@@
   (symbol (lib_id "Connector_Generic:Conn_01x03") (at 107.95 59.055 0) (mirror y) (unit 1)
     (in_bom yes) (on_board yes)
-    (property "Reference" "J4" (id 0) (at 109.22 50.8 0)
+    (property "Reference" "J7" (id 0) (at 109.22 50.8 0)
       (effects (font (size 1.27 1.27)) (justify left))
     )
@@
       (effects (font (size 1.27 1.27)) (justify left))
     )
-    (property "Footprint" "" (id 2) (at 107.95 59.055 0)
+    (property "Footprint" "Connector_PinSocket_2.54mm:PinSocket_1x03_P2.54mm_Vertical" (id 2) (at 107.95 59.055 0)
       (effects (font (size 1.27 1.27)) hide)
     )
@@
       (effects (font (size 1.27 1.27)) hide)
     )
-    (property "Field4" "2.54 mm" (id 4) (at 107.95 64.77 0))
+    (property "Field4" "2.54 mm Socket" (id 4) (at 114.3 64.77 0))
     (pin "1")
     (pin "2")
@@
   (symbol (lib_id "power:GND") (at 139.7 109.22 0) (mirror y) (unit 1)
     (in_bom yes) (on_board yes)
-    (property "Reference" "#PWR037" (id 0) (at 139.7 115.57 0)
+    (property "Reference" "#PWR046" (id 0) (at 139.7 115.57 0)
       (effects (font (size 1.27 1.27)) hide)
     )
@@
   (symbol (lib_id "power:GND") (at 191.135 74.295 0) (unit 1)
     (in_bom yes) (on_board yes)
-    (property "Reference" "#PWR031" (id 0) (at 191.135 80.645 0)
+    (property "Reference" "#PWR043" (id 0) (at 191.135 80.645 0)
       (effects (font (size 1.27 1.27)) hide)
     )
@@
   (symbol (lib_id "Jumper:SolderJumper_2_Open") (at 235.585 58.42 90) (unit 1)
     (in_bom yes) (on_board yes)
-    (property "Reference" "JP1" (id 0) (at 238.76 57.5499 90)
+    (property "Reference" "JP2" (id 0) (at 238.76 57.5499 90)
       (effects (font (size 1.27 1.27)) (justify right))
     )
@@
   (symbol (lib_id "Nav_Board:Conn_02x16_Separate") (at 99.695 75.565 0) (unit 1)
     (in_bom yes) (on_board yes)
-    (property "Reference" "J?" (id 0) (at 97.79 97.79 0)
+    (property "Reference" "J9" (id 0) (at 97.79 97.79 0)
       (effects (font (size 1.27 1.27)) (justify left))
     )
@@
   (symbol (lib_id "power:GND") (at 195.58 74.295 0) (unit 1)
     (in_bom yes) (on_board yes)
-    (property "Reference" "#PWR032" (id 0) (at 195.58 80.645 0)
+    (property "Reference" "#PWR044" (id 0) (at 195.58 80.645 0)
       (effects (font (size 1.27 1.27)) hide)
     )
@@
   (symbol (lib_id "power:GND") (at 104.775 137.795 0) (unit 1)
     (in_bom yes) (on_board yes)
-    (property "Reference" "#PWR?" (id 0) (at 104.775 144.145 0)
+    (property "Reference" "#PWR048" (id 0) (at 104.775 144.145 0)
       (effects (font (size 1.27 1.27)) hide)
     )
@@
   (symbol (lib_id "Connector_Generic:Conn_01x03") (at 149.225 59.055 0) (unit 1)
     (in_bom yes) (on_board yes)
-    (property "Reference" "J6" (id 0) (at 149.225 50.8 0))
+    (property "Reference" "J8" (id 0) (at 149.225 50.8 0))
     (property "Value" "01x03" (id 1) (at 149.225 53.34 0))
-    (property "Footprint" "" (id 2) (at 149.225 59.055 0)
+    (property "Footprint" "Connector_PinSocket_2.54mm:PinSocket_1x03_P2.54mm_Vertical" (id 2) (at 149.225 59.055 0)
       (effects (font (size 1.27 1.27)) hide)
     )
@@
       (effects (font (size 1.27 1.27)) hide)
     )
-    (property "Field4" "2.54 mm" (id 4) (at 149.225 64.77 0))
+    (property "Field4" "2.54 mm Socket" (id 4) (at 142.875 64.77 0))
     (pin "1")
     (pin "2")
@@
   (symbol (lib_id "Connector_Generic:Conn_01x06") (at 134.62 99.695 270) (mirror x) (unit 1)
     (in_bom yes) (on_board yes)
-    (property "Reference" "J5" (id 0) (at 133.985 92.71 90)
+    (property "Reference" "J10" (id 0) (at 133.985 92.71 90)
       (effects (font (size 1.27 1.27) bold))
     )
@@
   (symbol (lib_id "power:GND") (at 235.585 62.23 0) (unit 1)
     (in_bom yes) (on_board yes)
-    (property "Reference" "#PWR041" (id 0) (at 235.585 68.58 0)
+    (property "Reference" "#PWR042" (id 0) (at 235.585 68.58 0)
       (effects (font (size 1.27 1.27)) hide)
     )
@@
   (symbol (lib_id "power:+3V3") (at 235.585 46.355 0) (unit 1)
     (in_bom yes) (on_board yes)
-    (property "Reference" "#PWR?" (id 0) (at 235.585 50.165 0)
+    (property "Reference" "#PWR041" (id 0) (at 235.585 50.165 0)
       (effects (font (size 1.27 1.27)) hide)
     )
@@
   (symbol (lib_id "Nav_Board:Conn_02x16_Separate") (at 158.115 75.565 0) (mirror y) (unit 2)
     (in_bom yes) (on_board yes)
-    (property "Reference" "J?" (id 0) (at 158.115 97.79 0))
+    (property "Reference" "J9" (id 0) (at 158.115 97.79 0))
     (property "Value" "Conn_02x16_Separate" (id 1) (at 168.91 101.6 0)
       (effects (font (size 1.27 1.27)) (justify left) hide)
@@
   (symbol (lib_id "Device:R_US") (at 104.775 132.715 0) (unit 1)
     (in_bom yes) (on_board yes)
-    (property "Reference" "R?" (id 0) (at 106.68 131.445 0)
+    (property "Reference" "R13" (id 0) (at 106.68 131.445 0)
       (effects (font (size 1.27 1.27)) (justify left))
     )
@@
   (symbol (lib_id "Jumper:SolderJumper_2_Open") (at 235.585 50.165 270) (unit 1)
     (in_bom yes) (on_board yes)
-    (property "Reference" "JP?" (id 0) (at 241.935 47.625 90)
+    (property "Reference" "JP1" (id 0) (at 241.935 47.625 90)
       (effects (font (size 1.27 1.27)) (justify right))
     )
@@
   (symbol (lib_id "power:+5V") (at 144.145 100.965 0) (unit 1)
     (in_bom yes) (on_board yes)
-    (property "Reference" "#PWR036" (id 0) (at 144.145 104.775 0)
-      (effects (font (size 1.27 1.27)) hide)
-    )
+    (property "Reference" "#PWR045" (id 0) (at 144.145 104.775 0)
+      (effects (font (size 1.27 1.27)) hide)
+    )

Commit message: Corrected pinout of RJ45 symbol, squashed some bugs
Parts:
- J7: renamed from J9; Field4 2.54 mm -> 2.54 mm Pins
- renumbered J7 to J5, J8 to J6, J10 to J8
Changed lines of the file:
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@@
   (symbol (lib_id "power:GND") (at 100.33 137.795 0) (unit 1)
     (in_bom yes) (on_board yes)
-    (property "Reference" "#PWR047" (id 0) (at 100.33 144.145 0)
+    (property "Reference" "#PWR046" (id 0) (at 100.33 144.145 0)
       (effects (font (size 1.27 1.27)) hide)
     )
@@
   (symbol (lib_id "Connector_Generic:Conn_01x03") (at 107.95 59.055 0) (mirror y) (unit 1)
     (in_bom yes) (on_board yes)
-    (property "Reference" "J7" (id 0) (at 109.22 50.8 0)
+    (property "Reference" "J5" (id 0) (at 109.22 50.8 0)
       (effects (font (size 1.27 1.27)) (justify left))
     )
@@
   (symbol (lib_id "power:GND") (at 139.7 109.22 0) (mirror y) (unit 1)
     (in_bom yes) (on_board yes)
-    (property "Reference" "#PWR046" (id 0) (at 139.7 115.57 0)
+    (property "Reference" "#PWR045" (id 0) (at 139.7 115.57 0)
       (effects (font (size 1.27 1.27)) hide)
     )
@@
   (symbol (lib_id "power:GND") (at 191.135 74.295 0) (unit 1)
     (in_bom yes) (on_board yes)
-    (property "Reference" "#PWR043" (id 0) (at 191.135 80.645 0)
+    (property "Reference" "#PWR042" (id 0) (at 191.135 80.645 0)
       (effects (font (size 1.27 1.27)) hide)
     )
@@
   (symbol (lib_id "Nav_Board:Conn_02x16_Separate") (at 99.695 75.565 0) (unit 1)
     (in_bom yes) (on_board yes)
-    (property "Reference" "J9" (id 0) (at 97.79 97.79 0)
+    (property "Reference" "J7" (id 0) (at 97.79 97.79 0)
       (effects (font (size 1.27 1.27)) (justify left))
     )
@@
       (effects (font (size 1.27 1.27)) hide)
     )
-    (property "Field4" "2.54 mm" (id 4) (at 99.695 100.33 0))
+    (property "Field4" "2.54 mm Pins" (id 4) (at 99.695 100.33 0))
     (pin "1")
     (pin "10")
@@
   (symbol (lib_id "power:GND") (at 195.58 74.295 0) (unit 1)
     (in_bom yes) (on_board yes)
-    (property "Reference" "#PWR044" (id 0) (at 195.58 80.645 0)
+    (property "Reference" "#PWR043" (id 0) (at 195.58 80.645 0)
       (effects (font (size 1.27 1.27)) hide)
     )
@@
   (symbol (lib_id "power:GND") (at 104.775 137.795 0) (unit 1)
     (in_bom yes) (on_board yes)
-    (property "Reference" "#PWR048" (id 0) (at 104.775 144.145 0)
+    (property "Reference" "#PWR047" (id 0) (at 104.775 144.145 0)
       (effects (font (size 1.27 1.27)) hide)
     )
@@
   (symbol (lib_id "Connector_Generic:Conn_01x03") (at 149.225 59.055 0) (unit 1)
     (in_bom yes) (on_board yes)
-    (property "Reference" "J8" (id 0) (at 149.225 50.8 0))
+    (property "Reference" "J6" (id 0) (at 149.225 50.8 0))
     (property "Value" "01x03" (id 1) (at 149.225 53.34 0))
     (property "Footprint" "Connector_PinSocket_2.54mm:PinSocket_1x03_P2.54mm_Vertical" (id 2) (at 149.225 59.055 0)
@@
   (symbol (lib_id "Connector_Generic:Conn_01x06") (at 134.62 99.695 270) (mirror x) (unit 1)
     (in_bom yes) (on_board yes)
-    (property "Reference" "J10" (id 0) (at 133.985 92.71 90)
+    (property "Reference" "J8" (id 0) (at 133.985 92.71 90)
       (effects (font (size 1.27 1.27) bold))
     )
@@
   (symbol (lib_id "power:GND") (at 235.585 62.23 0) (unit 1)
     (in_bom yes) (on_board yes)
-    (property "Reference" "#PWR042" (id 0) (at 235.585 68.58 0)
+    (property "Reference" "#PWR041" (id 0) (at 235.585 68.58 0)
       (effects (font (size 1.27 1.27)) hide)
     )
@@
   (symbol (lib_id "power:+3V3") (at 235.585 46.355 0) (unit 1)
     (in_bom yes) (on_board yes)
-    (property "Reference" "#PWR041" (id 0) (at 235.585 50.165 0)
+    (property "Reference" "#PWR040" (id 0) (at 235.585 50.165 0)
       (effects (font (size 1.27 1.27)) hide)
     )
@@
   (symbol (lib_id "Nav_Board:Conn_02x16_Separate") (at 158.115 75.565 0) (mirror y) (unit 2)
     (in_bom yes) (on_board yes)
-    (property "Reference" "J9" (id 0) (at 158.115 97.79 0))
+    (property "Reference" "J7" (id 0) (at 158.115 97.79 0))
     (property "Value" "Conn_02x16_Separate" (id 1) (at 168.91 101.6 0)
       (effects (font (size 1.27 1.27)) (justify left) hide)
@@
       (effects (font (size 1.27 1.27)) hide)
     )
-    (property "Field4" "2.54 mm" (id 4) (at 158.115 100.33 0))
+    (property "Field4" "2.54 mm Pins" (id 4) (at 158.115 100.33 0))
     (pin "17")
     (pin "18")
@@
   (symbol (lib_id "power:+5V") (at 144.145 100.965 0) (unit 1)
     (in_bom yes) (on_board yes)
-    (property "Reference" "#PWR045" (id 0) (at 144.145 104.775 0)
-      (effects (font (size 1.27 1.27)) hide)
-    )
+    (property "Reference" "#PWR044" (id 0) (at 144.145 104.775 0)
+      (effects (font (size 1.27 1.27)) hide)
+    )

Commit message: Placed and aligned all headers
Parts:
- renumbered J5 to J6, J6 to J7, J7 to J8, J8 to J9
Changed lines of the file:
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@@
   (symbol (lib_id "power:GND") (at 100.33 137.795 0) (unit 1)
     (in_bom yes) (on_board yes)
-    (property "Reference" "#PWR046" (id 0) (at 100.33 144.145 0)
+    (property "Reference" "#PWR047" (id 0) (at 100.33 144.145 0)
       (effects (font (size 1.27 1.27)) hide)
     )
@@
   (symbol (lib_id "Connector_Generic:Conn_01x03") (at 107.95 59.055 0) (mirror y) (unit 1)
     (in_bom yes) (on_board yes)
-    (property "Reference" "J5" (id 0) (at 109.22 50.8 0)
+    (property "Reference" "J6" (id 0) (at 109.22 50.8 0)
       (effects (font (size 1.27 1.27)) (justify left))
     )
@@
   (symbol (lib_id "power:GND") (at 139.7 109.22 0) (mirror y) (unit 1)
     (in_bom yes) (on_board yes)
-    (property "Reference" "#PWR045" (id 0) (at 139.7 115.57 0)
+    (property "Reference" "#PWR046" (id 0) (at 139.7 115.57 0)
       (effects (font (size 1.27 1.27)) hide)
     )
@@
   (symbol (lib_id "power:GND") (at 191.135 74.295 0) (unit 1)
     (in_bom yes) (on_board yes)
-    (property "Reference" "#PWR042" (id 0) (at 191.135 80.645 0)
+    (property "Reference" "#PWR043" (id 0) (at 191.135 80.645 0)
       (effects (font (size 1.27 1.27)) hide)
     )
@@
   (symbol (lib_id "Nav_Board:Conn_02x16_Separate") (at 99.695 75.565 0) (unit 1)
     (in_bom yes) (on_board yes)
-    (property "Reference" "J7" (id 0) (at 97.79 97.79 0)
+    (property "Reference" "J8" (id 0) (at 97.79 97.79 0)
       (effects (font (size 1.27 1.27)) (justify left))
     )
@@
   (symbol (lib_id "power:GND") (at 195.58 74.295 0) (unit 1)
     (in_bom yes) (on_board yes)
-    (property "Reference" "#PWR043" (id 0) (at 195.58 80.645 0)
+    (property "Reference" "#PWR044" (id 0) (at 195.58 80.645 0)
       (effects (font (size 1.27 1.27)) hide)
     )
@@
   (symbol (lib_id "power:GND") (at 104.775 137.795 0) (unit 1)
     (in_bom yes) (on_board yes)
-    (property "Reference" "#PWR047" (id 0) (at 104.775 144.145 0)
+    (property "Reference" "#PWR048" (id 0) (at 104.775 144.145 0)
       (effects (font (size 1.27 1.27)) hide)
     )
@@
   (symbol (lib_id "Connector_Generic:Conn_01x03") (at 149.225 59.055 0) (unit 1)
     (in_bom yes) (on_board yes)
-    (property "Reference" "J6" (id 0) (at 149.225 50.8 0))
+    (property "Reference" "J7" (id 0) (at 149.225 50.8 0))
     (property "Value" "01x03" (id 1) (at 149.225 53.34 0))
     (property "Footprint" "Connector_PinSocket_2.54mm:PinSocket_1x03_P2.54mm_Vertical" (id 2) (at 149.225 59.055 0)
@@
   (symbol (lib_id "Connector_Generic:Conn_01x06") (at 134.62 99.695 270) (mirror x) (unit 1)
     (in_bom yes) (on_board yes)
-    (property "Reference" "J8" (id 0) (at 133.985 92.71 90)
+    (property "Reference" "J9" (id 0) (at 133.985 92.71 90)
       (effects (font (size 1.27 1.27) bold))
     )
@@
   (symbol (lib_id "power:GND") (at 235.585 62.23 0) (unit 1)
     (in_bom yes) (on_board yes)
-    (property "Reference" "#PWR041" (id 0) (at 235.585 68.58 0)
+    (property "Reference" "#PWR042" (id 0) (at 235.585 68.58 0)
       (effects (font (size 1.27 1.27)) hide)
     )
@@
   (symbol (lib_id "power:+3V3") (at 235.585 46.355 0) (unit 1)
     (in_bom yes) (on_board yes)
-    (property "Reference" "#PWR040" (id 0) (at 235.585 50.165 0)
+    (property "Reference" "#PWR041" (id 0) (at 235.585 50.165 0)
       (effects (font (size 1.27 1.27)) hide)
     )
@@
   (symbol (lib_id "Nav_Board:Conn_02x16_Separate") (at 158.115 75.565 0) (mirror y) (unit 2)
     (in_bom yes) (on_board yes)
-    (property "Reference" "J7" (id 0) (at 158.115 97.79 0))
+    (property "Reference" "J8" (id 0) (at 158.115 97.79 0))
     (property "Value" "Conn_02x16_Separate" (id 1) (at 168.91 101.6 0)
       (effects (font (size 1.27 1.27)) (justify left) hide)
@@
   (symbol (lib_id "power:+5V") (at 144.145 100.965 0) (unit 1)
     (in_bom yes) (on_board yes)
-    (property "Reference" "#PWR044" (id 0) (at 144.145 104.775 0)
-      (effects (font (size 1.27 1.27)) hide)
-    )
+    (property "Reference" "#PWR045" (id 0) (at 144.145 104.775 0)
+      (effects (font (size 1.27 1.27)) hide)
+    )

Commit message: Placed OKI SMD components, aligned ethernet pins
Connections:
- net Pin16L is gone; now on net GND: J8.16
- net Pin16R is gone; now on net GND: J8.32
Changed lines of the file:
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@@
+    (stroke (width 0) (type default) (color 0 0 0 0))
+  )
+  (wire (pts (xy 168.275 94.615) (xy 168.275 97.155))
     (stroke (width 0) (type default) (color 0 0 0 0))
   )
@@
     (stroke (width 0) (type default) (color 0 0 0 0))
   )
+  (wire (pts (xy 89.535 94.615) (xy 94.615 94.615))
+    (stroke (width 0) (type default) (color 0 0 0 0))
+  )
   (wire (pts (xy 195.58 59.055) (xy 195.58 65.405))
     (stroke (width 0) (type default) (color 0 0 0 0))
@@
     (stroke (width 0) (type default) (color 0 0 0 0))
   )
+  (wire (pts (xy 168.275 94.615) (xy 163.195 94.615))
+    (stroke (width 0) (type default) (color 0 0 0 0))
+  )
   (wire (pts (xy 129.54 104.775) (xy 129.54 113.665))
     (stroke (width 0) (type default) (color 0 0 0 0))
@@
   )
   (bus (pts (xy 76.835 79.375) (xy 76.835 76.835))
+    (stroke (width 0) (type default) (color 0 0 0 0))
+  )
+  (wire (pts (xy 89.535 94.615) (xy 89.535 97.155))
     (stroke (width 0) (type default) (color 0 0 0 0))
   )
@@
     (effects (font (size 1.27 1.27)) (justify left))
   )
-  (hierarchical_label "Pin16R" (shape input) (at 163.195 94.615 0)
-    (effects (font (size 1.27 1.27)) (justify left))
-  )
   (hierarchical_label "Reg_Ground" (shape input) (at 113.03 59.055 0)
     (effects (font (size 1.27 1.27)) (justify left))
@@
   (hierarchical_label "Pin2R" (shape input) (at 163.195 59.055 0)
     (effects (font (size 1.27 1.27)) (justify left))
-  )
-  (hierarchical_label "Pin16L" (shape input) (at 94.615 94.615 180)
-    (effects (font (size 1.27 1.27)) (justify right))
   )
   (hierarchical_label "Pin11L" (shape input) (at 94.615 81.915 180)
@@
     )
     (property "Datasheet" "" (id 3) (at 104.775 137.795 0)
+      (effects (font (size 1.27 1.27)) hide)
+    )
+    (pin "1")
+  )
+  (symbol (lib_id "power:GND") (at 168.275 97.155 0) (mirror y) (unit 1)
+    (in_bom yes) (on_board yes)
+    (property "Reference" "#PWR0107" (id 0) (at 168.275 103.505 0)
+      (effects (font (size 1.27 1.27)) hide)
+    )
+    (property "Value" "GND" (id 1) (at 168.148 101.5492 0))
+    (property "Footprint" "" (id 2) (at 168.275 97.155 0)
+      (effects (font (size 1.27 1.27)) hide)
+    )
+    (property "Datasheet" "" (id 3) (at 168.275 97.155 0)
       (effects (font (size 1.27 1.27)) hide)
     )
@@
     (pin "32")
   )
+  (symbol (lib_id "power:GND") (at 89.535 97.155 0) (unit 1)
+    (in_bom yes) (on_board yes)
+    (property "Reference" "#PWR0108" (id 0) (at 89.535 103.505 0)
+      (effects (font (size 1.27 1.27)) hide)
+    )
+    (property "Value" "GND" (id 1) (at 89.662 101.5492 0))
+    (property "Footprint" "" (id 2) (at 89.535 97.155 0)
+      (effects (font (size 1.27 1.27)) hide)
+    )
+    (property "Datasheet" "" (id 3) (at 89.535 97.155 0)
+      (effects (font (size 1.27 1.27)) hide)
+    )
+    (pin "1")
+  )
   (symbol (lib_id "Device:R_US") (at 104.775 132.715 0) (unit 1)
