File: NavBoard_Hardware/top_board.kicad_sch (KiCad schematic)
At the start: 10 parts, among them J6 01x03, J7 01x03, J8 Conn_02x16_Separate, J9 6 Pin Molex Micro-Fit

Commit message: Completed routing, added 3D models to IMUs
Parts:
- removed JP1, JP2: Solder Jumper, Jumper:SolderJumper-2_P1.3mm_Open_RoundedPad1.0x1.5mm, symbol Jumper:SolderJumper_2_Open
Connections:
- net Pin13R is gone; now on net GND: J8.29
- net Pin1L is gone; now on net GND: J8.1
- net Pin1R is gone; now on net GND: J8.17
Changed lines of the file:
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@@
 (kicad_sch (version 20211123) (generator eeschema)
   (paper "A4")
+  (junction (at 168.275 94.615) (diameter 0) (color 0 0 0 0)
+  )
   (junction (at 191.135 61.595) (diameter 0) (color 0 0 0 0)
   )
-  (junction (at 235.585 53.975) (diameter 0) (color 0 0 0 0)
-  )
   (junction (at 195.58 59.055) (diameter 0) (color 0 0 0 0)
   )
@@
     (stroke (width 0) (type default) (color 0 0 0 0))
   )
+  (wire (pts (xy 164.465 56.515) (xy 164.465 50.165))
+    (stroke (width 0) (type default) (color 0 0 0 0))
+  )
   (wire (pts (xy 168.275 94.615) (xy 168.275 97.155))
     (stroke (width 0) (type default) (color 0 0 0 0))
@@
     (stroke (width 0) (type default) (color 0 0 0 0))
   )
+  (wire (pts (xy 168.91 50.165) (xy 168.91 50.8))
+    (stroke (width 0) (type default) (color 0 0 0 0))
+  )
   (wire (pts (xy 127 104.775) (xy 127 113.665))
     (stroke (width 0) (type default) (color 0 0 0 0))
@@
     (stroke (width 0) (type default) (color 0 0 0 0))
   )
+  (wire (pts (xy 80.645 56.515) (xy 94.615 56.515))
+    (stroke (width 0) (type default) (color 0 0 0 0))
+  )
   (wire (pts (xy 191.135 61.595) (xy 212.725 61.595))
     (stroke (width 0) (type default) (color 0 0 0 0))
@@
     (stroke (width 0) (type default) (color 0 0 0 0))
   )
+  (wire (pts (xy 80.645 56.515) (xy 80.645 57.15))
+    (stroke (width 0) (type default) (color 0 0 0 0))
+  )
   (wire (pts (xy 104.775 136.525) (xy 104.775 137.795))
     (stroke (width 0) (type default) (color 0 0 0 0))
@@
     (stroke (width 0) (type default) (color 0 0 0 0))
   )
+  (wire (pts (xy 164.465 50.165) (xy 168.91 50.165))
+    (stroke (width 0) (type default) (color 0 0 0 0))
+  )
   (wire (pts (xy 191.135 73.025) (xy 191.135 74.295))
     (stroke (width 0) (type default) (color 0 0 0 0))
@@
     (stroke (width 0) (type default) (color 0 0 0 0))
   )
-  (wire (pts (xy 235.585 53.975) (xy 235.585 54.61))
+  (wire (pts (xy 235.585 53.975) (xy 235.585 62.23))
     (stroke (width 0) (type default) (color 0 0 0 0))
   )
@@
     (stroke (width 0) (type default) (color 0 0 0 0))
   )
+  (wire (pts (xy 168.275 94.615) (xy 168.275 86.995))
+    (stroke (width 0) (type default) (color 0 0 0 0))
+  )
   (wire (pts (xy 132.08 104.775) (xy 132.08 113.665))
     (stroke (width 0) (type default) (color 0 0 0 0))
@@
     (stroke (width 0) (type default) (color 0 0 0 0))
   )
+  (wire (pts (xy 163.195 56.515) (xy 164.465 56.515))
+    (stroke (width 0) (type default) (color 0 0 0 0))
+  )
   (wire (pts (xy 89.535 94.615) (xy 89.535 97.155))
+    (stroke (width 0) (type default) (color 0 0 0 0))
+  )
+  (wire (pts (xy 168.275 86.995) (xy 163.195 86.995))
     (stroke (width 0) (type default) (color 0 0 0 0))
   )
@@
     (effects (font (size 1.27 1.27)) (justify right bottom))
   )
-  (hierarchical_label "Pin1L" (shape input) (at 94.615 56.515 180)
-    (effects (font (size 1.27 1.27)) (justify right))
-  )
   (hierarchical_label "Pin12R" (shape input) (at 163.195 84.455 0)
     (effects (font (size 1.27 1.27)) (justify left))
@@
     (effects (font (size 1.27 1.27)) (justify right))
   )
-  (hierarchical_label "Pin13R" (shape input) (at 163.195 86.995 0)
-    (effects (font (size 1.27 1.27)) (justify left))
-  )
   (hierarchical_label "Reg_Ground" (shape input) (at 113.03 59.055 0)
     (effects (font (size 1.27 1.27)) (justify left))
   )
   (hierarchical_label "Pin5R" (shape input) (at 163.195 66.675 0)
-    (effects (font (size 1.27 1.27)) (justify left))
-  )
-  (hierarchical_label "Pin1R" (shape input) (at 163.195 56.515 0)
     (effects (font (size 1.27 1.27)) (justify left))
   )
@@
     (pin "2")
   )
+  (symbol (lib_id "power:GND") (at 80.645 57.15 0) (unit 1)
+    (in_bom yes) (on_board yes)
+    (property "Reference" "#PWR0115" (id 0) (at 80.645 63.5 0)
+      (effects (font (size 1.27 1.27)) hide)
+    )
+    (property "Value" "GND" (id 1) (at 80.772 61.5442 0))
+    (property "Footprint" "" (id 2) (at 80.645 57.15 0)
+      (effects (font (size 1.27 1.27)) hide)
+    )
+    (property "Datasheet" "" (id 3) (at 80.645 57.15 0)
+      (effects (font (size 1.27 1.27)) hide)
+    )
+    (pin "1")
+  )
   (symbol (lib_id "power:GND") (at 139.7 109.22 0) (mirror y) (unit 1)
     (in_bom yes) (on_board yes)
@@
     )
     (pin "1")
-  )
-  (symbol (lib_id "Jumper:SolderJumper_2_Open") (at 235.585 58.42 90) (unit 1)
-    (in_bom yes) (on_board yes)
-    (property "Reference" "JP2" (id 0) (at 238.76 57.5499 90)
-      (effects (font (size 1.27 1.27)) (justify right))
-    )
-    (property "Value" "Solder Jumper" (id 1) (at 238.76 60.325 90)
-      (effects (font (size 1.27 1.27)) (justify right))
-    )
-    (property "Footprint" "Jumper:SolderJumper-2_P1.3mm_Open_RoundedPad1.0x1.5mm" (id 2) (at 235.585 58.42 0)
-      (effects (font (size 1.27 1.27)) hide)
-    )
-    (property "Datasheet" "~" (id 3) (at 235.585 58.42 0)
-      (effects (font (size 1.27 1.27)) hide)
-    )
-    (pin "1")
-    (pin "2")
   )
   (symbol (lib_id "Nav_Board:Conn_02x16_Separate") (at 99.695 75.565 0) (unit 1)
@@
     )
     (property "Datasheet" "" (id 3) (at 235.585 62.23 0)
-      (effects (font (size 1.27 1.27)) hide)
-    )
-    (pin "1")
-  )
-  (symbol (lib_id "power:+3V3") (at 235.585 46.355 0) (unit 1)
-    (in_bom yes) (on_board yes)
-    (property "Reference" "#PWR041" (id 0) (at 235.585 50.165 0)
-      (effects (font (size 1.27 1.27)) hide)
-    )
-    (property "Value" "+3V3" (id 1) (at 235.585 41.91 0))
-    (property "Footprint" "" (id 2) (at 235.585 46.355 0)
-      (effects (font (size 1.27 1.27)) hide)
-    )
-    (property "Datasheet" "" (id 3) (at 235.585 46.355 0)
       (effects (font (size 1.27 1.27)) hide)
     )
@@
     (pin "32")
   )
+  (symbol (lib_id "power:GND") (at 168.91 50.8 0) (mirror y) (unit 1)
+    (in_bom yes) (on_board yes)
+    (property "Reference" "#PWR0116" (id 0) (at 168.91 57.15 0)
+      (effects (font (size 1.27 1.27)) hide)
+    )
+    (property "Value" "GND" (id 1) (at 168.783 55.1942 0))
+    (property "Footprint" "" (id 2) (at 168.91 50.8 0)
+      (effects (font (size 1.27 1.27)) hide)
+    )
+    (property "Datasheet" "" (id 3) (at 168.91 50.8 0)
+      (effects (font (size 1.27 1.27)) hide)
+    )
+    (pin "1")
+  )
   (symbol (lib_id "power:GND") (at 89.535 97.155 0) (unit 1)
     (in_bom yes) (on_board yes)
@@
       (effects (font (size 1.27 1.27)) hide)
     )
-    (pin "1")
-    (pin "2")
-  )
-  (symbol (lib_id "Jumper:SolderJumper_2_Open") (at 235.585 50.165 270) (unit 1)
-    (in_bom yes) (on_board yes)
-    (property "Reference" "JP1" (id 0) (at 241.935 47.625 90)
-      (effects (font (size 1.27 1.27)) (justify right))
-    )
-    (property "Value" "Solder Jumper" (id 1) (at 252.095 50.165 90)
-      (effects (font (size 1.27 1.27)) (justify right))
-    )
-    (property "Footprint" "Jumper:SolderJumper-2_P1.3mm_Open_RoundedPad1.0x1.5mm" (id 2) (at 235.585 50.165 0)
-      (effects (font (size 1.27 1.27)) hide)
-    )
-    (property "Datasheet" "~" (id 3) (at 235.585 50.165 0)
-      (effects (font (size 1.27 1.27)) hide)
-    )
