File: NavBoard_Hardware/_autosave-NavBoard_Hardware.kicad_pcb (KiCad board)
At the start: 4 copper layers, 100 x 31.6 mm, 11 parts, among them J3 Ethernet Jack w/ Magnetics, J9 6 Pin Molex Micro-Fit, U2 OKI-5V, U5 Teensy4.1, U6 TSR 2-2450

Commit message: Realized this could all fit on a single board
Parts:
- removed U5: Teensy4.1, Nav_Board:Teensy41_Suspended
- removed U6: TSR 2-2450, Converter_DCDC:Converter_DCDC_TRACO_TSR-1_THT
- added C1: 0.1uF, Capacitor_SMD:C_0603_1608Metric_Pad1.08x0.95mm_HandSolder, F.Cu at (62.9, 131.6)
- added C10: 0.1uF, Capacitor_SMD:C_0603_1608Metric_Pad1.08x0.95mm_HandSolder, F.Cu at (30.2, 84.6)
- added C11: 0.47uF, Capacitor_SMD:C_0603_1608Metric_Pad1.08x0.95mm_HandSolder, F.Cu at (30.2, 87.1)
- added C12: 0.1uF, Capacitor_SMD:C_0603_1608Metric_Pad1.08x0.95mm_HandSolder, F.Cu at (30.2, 50.6)
- added C2: 1uF, Capacitor_SMD:C_0603_1608Metric_Pad1.08x0.95mm_HandSolder, F.Cu at (58.5, 136.6)
- added C3: 0.1uF, Capacitor_SMD:C_0603_1608Metric_Pad1.08x0.95mm_HandSolder, F.Cu at (58.5, 134.1)
- added C4: 0.47uF, Capacitor_SMD:C_0603_1608Metric_Pad1.08x0.95mm_HandSolder, F.Cu at (62.9, 129.1)
- added C5: 22uF 50V, Capacitor_SMD:C_1206_3216Metric_Pad1.33x1.80mm_HandSolder, F.Cu at (87.9, 28.0)
- added C6: 10uF, Capacitor_SMD:C_0603_1608Metric_Pad1.08x0.95mm_HandSolder, F.Cu at (100.6, 17.3)
- added C7: 0.1uF, Capacitor_SMD:C_0603_1608Metric_Pad1.08x0.95mm_HandSolder, F.Cu at (87.1, 30.9)
- added C8: 10nF, Capacitor_SMD:C_0603_1608Metric_Pad1.08x0.95mm_HandSolder, F.Cu at (39.8, 77.5)
- added C9: 2.2uF, Capacitor_SMD:C_0603_1608Metric_Pad1.08x0.95mm_HandSolder, F.Cu at (34.6, 82.0)
- added D1: GREEN, LED_SMD:LED_0603_1608Metric_Pad1.05x0.95mm_HandSolder, F.Cu at (30.3, 42.2)
- added J3: Conn_02x16_Separate_1, Nav_Board:PinSocket_2x16_P2.54mm_Vertical_Nav_Board, B.Cu at (157.6, 98.8)
- added R1: 4.7k, Resistor_SMD:R_0603_1608Metric_Pad0.98x0.95mm_HandSolder, F.Cu at (58.5, 131.6)
- added R10: 4.7k, Resistor_SMD:R_0603_1608Metric_Pad0.98x0.95mm_HandSolder, F.Cu at (34.6, 44.8)
- added R11: 4.7k, Resistor_SMD:R_0603_1608Metric_Pad0.98x0.95mm_HandSolder, F.Cu at (73.0, 17.3)
- added R12: 100Ω, Resistor_SMD:R_0603_1608Metric_Pad0.98x0.95mm_HandSolder, F.Cu at (73.0, 19.8)
- added R2: 4.7k, Resistor_SMD:R_0603_1608Metric_Pad0.98x0.95mm_HandSolder, F.Cu at (58.5, 129.1)
- added R3: 4.7k, Resistor_SMD:R_0603_1608Metric_Pad0.98x0.95mm_HandSolder, F.Cu at (63.8, 124.2)
- added R4: 4.7k, Resistor_SMD:R_0603_1608Metric_Pad0.98x0.95mm_HandSolder, F.Cu at (67.2, 126.7)
- added R5: 4.7k, Resistor_SMD:R_0603_1608Metric_Pad0.98x0.95mm_HandSolder, F.Cu at (68.2, 124.2)
- added R6: 4.7k, Resistor_SMD:R_0603_1608Metric_Pad0.98x0.95mm_HandSolder, F.Cu at (35.4, 77.5)
- added R7: 4.7k, Resistor_SMD:R_0603_1608Metric_Pad0.98x0.95mm_HandSolder, F.Cu at (30.2, 82.0)
- added R8: 4.7k, Resistor_SMD:R_0603_1608Metric_Pad0.98x0.95mm_HandSolder, F.Cu at (30.2, 44.8)
- added R9: 4.7k, Resistor_SMD:R_0603_1608Metric_Pad0.98x0.95mm_HandSolder, F.Cu at (34.6, 42.2)
- added TP1: TestPoint, TestPoint:TestPoint_Pad_D1.5mm, F.Cu at (66.8, 129.7)
- added TP2: TestPoint, TestPoint:TestPoint_Pad_D1.5mm, F.Cu at (72.1, 124.7)
- added TP3: TestPoint, TestPoint:TestPoint_Pad_D1.5mm, F.Cu at (38.5, 80.5)
- added TP4: TestPoint, TestPoint:TestPoint_Pad_D1.5mm, F.Cu at (34.2, 85.1)
- added U3: OKI-5V, Nav_Board:OKI_Vertical_TSR, F.Cu at (120.4, 95.2)
- added U4: ICM-20608-G, Nav_Board:ICM-20608-G, F.Cu at (30.7, 78.5)
- H1, H2, H3, H4: renamed from ?; value (none) -> MountingHole_Pad
- U2: value OKI-5V -> BHI160B; footprint MRDT_Devices:OKI_Horizontal -> Nav_Board:BHI160B
- moved J4 113.2 mm to (282.1, 85.0)
- moved U2 77.6 mm to (59.1, 125.2), turned to 0 degrees
- moved U1 8.25 mm to (147.5, 97.6)
- renumbered J3 to J2, J9 to J4, U5 to U1
Connections:
- H1 pad 1: (no net) -> GND
- H2 pad 1: (no net) -> GND
- H3 pad 1: (no net) -> GND
- H4 pad 1: (no net) -> GND
- J4 pad 3: /Top Board/GPS-TX -> /Pin27
- J4 pad 4: /Top Board/GPS-RX -> /Pin26
- J4 pad 5: /Top Board/GPS-SDA -> /Pin17
- J4 pad 6: /Top Board/GPS-SCL -> /Pin16
- U1 pad 1: (no net) -> GND
- U1 pad 10: (no net) -> /Pin10
- U1 pad 11: (no net) -> /Pin11
- U1 pad 12: (no net) -> /Pin12
- U1 pad 13: (no net) -> /Pin13
- U1 pad 14: (no net) -> /Pin14
- U1 pad 15: (no net) -> +3V3
- U1 pad 16: (no net) -> /Pin16
- U1 pad 17: (no net) -> /Pin17
- U1 pad 18: (no net) -> /Pin18
- U1 pad 19: (no net) -> /Pin19
- U1 pad 2: (no net) -> /Pin2
- U1 pad 20: (no net) -> /Pin20
- U1 pad 21: (no net) -> /Pin21
- U1 pad 22: (no net) -> /Pin22
- U1 pad 23: (no net) -> /Pin23
- U1 pad 24: (no net) -> GND
- U1 pad 25: (no net) -> GND
- U1 pad 26: (no net) -> /Pin26
- U1 pad 27: (no net) -> /Pin27
- U1 pad 28: (no net) -> GND
- U1 pad 29: (no net) -> /Pin29
- U1 pad 3: (no net) -> /Pin3
- U1 pad 30: (no net) -> /Pin30
- U1 pad 31: (no net) -> /Pin31
- U1 pad 32: (no net) -> /Pin32
- U1 pad 33: (no net) -> /Pin33
- U1 pad 34: (no net) -> GND
- U1 pad 35: (no net) -> /Pin35
- U1 pad 36: (no net) -> /Pin36
- U1 pad 37: (no net) -> /Pin37
- U1 pad 38: (no net) -> /Pin38
- U1 pad 39: (no net) -> /Pin39
- U1 pad 4: (no net) -> /Pin4
- U1 pad 40: (no net) -> GND
- U1 pad 41: (no net) -> /Pin41
- U1 pad 42: (no net) -> /Pin42
- U1 pad 43: (no net) -> /Pin43
- U1 pad 44: (no net) -> /Pin44
- U1 pad 45: (no net) -> /Pin45
- U1 pad 46: (no net) -> +3V3
- U1 pad 47: (no net) -> GND
- U1 pad 48: (no net) -> +5V
- U1 pad 5: (no net) -> /Pin5
- U1 pad 6: (no net) -> /Pin6
- U1 pad 60: (no net) -> /PinEthernet_R+
- U1 pad 61: (no net) -> /PinEthernet_LED+
- U1 pad 62: (no net) -> /PinEthernet_T-
- U1 pad 63: (no net) -> /PinEthernet_T+
- U1 pad 64: (no net) -> GND
- U1 pad 65: (no net) -> /PinEthernet_R-
- U1 pad 7: (no net) -> /Pin7
- U1 pad 8: (no net) -> /Pin8
- U1 pad 9: (no net) -> GND
- U2 pad 1: +12V -> (no net)
- U2 pad 2: GND -> (no net)
- U2 pad 3: +5V -> Net-(R2-Pad1)
Other:
- board text removed: "TSR 5V"

Commit message: Most connections made on schematic
Parts:
- removed J3: Conn_02x16_Separate_1, Nav_Board:PinSocket_2x16_P2.54mm_Vertical_Nav_Board
- removed the U2 at (59.1, 125.2)
- added D2: BLUE, LED_SMD:LED_0603_1608Metric_Pad1.05x0.95mm_HandSolder, F.Cu at (214.0, 117.6)
- added D3: BLUE, LED_SMD:LED_0603_1608Metric_Pad1.05x0.95mm_HandSolder, F.Cu at (218.4, 115.0)
- added D4: BLUE, LED_SMD:LED_0603_1608Metric_Pad1.05x0.95mm_HandSolder, F.Cu at (214.0, 115.0)
- added R13: 4.7k, Resistor_SMD:R_0603_1608Metric_Pad0.98x0.95mm_HandSolder, F.Cu at (193.9, 130.3)
- added R14: 4.7k, Resistor_SMD:R_0603_1608Metric_Pad0.98x0.95mm_HandSolder, F.Cu at (188.7, 134.9)
- added R15: 100, Resistor_SMD:R_0603_1608Metric_Pad0.98x0.95mm_HandSolder, F.Cu at (222.7, 115.0)
- added R16: 100, Resistor_SMD:R_0603_1608Metric_Pad0.98x0.95mm_HandSolder, F.Cu at (218.3, 117.6)
- added R17: 100, Resistor_SMD:R_0603_1608Metric_Pad0.98x0.95mm_HandSolder, F.Cu at (214.0, 120.2)
- added U3: BHI160B, Nav_Board:BHI160B, F.Cu at (77.4, 65.0)
- C10: value 0.1uF -> 2.2uF
- C11, C4: value 0.47uF -> 0.1uF
- C12: value 0.1uF -> 0.47uF
- C2: value 1uF -> 22uF 50V; footprint Capacitor_SMD:C_0603_1608Metric_Pad1.08x0.95mm_HandSolder -> Capacitor_SMD:C_1206_3216Metric_Pad1.33x1.80mm_HandSolder
- C3: value 0.1uF -> 10uF
- C5: value 22uF 50V -> 0.1uF; footprint Capacitor_SMD:C_1206_3216Metric_Pad1.33x1.80mm_HandSolder -> Capacitor_SMD:C_0603_1608Metric_Pad1.08x0.95mm_HandSolder
- C6: value 10uF -> 1uF
- C8: value 10nF -> 0.47uF
- C9: value 2.2uF -> 10nF
- R1, R2: value 4.7k -> 0ohm
- R12: value 100Ω -> 4.7k
- R5: value 4.7k -> 100Ω
- moved C12 184.5 mm to (193.1, 137.4)
- moved C9 170.6 mm to (198.2, 130.3)
- moved C10 170.4 mm to (193.1, 134.9)
- moved TP3 170.4 mm to (200.6, 133.4)
- moved TP4 169.8 mm to (197.0, 133.4)
- moved U4 167.1 mm to (189.2, 131.4)
- moved C11 166.3 mm to (188.7, 137.4)
- moved R1 110.0 mm to (129.0, 47.2)
- moved R7 103.1 mm to (128.9, 52.2)
- moved C1 102.5 mm to (124.6, 49.8)
- moved J1 101.8 mm to (180.4, 89.5), turned to -90 degrees
- moved R2 100.5 mm to (120.2, 49.8)
- moved R3 98.9 mm to (128.9, 49.7)
- moved C2 96.1 mm to (118.6, 61.6)
- moved R5 95.4 mm to (124.6, 47.2)
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- renumbered J4 to J1, U3 to U2
Connections:
- net /Main Board/ETHERNET_LED renamed /ETHERNET_LED
- net /Main Board/ETHERNET_RX+ renamed /ETHERNET_RX+
- net /Main Board/ETHERNET_RX- renamed /ETHERNET_RX-
- net /Main Board/ETHERNET_TX+ renamed /ETHERNET_TX+
- net /Main Board/ETHERNET_TX- renamed /ETHERNET_TX-
- C1 pad 1: +3V3 -> Net-(C1-Pad1)
- C11 pad 1: Net-(C11-Pad1) -> +3V3
- C2 pad 1: +3V3 -> +12V
- C3 pad 1: +3V3 -> +5V
- C4 pad 1: Net-(C4-Pad1) -> +5V
- C5 pad 1: +12V -> +3V3
- C6 pad 1: +5V -> +3V3
- C7 pad 1: +5V -> +3V3
- C8 pad 1: +3V3 -> Net-(C8-Pad1)
- J1 pad 3: /Pin27 -> /GPS-TX
- J1 pad 4: /Pin26 -> /GPS-RX
- J1 pad 5: /Pin17 -> /GPS-SDA
- J1 pad 6: /Pin16 -> /GPS-SCL
- J2 pad 2: Net-(C12-Pad1) -> Net-(C1-Pad1)
- J2 pad 5: Net-(C12-Pad1) -> Net-(C1-Pad1)
- R1 pad 1: Net-(R1-Pad1) -> /GPS-SCL
- R1 pad 2: GND -> Net-(R1-Pad2)
- R10 pad 1: /Pin17 -> Net-(R10-Pad1)
- R11 pad 1: /Pin16 -> Net-(R11-Pad1)
- R12 pad 1: +5V -> Net-(R12-Pad1)
- R12 pad 2: Net-(D1-Pad2) -> GND
- R2 pad 1: Net-(R2-Pad1) -> /GPS-SDA
- R2 pad 2: GND -> Net-(R2-Pad2)
- R3 pad 1: Net-(R3-Pad1) -> Net-(R2-Pad2)
- R4 pad 1: Net-(R4-Pad1) -> Net-(R1-Pad2)
- R5 pad 1: Net-(R5-Pad1) -> +5V
- R5 pad 2: GND -> Net-(D1-Pad2)
- R6 pad 1: Net-(R6-Pad1) -> /BHI-SCL
- R7 pad 1: Net-(R7-Pad1) -> /BHI-SDA
- R8 pad 1: /Pin38 -> Net-(R8-Pad1)
- R9 pad 1: /Pin39 -> Net-(R9-Pad1)
- TP1 pad 1: Net-(R2-Pad1) -> Net-(R9-Pad1)
- TP2 pad 1: Net-(R1-Pad1) -> Net-(R8-Pad1)
- TP3 pad 1: Net-(R6-Pad1) -> Net-(R13-Pad1)
- TP4 pad 1: Net-(R7-Pad1) -> Net-(R14-Pad1)
- U1 pad 10: /Pin10 -> /BHI-SDA
- U1 pad 11: /Pin11 -> /BHI-SCL
- U1 pad 12: /Pin12 -> unconnected-(U1-Pad12)
- U1 pad 13: /Pin13 -> unconnected-(U1-Pad13)
- U1 pad 14: /Pin14 -> /ICM-SCLK
- U1 pad 16: /Pin16 -> unconnected-(U1-Pad16)
- U1 pad 17: /Pin17 -> unconnected-(U1-Pad17)
- U1 pad 18: /Pin18 -> unconnected-(U1-Pad18)
- U1 pad 19: /Pin19 -> unconnected-(U1-Pad19)
- U1 pad 2: /Pin2 -> unconnected-(U1-Pad2)
- U1 pad 20: /Pin20 -> unconnected-(U1-Pad20)
- U1 pad 21: /Pin21 -> unconnected-(U1-Pad21)
- U1 pad 22: /Pin22 -> /GPS-TX
- U1 pad 23: /Pin23 -> /GPS-RX
- U1 pad 24: GND -> unconnected-(U1-Pad24)
- U1 pad 25: GND -> unconnected-(U1-Pad25)
- U1 pad 26: /Pin26 -> unconnected-(U1-Pad26)
- U1 pad 27: /Pin27 -> unconnected-(U1-Pad27)
- U1 pad 28: GND -> unconnected-(U1-Pad28)
- U1 pad 29: /Pin29 -> unconnected-(U1-Pad29)
- U1 pad 3: /Pin3 -> unconnected-(U1-Pad3)
- U1 pad 30: /Pin30 -> unconnected-(U1-Pad30)
- U1 pad 31: /Pin31 -> unconnected-(U1-Pad31)
- U1 pad 32: /Pin32 -> /GPS-SDA
- U1 pad 33: /Pin33 -> /GPS-SCL
- U1 pad 35: /Pin35 -> /ICM-MISO
- U1 pad 36: /Pin36 -> /ICM-MOSI
- U1 pad 37: /Pin37 -> /ICM-CS
- U1 pad 38: /Pin38 -> unconnected-(U1-Pad38)
- U1 pad 39: /Pin39 -> unconnected-(U1-Pad39)
- U1 pad 4: /Pin4 -> unconnected-(U1-Pad4)
- U1 pad 40: GND -> unconnected-(U1-Pad40)
- U1 pad 41: /Pin41 -> unconnected-(U1-Pad41)
- U1 pad 42: /Pin42 -> unconnected-(U1-Pad42)
- U1 pad 43: /Pin43 -> unconnected-(U1-Pad43)
- U1 pad 44: /Pin44 -> unconnected-(U1-Pad44)
- U1 pad 45: /Pin45 -> unconnected-(U1-Pad45)
- U1 pad 5: /Pin5 -> unconnected-(U1-Pad5)
- U1 pad 6: /Pin6 -> unconnected-(U1-Pad6)
- U1 pad 7: /Pin7 -> unconnected-(U1-Pad7)
- U1 pad 8: /Pin8 -> unconnected-(U1-Pad8)
- U1 pad 9: GND -> unconnected-(U1-Pad9)
- U4 pad 14: Net-(C11-Pad1) -> Net-(C12-Pad1)
- U4 pad 2: /Pin35 -> /ICM-SCLK
- U4 pad 3: /Pin13 -> /ICM-MOSI
- U4 pad 4: /Pin14 -> /ICM-MISO
- U4 pad 5: /Pin12 -> /ICM-CS
- U4 pad 6: Net-(R6-Pad1) -> Net-(R13-Pad1)
- U4 pad 8: Net-(R7-Pad1) -> Net-(R14-Pad1)
Routing:
- added copper zone on In2.Cu, net +3V3
- added copper zone on B.Cu, net GND
- added copper zone on F.Cu, net GND
- added copper zone on In1.Cu, net GND
