File: NavBoard_Hardware/component_sheets/ICM-20608.kicad_sch (KiCad schematic)
At the start: 9 parts, among them U4 ICM-20608-G

Commit message: Most connections made on schematic
Parts:
- renumbered C9 to C10, C10 to C11, C11 to C12, C8 to C9, R6 to R13, R7 to R14
Other:
- title: MRDT NavBoard - ICM-20608-G -> MRDT NavBoard
Changed lines of the file:
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@@
   (paper "A4")
   (title_block
-    (title "MRDT NavBoard - ICM-20608-G")
-    (date "2022-09-15")
-    (rev "1, 2023")
+    (title "MRDT NavBoard")
+    (date "2022-10-08")
+    (rev "3, 2023")
     (company "Thomas Francois, Missouri S&T Mars Rover Design Team")
-    (comment 1 "Inertial Measurement Unit and Supporting Components")
-    (comment 2 "Provides Position & Acceleration Data")
+    (comment 1 "Teensy 4.1 Daughter Boards and Modules")
+    (comment 2 "and accelerometers")
+    (comment 3 "These boards are to be stacked together, and connects the Teensy to power, ethernet, ")
   )
   (junction (at 142.24 71.12) (diameter 0) (color 0 0 0 0)
@@
     (effects (font (size 1.27 1.27)) (justify right))
   )
-  (symbol (lib_id "Device:R_US") (at 117.475 106.045 0) (unit 1)
-    (in_bom yes) (on_board yes)
-    (property "Reference" "R7" (id 0) (at 111.76 105.41 0)
+  (symbol (lib_id "Device:R_US") (at 117.475 106.045 0)
+    (in_bom yes) (on_board yes)
+    (property "Reference" "R14" (id 0) (at 111.76 105.41 0)
       (effects (font (size 1.27 1.27)) (justify left))
     )
@@
     (pin "2")
   )
-  (symbol (lib_id "Device:R_US") (at 175.26 97.155 0) (unit 1)
-    (in_bom yes) (on_board yes)
-    (property "Reference" "R6" (id 0) (at 177.165 96.52 0)
+  (symbol (lib_id "Device:R_US") (at 175.26 97.155 0)
+    (in_bom yes) (on_board yes)
+    (property "Reference" "R13" (id 0) (at 177.165 96.52 0)
       (effects (font (size 1.27 1.27)) (justify left))
     )
@@
     (pin "2")
   )
-  (symbol (lib_id "Device:C") (at 142.24 76.2 0) (unit 1)
-    (in_bom yes) (on_board yes)
-    (property "Reference" "C10" (id 0) (at 137.16 74.93 0)
+  (symbol (lib_id "Device:C") (at 142.24 76.2 0)
+    (in_bom yes) (on_board yes)
+    (property "Reference" "C11" (id 0) (at 137.16 74.93 0)
       (effects (font (size 1.27 1.27)) (justify left))
     )
@@
     (pin "2")
   )
-  (symbol (lib_id "power:GND") (at 163.83 81.28 0) (unit 1)
-    (in_bom yes) (on_board yes)
-    (property "Reference" "#PWR026" (id 0) (at 163.83 87.63 0)
+  (symbol (lib_id "power:GND") (at 163.83 81.28 0)
+    (in_bom yes) (on_board yes)
+    (property "Reference" "#PWR040" (id 0) (at 163.83 87.63 0)
       (effects (font (size 1.27 1.27)) hide)
     )
@@
     (pin "1")
   )
-  (symbol (lib_id "Device:C") (at 133.35 76.2 0) (mirror y) (unit 1)
-    (in_bom yes) (on_board yes)
-    (property "Reference" "C9" (id 0) (at 130.429 75.0316 0)
+  (symbol (lib_id "Device:C") (at 133.35 76.2 0) (mirror y)
+    (in_bom yes) (on_board yes)
+    (property "Reference" "C10" (id 0) (at 130.429 75.0316 0)
       (effects (font (size 1.27 1.27)) (justify left))
     )
@@
     (pin "2")
   )
-  (symbol (lib_id "power:GND") (at 175.26 102.87 0) (unit 1)
-    (in_bom yes) (on_board yes)
-    (property "Reference" "#PWR027" (id 0) (at 175.26 109.22 0)
+  (symbol (lib_id "power:GND") (at 175.26 102.87 0)
+    (in_bom yes) (on_board yes)
+    (property "Reference" "#PWR041" (id 0) (at 175.26 109.22 0)
       (effects (font (size 1.27 1.27)) hide)
     )
@@
     (pin "1")
   )
-  (symbol (lib_id "Device:C") (at 123.825 76.2 0) (mirror y) (unit 1)
-    (in_bom yes) (on_board yes)
-    (property "Reference" "C8" (id 0) (at 120.65 74.93 0)
+  (symbol (lib_id "Device:C") (at 123.825 76.2 0) (mirror y)
+    (in_bom yes) (on_board yes)
+    (property "Reference" "C9" (id 0) (at 120.65 74.93 0)
       (effects (font (size 1.27 1.27)) (justify left))
     )
@@
     (pin "2")
   )
-  (symbol (lib_id "power:GND") (at 133.35 81.28 0) (unit 1)
-    (in_bom yes) (on_board yes)
-    (property "Reference" "#PWR025" (id 0) (at 133.35 87.63 0)
+  (symbol (lib_id "power:GND") (at 133.35 81.28 0)
+    (in_bom yes) (on_board yes)
+    (property "Reference" "#PWR039" (id 0) (at 133.35 87.63 0)
       (effects (font (size 1.27 1.27)) hide)
     )
@@
     (pin "1")
   )
-  (symbol (lib_id "power:GND") (at 117.475 111.76 0) (unit 1)
-    (in_bom yes) (on_board yes)
-    (property "Reference" "#PWR028" (id 0) (at 117.475 118.11 0)
+  (symbol (lib_id "power:GND") (at 117.475 111.76 0)
+    (in_bom yes) (on_board yes)
+    (property "Reference" "#PWR042" (id 0) (at 117.475 118.11 0)
       (effects (font (size 1.27 1.27)) hide)
     )
@@
     (pin "1")
   )
-  (symbol (lib_id "Connector:TestPoint") (at 117.475 99.695 0) (mirror y) (unit 1)
+  (symbol (lib_id "Connector:TestPoint") (at 117.475 99.695 0) (mirror y)
     (in_bom yes) (on_board yes)
     (property "Reference" "TP4" (id 0) (at 116.205 96.52 0)
@@
     (pin "1")
   )
-  (symbol (lib_id "power:GND") (at 147.32 113.665 0) (unit 1)
-    (in_bom yes) (on_board yes)
-    (property "Reference" "#PWR029" (id 0) (at 147.32 120.015 0)
+  (symbol (lib_id "power:GND") (at 147.32 113.665 0)
+    (in_bom yes) (on_board yes)
+    (property "Reference" "#PWR043" (id 0) (at 147.32 120.015 0)
       (effects (font (size 1.27 1.27)) hide)
     )
@@
     (pin "1")
   )
-  (symbol (lib_id "Device:C") (at 163.83 76.2 0) (unit 1)
-    (in_bom yes) (on_board yes)
-    (property "Reference" "C11" (id 0) (at 166.37 74.93 0)
+  (symbol (lib_id "Device:C") (at 163.83 76.2 0)
+    (in_bom yes) (on_board yes)
+    (property "Reference" "C12" (id 0) (at 166.37 74.93 0)
       (effects (font (size 1.27 1.27)) (justify left))
     )
@@
     (pin "2")
   )
-  (symbol (lib_id "MRDT_Sensors:ICM-20608-G") (at 148.59 97.79 0) (unit 1)
+  (symbol (lib_id "MRDT_Sensors:ICM-20608-G") (at 148.59 97.79 0)
     (in_bom yes) (on_board yes)
     (property "Reference" "U4" (id 0) (at 160.655 110.49 0)
@@
     (pin "9")
   )
-  (symbol (lib_id "power:+3V3") (at 133.35 69.215 0) (unit 1)
-    (in_bom yes) (on_board yes)
-    (property "Reference" "#PWR024" (id 0) (at 133.35 73.025 0)
+  (symbol (lib_id "power:+3V3") (at 133.35 69.215 0)
+    (in_bom yes) (on_board yes)
+    (property "Reference" "#PWR038" (id 0) (at 133.35 73.025 0)
       (effects (font (size 1.27 1.27)) hide)
     )
@@
     (pin "1")
   )
-  (symbol (lib_id "Connector:TestPoint") (at 175.26 89.535 0) (unit 1)
+  (symbol (lib_id "Connector:TestPoint") (at 175.26 89.535 0)
     (in_bom yes) (on_board yes)
     (property "Reference" "TP3" (id 0) (at 176.53 86.36 0)
