File: NavBoard_Hardware/component_sheets/OKI-5V.kicad_sch (KiCad schematic)
At the start: 4 parts, among them U3 OKI-5V

Commit message: Most connections made on schematic
Parts:
- renumbered C5 to C2, C6 to C3, C7 to C4, U3 to U2
Changed lines of the file:
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@@
   (title_block
     (title "MRDT NavBoard")
-    (rev "1, 2023")
+    (date "2022-10-08")
+    (rev "3, 2023")
     (company "Thomas Francois, Missouri S&T Mars Rover Design Team")
-    (comment 1 "OKI 5V Voltage Regulator")
-    (comment 2 "Provides stable 5V from 12V input")
+    (comment 1 "Teensy 4.1 Daughter Boards and Modules")
+    (comment 2 "and accelerometers")
+    (comment 3 "These boards are to be stacked together, and connects the Teensy to power, ethernet, ")
   )
   (junction (at 146.05 102.235) (diameter 0) (color 0 0 0 0)
@@
     (effects (font (size 1.27 1.27)) (justify right))
   )
-  (symbol (lib_id "Device:C_Polarized_US") (at 127.635 97.155 0) (unit 1)
+  (symbol (lib_id "Device:C_Polarized_US") (at 127.635 97.155 0)
     (in_bom yes) (on_board yes)
-    (property "Reference" "C5" (id 0) (at 130.556 95.9866 0)
+    (property "Reference" "C2" (id 0) (at 130.556 95.9866 0)
       (effects (font (size 1.27 1.27)) (justify left))
     )
@@
     (pin "2")
   )
-  (symbol (lib_id "Device:C_Polarized_US") (at 158.115 97.155 0) (unit 1)
+  (symbol (lib_id "Device:C_Polarized_US") (at 158.115 97.155 0)
     (in_bom yes) (on_board yes)
-    (property "Reference" "C6" (id 0) (at 161.1122 95.9866 0)
+    (property "Reference" "C3" (id 0) (at 161.1122 95.9866 0)
       (effects (font (size 1.27 1.27)) (justify left))
     )
@@
     (pin "2")
   )
-  (symbol (lib_id "power:+5V") (at 169.545 88.265 0) (unit 1)
+  (symbol (lib_id "power:+5V") (at 169.545 88.265 0)
     (in_bom yes) (on_board yes) (fields_autoplaced)
-    (property "Reference" "#PWR022" (id 0) (at 169.545 92.075 0)
+    (property "Reference" "#PWR027" (id 0) (at 169.545 92.075 0)
       (effects (font (size 1.27 1.27)) hide)
     )
@@
     (pin "1")
   )
-  (symbol (lib_id "power:+12V") (at 127.635 88.265 0) (unit 1)
+  (symbol (lib_id "power:+12V") (at 127.635 88.265 0)
     (in_bom yes) (on_board yes) (fields_autoplaced)
-    (property "Reference" "#PWR021" (id 0) (at 127.635 92.075 0)
+    (property "Reference" "#PWR026" (id 0) (at 127.635 92.075 0)
       (effects (font (size 1.27 1.27)) hide)
     )
@@
     (pin "1")
   )
-  (symbol (lib_id "Device:C_Polarized_US") (at 169.545 97.155 0) (unit 1)
+  (symbol (lib_id "Device:C_Polarized_US") (at 169.545 97.155 0)
     (in_bom yes) (on_board yes)
-    (property "Reference" "C7" (id 0) (at 172.5422 95.9866 0)
+    (property "Reference" "C4" (id 0) (at 172.5422 95.9866 0)
       (effects (font (size 1.27 1.27)) (justify left))
     )
@@
     (pin "2")
   )
-  (symbol (lib_id "MRDT_Devices:OKI") (at 139.065 93.345 0) (unit 1)
+  (symbol (lib_id "MRDT_Devices:OKI") (at 139.065 93.345 0)
     (in_bom yes) (on_board yes)
-    (property "Reference" "U3" (id 0) (at 140.335 94.615 0)
+    (property "Reference" "U2" (id 0) (at 140.335 94.615 0)
       (effects (font (size 1.524 1.524)))
     )
@@
     (pin "3")
   )
-  (symbol (lib_id "power:GND") (at 146.05 104.775 0) (unit 1)
+  (symbol (lib_id "power:GND") (at 146.05 104.775 0)
     (in_bom yes) (on_board yes) (fields_autoplaced)
-    (property "Reference" "#PWR023" (id 0) (at 146.05 111.125 0)
+    (property "Reference" "#PWR028" (id 0) (at 146.05 111.125 0)
       (effects (font (size 1.27 1.27)) hide)
     )
